File: mcu.kicad_sch (KiCad schematic)
At the start: 27 parts, among them J2 Conn_01x40, Q5 Q_NMOS_GSD, SW1 BOOT, SW2 RESET, U2 ESP32-C6-WROOM-1, U4 RV-3028-C7

Commit message: KiCad schematic updates - 2026-09-07
Parts:
- added TP6, TP7, TP8: TestPoint, symbol Connector:TestPoint
- C5, C6, C7: footprint (none) -> Capacitor_SMD:C_01005_0402Metric
- J2: footprint (none) -> Molex_541324062:CON_541324062_MOL
- R1, R15, R16, R17, R18, R19, R20, R22, R25, R26: footprint (none) -> Resistor_SMD:R_01005_0402Metric
Connections:
- net RTC_I2C_SDA is gone; now on net RTC_SDA: R26.1, U4.4 (SDA)
- net BL_SINK: now also R15.1, R16.1, R18.1
- net MCU_3V3: no longer C5.1, C6.1, C9.1, R25.1, U2.2 (3V3), U4.7 (VDD)
- net PD_I2C_SCL_3V3: now also TP6.1
- net PD_I2C_SDA_3V3: now also TP7.1
- net PD_INT_3V3: now also TP8.1
- net at R22.1: now also C10.1, U4.6 (VBACKUP); no longer BT1.1 (+)
- new net: BT1.1 (+), R22.2
- new net +3.3V: C5.1, C6.1, C9.1, R25.1, U2.2 (3V3), U4.7 (VDD)
Other:
- note added: "Boşta kalan pinlere 22R sonrası bir test point koyarak daha sonra kullanılabilir halde tasarım yapalım."
- note added: "ESP32 decoupling kapasiteleri pin ile bağlantılı gösterilmesi layout çiziminde bunların pine yakın konumlandırılması gerektiğini hatırlatır."
- note added: "ESP32'yi nasıl programlayacağız? Uart pinlerini bağlamamız gerekiyor mu?"
- note added: "Encoder seçimi yapılarak uygun şekilde bağlantısı yapılmalı!"
- note added: "LCD konnektörü başka bir sayfaya taşınmalı"
- note added: "PORT tanımlamaları yatay konumlandırılmalı ve giriş, çıkış gibi gösterimleri doğru yapılmalı."
- note added: "Pin ataması ESP32'nin uygunlupu kontrol edilerek birbirine yakın pinler ile bağlanmalı. Bu layout çizimini kolaylaştırır."
- note added: "RTC pil konusu netleştirilecek."
- moved on the sheet: BT1, C5, C6, J2, Q5, R1, R10, R15, R16, R17, R18, R19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

Commit message: 08/09/26
Parts:
- removed J2: Conn_01x40, Molex_541324062:CON_541324062_MOL, symbol Connector_Generic:Conn_01x40
- removed Q5: Q_NMOS_GSD, symbol Transistor_FET:Q_NMOS_GSD
- removed R17, R18: 15R, Resistor_SMD:R_01005_0402Metric, symbol Device:R
- removed R19: 100R, Resistor_SMD:R_01005_0402Metric, symbol Device:R
- removed R20: 100k, Resistor_SMD:R_01005_0402Metric, symbol Device:R
- added TP10, TP9: TestPoint, symbol Connector:TestPoint
- R15: value 15R -> 22 R; footprint Resistor_SMD:R_01005_0402Metric -> (none)
- R16: value 15R -> 22R; footprint Resistor_SMD:R_01005_0402Metric -> (none)
Connections:
- net MCU_3V3 is gone; now on net +3.3V: R1.1, R10.2, R24.1, R26.2
- net ENCODER_SW: now also U2.19 (GPIO21); no longer U2.8 (GPIO0/ADC1_CH0/XTAL_32K_P)
- net TFT_RST: now also U2.23 (GPIO15); no longer U2.19 (GPIO21)
- net at R16.2: now also U2.8 (GPIO0/ADC1_CH0/XTAL_32K_P)
- net at R15.2: now also TP9.1
- net at U2.10 (GPIO8): now also R15.1
- net BL_SINK: no longer names the net of R16.1
- net BL_SINK: now also TP10.1; no longer R15.1
- net RTC_I2C_SCL: no longer names the net of R25.2, U4.3 (SCL)
- no-connect marks 24 -> 1
Other:
- note removed: "LCD konnektörü başka bir sayfaya taşınmalı"
- moved on the sheet: BT1, C10, C5, C6, C7, C9, R1, R10, R2, R22, R23, R24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
