File: mcu.kicad_sch (KiCad schematic)
At the start: 28 parts, among them J2 DS1021-1X3SF11-B, SW1 BOOT, SW2 RESET, U2 ESP32-C6-WROOM-1, U4 RV-3028-C7

Commit message: 11 Eylül
Parts:
- BT1: value Battery_Cell -> CR2032 holder; footprint (none) -> Power_Output_Custom:KLS_CR2032_05; Battery (none) -> CR2032 3V PRIMARY; cell purchased separately; RTC trickle c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; MPN (none) -> L-KLS5-CR2032-05-R1; Manufacturer (none) -> KLS Electronic; Supplier (none) -> Ozdisan 497433
- C10, C9: footprint (none) -> Capacitor_SMD:C_0402_1005Metric
- C6, C7: footprint Capacitor_SMD:C_01005_0402Metric -> Capacitor_SMD:C_0402_1005Metric
- R1, R22, R25, R26: footprint Resistor_SMD:R_01005_0402Metric -> Resistor_SMD:R_0402_1005Metric
- R10, R15, R16, R2, R23, R24, R3: footprint (none) -> Resistor_SMD:R_0402_1005Metric
- R37: footprint Resistor_SMD:R_0603_1608Metric -> Resistor_SMD:R_0402_1005Metric
- SW1: value BOOT -> BOOT / PTS810; footprint (none) -> Button_Switch_SMD:SW_SPST_PTS810
- SW2: value RESET -> RESET / PTS810; footprint (none) -> Button_Switch_SMD:SW_SPST_PTS810
- TP10, TP6, TP7, TP8, TP9: footprint (none) -> TestPoint:TestPoint_Pad_D1.0mm
Other:
- note added: "BT1: L-KLS5-CR2032-05-R1 holder. CR2032 primary cell: disable RTC trickle charge. Pad 1 positive, pad 2 GND."
- moved on the sheet: BT1, C10, C7, C9, R1, R10, R15, R16, R2, R22, R23, R24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
