File: powergeneration.kicad_sch (KiCad schematic)
At the start: 1 part, among them U6 TPS54561

Commit message: KiCad schematic updates - 2026-09-07
Parts:
- added C12: 100 nF, symbol Device:C
- added D2: D, symbol Device:D
Connections:
- net at U6.1 (BOOT): now also C12.1
- net GND: now reaches U6.11 (GND), U6.8 (GND)
- net GND: now also D2.2 (A)
- net PD_VOUT: now reaches U6.2 (VIN)
- net at U6.9 (SW): now also C12.2, D2.1 (K)
Other:
- note added: "SERAMİK OLMALI X5R/X7R"

Commit message: 08/09/26
Parts:
- removed C12: 100 nF, symbol Device:C
- removed D2: D, symbol Device:D
- removed U6: TPS54561, Package_SON:WSON-10-1EP_4x4mm_P0.8mm_EP2.6x3mm_ThermalVias, symbol Regulator_Switching:TPS54561
Other:
- note removed: "SERAMİK OLMALI X5R/X7R"
