File: powergeneration.kicad_sch (KiCad schematic)
At the start: 18 parts, among them U5 AOZ1284PI, U6 TL431BIDBZR

Commit message: 11 Eylül
Parts:
- C14, C17, C18, C19: footprint Capacitor_SMD:C_0603_1608Metric -> Capacitor_SMD:C_0402_1005Metric
- D2: value 60V / 2A -> SS2060FL_R1_00001; footprint (none) -> Diode_SMD:D_SOD-123F; DesignNote Cathode LX; anode GND. VF/thermal/surge MPN qualification U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 -> PANJIT 60V 2A Schottky, SOD-123FL; cathode LX, anode GND; O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
- L1: value 22uH -> SRI0704-220M; footprint (none) -> Inductor_SMD:L_7.3x7.3_H4.5; DesignNote Isat >=2A and Irms >=1.5A at max temperature; fault current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 -> CORE MASTER 22uH, 1.95A rated, 0.11ohm max; 18.2uH at 1.95A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
- R38, R39, R40, R41, R42: footprint Resistor_SMD:R_0603_1608Metric -> Resistor_SMD:R_0402_1005Metric
Changed lines of the file:
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@@
 	(wire
 		(pts
+			(xy 195.58 76.2) (xy 195.58 69.85)
+		)
+		(stroke
+			(width 0)
+			(type default)
+		)
+	)
+	(wire
+		(pts
 			(xy 137.16 81.28) (xy 142.24 81.28)
 		)
@@
 	(wire
 		(pts
-			(xy 34.925 154.94) (xy 46.99 154.94)
+			(xy 35.56 154.94) (xy 46.99 154.94)
 		)
 		(stroke
@@
 	)
 	(label "COMP_NODE"
-		(at 34.925 154.94 0)
+		(at 35.56 154.94 0)
 		(effects
 			(font
@@
 	)
 	(label "LX_SW"
-		(at 137.795 76.2 0)
+		(at 138.43 76.2 0)
 		(effects
 			(font
@@
 	)
 	(global_label "PD_VOUT"
-		(shape input)
+		(shape passive)
 		(at 243.84 110.49 0)
 		(fields_autoplaced yes)
@@
 		)
 		(property "Intersheetrefs" "${INTERSHEET_REFS}"
-			(at 255.05 110.49 0)
+			(at 255.27 110.49 0)
 			(hide yes)
 			(show_name no)
@@
 	)
 	(global_label "PD_VOUT"
-		(shape output)
+		(shape passive)
 		(at 40.64 50.8 180)
 		(fields_autoplaced yes)
@@
 		)
 		(property "Intersheetrefs" "${INTERSHEET_REFS}"
-			(at 29.43 50.8 0)
+			(at 29.21 50.8 0)
 			(hide yes)
 			(show_name no)
@@
 			)
 		)
-		(property "Footprint" "Resistor_SMD:R_0603_1608Metric"
+		(property "Footprint" "Resistor_SMD:R_0402_1005Metric"
 			(at 203.2 120.65 0)
 			(hide yes)
@@
 			)
 		)
-		(property "Footprint" "Capacitor_SMD:C_0603_1608Metric"
+		(property "Footprint" "Capacitor_SMD:C_0402_1005Metric"
 			(at 96.52 60.96 0)
 			(hide yes)
@@
 			)
 		)
-		(property "Footprint" "Resistor_SMD:R_0603_1608Metric"
+		(property "Footprint" "Resistor_SMD:R_0402_1005Metric"
 			(at 50.8 154.94 0)
 			(hide yes)
@@
 			)
 		)
-		(property "Footprint" "Resistor_SMD:R_0603_1608Metric"
+		(property "Footprint" "Resistor_SMD:R_0402_1005Metric"
 			(at 203.2 138.43 0)
 			(hide yes)
@@
 			)
 		)
-		(property "Footprint" "Resistor_SMD:R_0603_1608Metric"
+		(property "Footprint" "Resistor_SMD:R_0402_1005Metric"
 			(at 50.8 120.65 0)
 			(hide yes)
@@
 	)
 	(symbol
+		(lib_id "power:PWR_FLAG")
+		(at 195.58 69.85 0)
+		(unit 1)
+		(body_style 1)
+		(exclude_from_sim no)
+		(in_bom yes)
+		(on_board yes)
+		(in_pos_files yes)
+		(dnp no)
+		(property "Reference" "#FLG04"
+			(at 195.58 66.04 0)
+			(hide yes)
+			(show_name no)
+			(do_not_autoplace no)
+			(effects
+				(font
+					(size 1.27 1.27)
+				)
+				(justify left)
+			)
+		)
+		(property "Value" "PWR_FLAG"
+			(at 195.58 66.04 0)
+			(show_name no)
+			(do_not_autoplace no)
+			(effects
+				(font
+					(size 1.27 1.27)
+				)
+			)
+		)
+		(property "Footprint" ""
+			(at 195.58 66.04 0)
+			(hide yes)
+			(show_name no)
+			(do_not_autoplace no)
+			(effects
+				(font
+					(size 1.27 1.27)
+				)
+				(justify left)
+			)
+		)
+		(property "Datasheet" ""
+			(at 195.58 66.04 0)
+			(show_name no)
+			(do_not_autoplace no)
+			(effects
+				(font
+					(size 1.27 1.27)
+				)
+			)
+		)
+		(property "Description" ""
+			(at 195.58 66.04 0)
+			(show_name no)
+			(do_not_autoplace no)
+			(effects
+				(font
+					(size 1.27 1.27)
+				)
+			)
+		)
+		(property "DesignNote" ""
+			(at 195.58 66.04 0)
+			(hide yes)
+			(show_name no)
+			(do_not_autoplace no)
+			(effects
+				(font
+					(size 1.27 1.27)
+				)
+				(justify left)
+			)
+		)
+		(pin "1"
+		)
+		(instances
+			(project "masaüstü güç kaynağı"
+				(path "/a43081a6-9aa2-4898-9347-bbcb5849dafd/5dec5942-8798-43d7-9ae8-350e99f1540a"
+					(reference "#FLG04")
+					(unit 1)
+				)
+			)
+		)
+	)
+	(symbol
 		(lib_id "power:GND")
 		(at 50.8 132.08 0)
@@
 			)
 		)
-		(property "Footprint" "Resistor_SMD:R_0603_1608Metric"
+		(property "Footprint" "Resistor_SMD:R_0402_1005Metric"
 			(at 111.76 120.65 0)
 			(hide yes)
@@
 			)
 		)
-		(property "Footprint" "Capacitor_SMD:C_0603_1608Metric"
+		(property "Footprint" "Capacitor_SMD:C_0402_1005Metric"
 			(at 81.28 120.65 0)
 			(hide yes)
@@
 		(dnp no)
 		(property "Reference" "C15"
-			(at 199.39 87.63 0)
+			(at 187.198 88.392 0)
 			(show_name no)
 			(do_not_autoplace no)
@@
 		)
 		(property "Value" "47uF"
-			(at 199.39 90.17 0)
+			(at 186.944 91.44 0)
 			(show_name no)
 			(do_not_autoplace no)
@@
 			)
 		)
-		(property "Footprint" "Capacitor_SMD:C_0603_1608Metric"
+		(property "Footprint" "Capacitor_SMD:C_0402_1005Metric"
 			(at 147.32 71.12 0)
 			(hide yes)
@@
 			)
 		)
-		(property "Footprint" "Capacitor_SMD:C_0603_1608Metric"
+		(property "Footprint" "Capacitor_SMD:C_0402_1005Metric"
 			(at 77.47 154.94 0)
 			(hide yes)
@@
 			)
 		)
-		(property "Value" "60V / 2A"
-			(at 162.56 90.17 90)
+		(property "Value" "SS2060FL_R1_00001"
+			(at 161.798 91.186 90)
 			(show_name no)
 			(do_not_autoplace no)
@@
 			)
 		)
-		(property "Footprint" ""
+		(property "Footprint" "Diode_SMD:D_SOD-123F"
 			(at 158.75 88.9 0)
 			(hide yes)
@@
 			)
 		)
-		(property "Datasheet" ""
+		(property "Datasheet" "https://www.ozdisan.com/p/schottky-diyotlar-385/panjit-ss2060fl-r1-00001-574723"
 			(at 158.75 88.9 0)
+			(hide yes)
 			(show_name no)
 			(do_not_autoplace no)
@@
 			)
 		)
-		(property "DesignNote" "Cathode LX; anode GND. VF/thermal/surge MPN qualification UNRESOLVED"
+		(property "DesignNote" "PANJIT 60V 2A Schottky, SOD-123FL; cathode LX, anode GND; Ozdisan stocked selection"
 			(at 158.75 88.9 0)
 			(hide yes)
@@
 			)
 		)
-		(property "Value" "22uH"
-			(at 173.355 73.66 90)
+		(property "Value" "SRI0704-220M"
+			(at 188.722 78.232 90)
 			(show_name no)
 			(do_not_autoplace no)
@@
 			)
 		)
-		(property "Footprint" ""
+		(property "Footprint" "Inductor_SMD:L_7.3x7.3_H4.5"
 			(at 171.45 76.2 0)
 			(hide yes)
@@
 			)
 		)
-		(property "Datasheet" ""
-			(at 171.45 76.2 0)
+		(property "Datasheet" "https://store.comet.bg/download-file.php?id=16477"
+			(at 174.752 107.95 0)
+			(hide yes)
 			(show_name no)
 			(do_not_autoplace no)
@@
 			)
 		)
-		(property "DesignNote" "Isat >=2A and Irms >=1.5A at max temperature; fault current capability UNRESOLVED"
+		(property "DesignNote" "CORE MASTER 22uH, 1.95A rated, 0.11ohm max; 18.2uH at 1.95A and 16.4uH at 2.14A; Ozdisan stocked"
 			(at 171.45 76.2 0)
 			(hide yes)
