File: powersensing.kicad_sch (KiCad schematic)
At the start: 4 parts, among them U3 INA228

Commit message: KiCad schematic updates - 2026-09-07
Parts:
- C11: footprint (none) -> Capacitor_SMD:C_01005_0402Metric
- R27, RShunt: footprint (none) -> Resistor_SMD:R_01005_0402Metric
Connections:
- net GND: now also U3.1 (A1), U3.2 (A0)
- net MCU_3V3: now also C11.1, U3.6 (VS)
- net OUT_POS: now also U3.9 (Vin-)
- net PD_VOUT: now also U3.10 (Vin+)
Other:
- moved on the sheet: C11, RShunt

Commit message: 08/09/26
Connections:
- net INA_ALERT: now also R27.2
- net MCU_3V3 renamed +3.3V
Other:
- moved on the sheet: C11, R27, RShunt, U3
