File: powersensing.kicad_sch (KiCad schematic)
At the start: 4 parts, among them U3 INA228

Commit message: 11 Eylül
Parts:
- C11: footprint Capacitor_SMD:C_01005_0402Metric -> Capacitor_SMD:C_0402_1005Metric
- R27: footprint Resistor_SMD:R_01005_0402Metric -> Resistor_SMD:R_0402_1005Metric
Other:
- moved on the sheet: C11, RShunt
Changed lines of the file:
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@@
 	(paper "A4")
 	(junction
-		(at 140.97 73.025)
+		(at 140.97 73.66)
 		(diameter 0)
 		(color 0 0 0 0)
@@
 	)
 	(junction
-		(at 75.565 118.11)
+		(at 76.2 118.11)
 		(diameter 0)
 		(color 0 0 0 0)
@@
 	(wire
 		(pts
-			(xy 96.52 118.11) (xy 102.235 118.11)
-		)
-		(stroke
-			(width 0)
-			(type default)
-		)
-	)
-	(wire
-		(pts
-			(xy 75.565 104.14) (xy 75.565 118.11)
+			(xy 96.52 118.11) (xy 102.87 118.11)
+		)
+		(stroke
+			(width 0)
+			(type default)
+		)
+	)
+	(wire
+		(pts
+			(xy 76.2 104.14) (xy 76.2 118.11)
 		)
 		(stroke
@@
 	(wire
 		(pts
-			(xy 70.485 118.11) (xy 75.565 118.11)
+			(xy 71.12 118.11) (xy 76.2 118.11)
 		)
 		(stroke
@@
 	(wire
 		(pts
-			(xy 140.97 73.025) (xy 140.97 88.9)
+			(xy 140.97 73.66) (xy 140.97 88.9)
 		)
 		(stroke
@@
 	(wire
 		(pts
-			(xy 150.495 73.025) (xy 140.97 73.025)
-		)
-		(stroke
-			(width 0)
-			(type default)
-		)
-	)
-	(wire
-		(pts
-			(xy 130.81 73.025) (xy 140.97 73.025)
+			(xy 151.13 73.66) (xy 140.97 73.66)
+		)
+		(stroke
+			(width 0)
+			(type default)
+		)
+	)
+	(wire
+		(pts
+			(xy 130.81 73.66) (xy 140.97 73.66)
 		)
 		(stroke
@@
 	(wire
 		(pts
-			(xy 150.495 74.295) (xy 150.495 73.025)
+			(xy 151.13 74.93) (xy 151.13 73.66)
 		)
 		(stroke
@@
 	(wire
 		(pts
-			(xy 75.565 118.11) (xy 81.915 118.11)
-		)
-		(stroke
-			(width 0)
-			(type default)
-		)
-	)
-	(wire
-		(pts
-			(xy 130.81 104.14) (xy 75.565 104.14)
-		)
-		(stroke
-			(width 0)
-			(type default)
-		)
-	)
-	(wire
-		(pts
-			(xy 150.495 81.915) (xy 150.495 83.82)
-		)
-		(stroke
-			(width 0)
-			(type default)
-		)
-	)
-	(wire
-		(pts
-			(xy 89.535 118.11) (xy 96.52 118.11)
+			(xy 76.2 118.11) (xy 82.55 118.11)
+		)
+		(stroke
+			(width 0)
+			(type default)
+		)
+	)
+	(wire
+		(pts
+			(xy 130.81 104.14) (xy 76.2 104.14)
+		)
+		(stroke
+			(width 0)
+			(type default)
+		)
+	)
+	(wire
+		(pts
+			(xy 151.13 82.55) (xy 151.13 83.82)
+		)
+		(stroke
+			(width 0)
+			(type default)
+		)
+	)
+	(wire
+		(pts
+			(xy 90.17 118.11) (xy 96.52 118.11)
 		)
 		(stroke
@@
 	)
 	(global_label "OUT_POS"
-		(shape input)
+		(shape passive)
 		(at 128.27 93.98 180)
 		(fields_autoplaced yes)
@@
 		)
 		(property "Intersheetrefs" "${INTERSHEET_REFS}"
-			(at 116.8786 93.98 0)
+			(at 116.84 93.98 0)
 			(hide yes)
 			(show_name no)
@@
 	)
 	(global_label "PD_I2C_SDA_3V3"
-		(shape input)
+		(shape bidirectional)
 		(at 165.1 101.6 0)
 		(fields_autoplaced yes)
@@
 		)
 		(property "Intersheetrefs" "${INTERSHEET_REFS}"
-			(at 183.688 101.6 0)
+			(at 184.15 101.6 0)
 			(hide yes)
 			(show_name no)
@@
 	)
 	(global_label "OUT_POS"
-		(shape input)
-		(at 102.235 118.11 0)
+		(shape passive)
+		(at 102.87 118.11 0)
 		(fields_autoplaced yes)
 		(effects
@@
 		)
 		(property "Intersheetrefs" "${INTERSHEET_REFS}"
-			(at 113.6264 118.11 0)
+			(at 113.03 118.11 0)
 			(hide yes)
 			(show_name no)
@@
 	)
 	(global_label "PD_VOUT"
-		(shape input)
-		(at 70.485 118.11 180)
+		(shape passive)
+		(at 71.12 118.11 180)
 		(fields_autoplaced yes)
 		(effects
@@
 		)
 		(property "Intersheetrefs" "${INTERSHEET_REFS}"
-			(at 59.275 118.11 0)
+			(at 59.69 118.11 0)
 			(hide yes)
 			(show_name no)
@@
 	)
 	(global_label "PD_I2C_SCL_3V3"
-		(shape input)
+		(shape bidirectional)
 		(at 165.1 104.14 0)
 		(fields_autoplaced yes)
@@
 		)
 		(property "Intersheetrefs" "${INTERSHEET_REFS}"
-			(at 183.6275 104.14 0)
+			(at 184.15 104.14 0)
 			(hide yes)
 			(show_name no)
@@
 		)
 		(property "Intersheetrefs" "${INTERSHEET_REFS}"
-			(at 215.68 109.22 0)
+			(at 215.9 109.22 0)
 			(hide yes)
 			(show_name no)
@@
 			)
 		)
-		(property "Footprint" "Resistor_SMD:R_01005_0402Metric"
+		(property "Footprint" "Resistor_SMD:R_0402_1005Metric"
 			(at 193.802 96.52 90)
 			(hide yes)
@@
 	(symbol
 		(lib_id "Device:C")
-		(at 150.495 78.105 0)
+		(at 151.13 78.74 0)
 		(unit 1)
 		(body_style 1)
@@
 		(dnp no)
 		(property "Reference" "C11"
-			(at 153.67 75.565 0)
+			(at 154.305 76.2 0)
 			(show_name no)
 			(do_not_autoplace no)
@@
 		)
 		(property "Value" "100nF"
-			(at 154.305 80.645 0)
-			(show_name no)
-			(do_not_autoplace no)
-			(effects
-				(font
-					(size 1.27 1.27)
-				)
-			)
-		)
-		(property "Footprint" "Capacitor_SMD:C_01005_0402Metric"
-			(at 151.4602 81.915 0)
+			(at 154.94 81.28 0)
+			(show_name no)
+			(do_not_autoplace no)
+			(effects
+				(font
+					(size 1.27 1.27)
+				)
+			)
+		)
+		(property "Footprint" "Capacitor_SMD:C_0402_1005Metric"
+			(at 152.0952 82.55 0)
 			(hide yes)
 			(show_name no)
@@
 		)
 		(property "Datasheet" ""
-			(at 150.495 78.105 0)
+			(at 151.13 78.74 0)
 			(hide yes)
 			(show_name no)
@@
 		)
 		(property "Description" "Unpolarized capacitor"
-			(at 150.495 78.105 0)
+			(at 151.13 78.74 0)
 			(hide yes)
 			(show_name no)
@@
 	(symbol
 		(lib_id "Device:R")
-		(at 85.725 118.11 90)
+		(at 86.36 118.11 90)
 		(unit 1)
 		(body_style 1)
@@
 		(fields_autoplaced yes)
 		(property "Reference" "RShunt"
-			(at 85.725 111.76 90)
+			(at 86.36 111.76 90)
 			(show_name no)
 			(do_not_autoplace no)
@@
 		)
 		(property "Value" "5mR / 1W"
-			(at 85.725 114.3 90)
+			(at 86.36 114.3 90)
 			(show_name no)
 			(do_not_autoplace no)
@@
 		)
 		(property "Footprint" "Resistor_SMD:R_2512_6332Metric"
-			(at 85.725 119.888 90)
+			(at 86.36 119.888 90)
 			(hide yes)
 			(show_name no)
@@
 		)
 		(property "Datasheet" ""
-			(at 85.725 118.11 0)
+			(at 86.36 118.11 0)
 			(hide yes)
 			(show_name no)
@@
 		)
 		(property "Description" "Resistor"
-			(at 85.725 118.11 0)
+			(at 86.36 118.11 0)
 			(hide yes)
 			(show_name no)
@@
 	(symbol
 		(lib_id "power:+3.3V")
-		(at 130.81 73.025 0)
+		(at 130.81 73.66 0)
 		(unit 1)
 		(body_style 1)
@@
 		(fields_autoplaced yes)
 		(property "Reference" "#PWR048"
-			(at 130.81 76.835 0)
+			(at 130.81 77.47 0)
 			(hide yes)
 			(show_name no)
@@
 		)
 		(property "Value" "+3.3V"
-			(at 130.81 67.945 0)
+			(at 130.81 68.58 0)
 			(show_name no)
 			(do_not_autoplace no)
@@
 		)
 		(property "Footprint" ""
-			(at 130.81 73.025 0)
+			(at 130.81 73.66 0)
 			(hide yes)
 			(show_name no)
@@
 		)
 		(property "Datasheet" ""
-			(at 130.81 73.025 0)
+			(at 130.81 73.66 0)
 			(hide yes)
 			(show_name no)
@@
 		)
 		(property "Description" "Power symbol creates a global label with name \"+3.3V\""
-			(at 130.81 73.025 0)
+			(at 130.81 73.66 0)
 			(hide yes)
 			(show_name no)
@@
 	(symbol
 		(lib_id "power:GND")
-		(at 150.495 83.82 0)
+		(at 151.13 83.82 0)
 		(unit 1)
 		(body_style 1)
@@
 		(fields_autoplaced yes)
 		(property "Reference" "#PWR029"
-			(at 150.495 90.17 0)
+			(at 151.13 90.17 0)
 			(hide yes)
 			(show_name no)
@@
 		)
 		(property "Value" "GND"
-			(at 152.4 85.0899 0)
+			(at 153.035 85.0899 0)
 			(show_name no)
 			(do_not_autoplace no)
@@
 		)
 		(property "Footprint" ""
-			(at 150.495 83.82 0)
+			(at 151.13 83.82 0)
 			(hide yes)
 			(show_name no)
@@
 		)
 		(property "Datasheet" ""
-			(at 150.495 83.82 0)
+			(at 151.13 83.82 0)
 			(hide yes)
 			(show_name no)
@@
 		)
 		(property "Description" "Power symbol creates a global label with name \"GND\" , ground"
-			(at 150.495 83.82 0)
-			(hide yes)
-			(show_name no)
+			(at 151.13 83.82 0)
+			(hide yes)
+			(show_name no)
