File: usb_c_input.kicad_sch (KiCad schematic)
At the start: 1 part, among them J1 DX07B024JJ1R1500

Commit message: 11 Eylül
Parts:
- added D3, D4, D5: AQ3130E-01ETG (bidirectional), Diode_SMD:D_SOD-882, symbol Device:D_TVS
- added U9: TPD4E05U06QDQARQ1, USB_ESD:antmicro_tpd4e05u06qdqarq1, symbol USB_ESD:TPD4E05U06QDQARQ1
- J1: footprint (none) -> USB_Connector_Custom:JAE_DX07B024JJ1R1500
Connections:
- net GND: now also D3.1 (A1), D4.2 (A2), D5.2 (A2), U9.3 (GND), U9.8 (GND)
- net USB_CC1: now also D4.1 (A1)
- net USB_CC2: now also D5.1 (A1)
- net USB_DM: now also U9.2 (D1-)
- net USB_DP: now also U9.1 (D1+)
- net USB_VBUS: now also D3.2 (A2)
- no-connect marks 10 -> 16
Other:
- note added: "USB PORT ESD U9: D+/D-; IEC 12kV contact, 15kV air. D4/D5: CC1/CC2, 28V VRWM; IEC 30kV contact/air. D3: 28V VBUS TVS; IEC 30kV contact/air. Place directly behind J1; shortest GND return."
- note added: "VBUS LIMIT: AQ3130E clamps 39..44V @1A. AP33772 VCC abs max 34V and VOUT 31V. ESD robustness improves, but surge immunity needs system test / surge stopper."
- moved on the sheet: J1
