File: userinterface.kicad_sch (KiCad schematic)
At the start: 0 parts

Commit message: 08/09/26
Parts:
- added J3: Conn_01x40, Molex_541324062:CON_541324062_MOL, symbol Connector_Generic:Conn_01x40
- added Q6: Q_NMOS_GSD, symbol Transistor_FET:Q_NMOS_GSD
- added R28: 100R, Resistor_SMD:R_01005_0402Metric, symbol Device:R
- added R29: 100k, Resistor_SMD:R_01005_0402Metric, symbol Device:R
- added R30, R31, R32, R33: 15R, Resistor_SMD:R_01005_0402Metric, symbol Device:R
Connections:
- new net: Q6.1 (G), R28.2, R29.1
- new net: J3.34 (Pin_34), R33.2
- new net: J3.35 (Pin_35), R32.2
- new net: J3.36 (Pin_36), R31.2
- new net: J3.37 (Pin_37), R30.2
- new net +3.3V: J3.32 (Pin_32), J3.33 (Pin_33), J3.7 (Pin_7), J3.8 (Pin_8)
- new net BACKLIGHT_3V0: J3.38 (Pin_38)
- new net BL_SINK: R30.1, R31.1, R32.1, R33.1
- new net GND: J3.1 (Pin_1), J3.31 (Pin_31), J3.39 (Pin_39), Q6.2 (S), R29.2
- new net TFT_BL_PWM: R28.1
- new net TFT_CS: J3.10 (Pin_10)
- new net TFT_DC: J3.12 (Pin_12)
- new net TFT_MOSI: J3.9 (Pin_9)
- new net TFT_RST: J3.30 (Pin_30)
- new net TFT_SCLK: J3.11 (Pin_11)
- no-connect marks 0 -> 23
Other:
- added sheet USER (USER_İNTERFACE.kicad_sch)
