File: userinterface.kicad_sch (KiCad schematic)
At the start: 12 parts, among them J3 Conn_01x40, Q5 AO3400A, SW3 L-KLS4-EC12-012424-W

Commit message: 11 Eylül
Parts:
- removed Q5: AO3400A, AO3400A:SOT95P280X125-3N, symbol AO3400A:AO3400A
- removed R30, R31, R32, R33: 15R, Resistor_SMD:R_01005_0402Metric, symbol Device:R
- added C20, C21: 22uF, Capacitor_SMD:C_1206_3216Metric, symbol Device:C
- added C22: 100nF / 16V, Capacitor_SMD:C_0402_1005Metric, symbol Device:C
- added L2: 2.2uH, Inductor_SMD:L_Wuerth_MAPI-4030, symbol Device:L
- added R44: 604kR 0.1%, Resistor_SMD:R_0402_1005Metric, symbol Device:R
- added R45: 100kR 0.1%, Resistor_SMD:R_0402_1005Metric, symbol Device:R
- added R46: 3.24kR 0.1%, Resistor_SMD:R_0402_1005Metric, symbol Device:R
- added U7: TPS61023DRLR, Package_TO_SOT_SMD:SOT-563, symbol Power_Supply_Custom:TPS61023DRLR
- added U8: CAT4104V-GT3, Package_SO:SOIC-8_3.9x4.9mm_P1.27mm, symbol Power_Supply_Custom:CAT4104V-GT3
- J3: value Conn_01x40 -> NHD-2.4-240320AF-CSXP; DisplayMPN (none) -> NHD-2.4-240320AF-CSXP; MPN (none) -> 54132-4062; Manufacturer (none) -> Molex
- R28: footprint Resistor_SMD:R_01005_0402Metric -> Resistor_SMD:R_0402_1005Metric
- R29: value 100k -> 100kR; footprint Resistor_SMD:R_01005_0402Metric -> Resistor_SMD:R_0402_1005Metric
- R34, R35, R36: footprint Resistor_SMD:R_0603_1608Metric -> Resistor_SMD:R_0402_1005Metric
Connections:
- net +3.3V: now also C20.1, L2.1, U7.2 (EN), U7.3 (VIN)
- net GND: now also J3.13 (Pin_13), J3.14 (Pin_14), J3.15 (Pin_15), J3.16 (Pin_16), J3.17 (Pin_17), J3.18 (Pin_18), J3.19 (Pin_19), J3.20 (Pin_20), J3.21 (Pin_21), J3.22 (Pin_22), J3.23 (Pin_23), J3.24 (Pin_24), J3.25 (Pin_25), J3.26 (Pin_26), J3.27 (Pin_27), J3.28 (Pin_28), J3.29 (Pin_29), C20.2, C21.2, C22.2, R45.2, R46.2, U7.4 (GND), U8.5 (GND)
- net at R28.2, R29.1: now also U8.6 (EN_PWM)
- net BL_K1: now reaches J3.34 (Pin_34)
- net BL_K1: now also U8.1 (LED1)
- net BL_K2: now reaches J3.35 (Pin_35)
- net BL_K2: now also U8.2 (LED2)
- net BL_K3: now reaches J3.36 (Pin_36)
- net BL_K3: now also U8.3 (LED3)
- net BL_K4: now reaches J3.37 (Pin_37)
- net BL_K4: now also U8.4 (LED4)
- net BACKLIGHT_3V0 renamed BACKLIGHT_4V2
- net BACKLIGHT_4V2: now also C21.1, C22.1, R44.1, U7.6 (VOUT), U8.7 (VIN)
- new net: R46.1, U8.8 (RSET)
- new net BL_BOOST_FB: R44.2, R45.1, U7.1 (FB)
- new net BL_BOOST_SW: L2.2, U7.5 (SW)
- no-connect marks 23 -> 6
Other:
- note added: "4-wire SPI: IM2/IM1/IM0 = 1/1/0. RDX and DB0..DB15 tied GND per TFT wiring diagram."
- note added: "BACKLIGHT: 4 x ~40mA constant-current sinks. R46 from CAT4104 nonlinear RSET equation. PWM: 1kHz recommended; duty 0 or >=1%."
- note added: "BOOST: +3.3V -> ~4.2V; 0.20A output design. C20 effective >=10uF; C21 effective 4..30uF. R/C 0402 except boost bulk C20/C21 (1206)."
- moved on the sheet: J3, SW3

Commit message: 12/09/26
Other:
- moved on the sheet: R34, R35, R36
Changed lines of the file:
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@@
 	(wire
 		(pts
-			(xy 256.54 133.35) (xy 256.54 128.27)
+			(xy 262.89 128.27) (xy 262.89 123.19)
 		)
 		(stroke
@@
 	(wire
 		(pts
-			(xy 256.54 140.97) (xy 256.54 146.05)
+			(xy 262.89 135.89) (xy 262.89 140.97)
 		)
 		(stroke
@@
 	(wire
 		(pts
-			(xy 223.52 140.97) (xy 223.52 146.05)
+			(xy 229.87 135.89) (xy 229.87 140.97)
 		)
 		(stroke
@@
 	(wire
 		(pts
-			(xy 190.5 140.97) (xy 190.5 146.05)
+			(xy 196.85 135.89) (xy 196.85 140.97)
 		)
 		(stroke
@@
 	(wire
 		(pts
-			(xy 223.52 133.35) (xy 223.52 128.27)
+			(xy 229.87 128.27) (xy 229.87 123.19)
 		)
 		(stroke
@@
 	(wire
 		(pts
-			(xy 190.5 133.35) (xy 190.5 128.27)
+			(xy 196.85 128.27) (xy 196.85 123.19)
 		)
 		(stroke
@@
 	(global_label "ENCODER_SW"
 		(shape output)
-		(at 256.54 146.05 0)
+		(at 262.89 140.97 0)
 		(effects
 			(font
@@
 		)
 		(property "Intersheetrefs" "${INTERSHEET_REFS}"
-			(at 256.54 146.05 0)
+			(at 262.89 140.97 0)
 			(hide yes)
 			(show_name no)
@@
 	(global_label "ENCODER_A"
 		(shape output)
-		(at 190.5 146.05 0)
+		(at 196.85 140.97 0)
 		(effects
 			(font
@@
 		)
 		(property "Intersheetrefs" "${INTERSHEET_REFS}"
-			(at 190.5 146.05 0)
+			(at 196.85 140.97 0)
 			(hide yes)
 			(show_name no)
@@
 	(global_label "ENCODER_B"
 		(shape output)
-		(at 223.52 146.05 0)
+		(at 229.87 140.97 0)
 		(effects
 			(font
@@
 		)
 		(property "Intersheetrefs" "${INTERSHEET_REFS}"
-			(at 223.52 146.05 0)
+			(at 229.87 140.97 0)
 			(hide yes)
 			(show_name no)
@@
 	(symbol
 		(lib_id "Device:R")
-		(at 256.54 137.16 0)
+		(at 262.89 132.08 0)
 		(unit 1)
 		(body_style 1)
@@
 		(dnp no)
 		(property "Reference" "R36"
-			(at 251.46 137.16 0)
+			(at 257.81 132.08 0)
 			(show_name no)
 			(do_not_autoplace no)
@@
 		)
 		(property "Value" "10k"
-			(at 250.19 139.7 0)
+			(at 256.54 134.62 0)
 			(show_name no)
 			(do_not_autoplace no)
@@
 		)
 		(property "Footprint" "Resistor_SMD:R_0402_1005Metric"
-			(at 254.762 137.16 0)
+			(at 261.112 132.08 0)
 			(hide yes)
 			(show_name no)
@@
 		)
 		(property "Datasheet" ""
-			(at 256.54 137.16 0)
+			(at 262.89 132.08 0)
 			(hide yes)
 			(show_name no)
@@
 		)
 		(property "Description" "Resistor"
-			(at 256.54 137.16 0)
+			(at 262.89 132.08 0)
 			(hide yes)
 			(show_name no)
@@
 	(symbol
 		(lib_id "power:+3.3V")
-		(at 223.52 128.27 0)
+		(at 229.87 123.19 0)
 		(unit 1)
 		(body_style 1)
@@
 		(fields_autoplaced yes)
 		(property "Reference" "#PWR055"
-			(at 223.52 132.08 0)
+			(at 229.87 127 0)
 			(hide yes)
 			(show_name no)
@@
 		)
 		(property "Value" "+3.3V"
-			(at 223.52 123.19 0)
+			(at 229.87 118.11 0)
 			(show_name no)
 			(do_not_autoplace no)
@@
 		)
 		(property "Footprint" ""
-			(at 223.52 128.27 0)
+			(at 229.87 123.19 0)
 			(hide yes)
 			(show_name no)
@@
 		)
 		(property "Datasheet" ""
-			(at 223.52 128.27 0)
+			(at 229.87 123.19 0)
 			(hide yes)
 			(show_name no)
@@
 		)
 		(property "Description" "Power symbol creates a global label with name \"+3.3V\""
-			(at 223.52 128.27 0)
+			(at 229.87 123.19 0)
 			(hide yes)
 			(show_name no)
@@
 	(symbol
 		(lib_id "power:+3.3V")
-		(at 256.54 128.27 0)
+		(at 262.89 123.19 0)
 		(unit 1)
 		(body_style 1)
@@
 		(fields_autoplaced yes)
 		(property "Reference" "#PWR056"
-			(at 256.54 132.08 0)
+			(at 262.89 127 0)
 			(hide yes)
 			(show_name no)
@@
 		)
 		(property "Value" "+3.3V"
-			(at 256.54 123.19 0)
+			(at 262.89 118.11 0)
 			(show_name no)
 			(do_not_autoplace no)
@@
 		)
 		(property "Footprint" ""
-			(at 256.54 128.27 0)
+			(at 262.89 123.19 0)
 			(hide yes)
 			(show_name no)
@@
 		)
 		(property "Datasheet" ""
-			(at 256.54 128.27 0)
+			(at 262.89 123.19 0)
 			(hide yes)
 			(show_name no)
@@
 		)
 		(property "Description" "Power symbol creates a global label with name \"+3.3V\""
-			(at 256.54 128.27 0)
+			(at 262.89 123.19 0)
 			(hide yes)
 			(show_name no)
@@
 	(symbol
 		(lib_id "Device:R")
-		(at 223.52 137.16 0)
+		(at 229.87 132.08 0)
 		(unit 1)
 		(body_style 1)
@@
 		(dnp no)
 		(property "Reference" "R35"
-			(at 218.44 137.16 0)
+			(at 224.79 132.08 0)
 			(show_name no)
 			(do_not_autoplace no)
@@
 		)
 		(property "Value" "10k"
-			(at 217.17 139.7 0)
+			(at 223.52 134.62 0)
 			(show_name no)
 			(do_not_autoplace no)
@@
 		)
 		(property "Footprint" "Resistor_SMD:R_0402_1005Metric"
-			(at 221.742 137.16 0)
+			(at 228.092 132.08 0)
 			(hide yes)
 			(show_name no)
@@
 		)
 		(property "Datasheet" ""
-			(at 223.52 137.16 0)
+			(at 229.87 132.08 0)
 			(hide yes)
 			(show_name no)
@@
 		)
 		(property "Description" "Resistor"
-			(at 223.52 137.16 0)
+			(at 229.87 132.08 0)
 			(hide yes)
 			(show_name no)
@@
 	(symbol
 		(lib_id "power:+3.3V")
-		(at 190.5 128.27 0)
+		(at 196.85 123.19 0)
 		(unit 1)
 		(body_style 1)
@@
 		(fields_autoplaced yes)
 		(property "Reference" "#PWR054"
-			(at 190.5 132.08 0)
+			(at 196.85 127 0)
 			(hide yes)
 			(show_name no)
@@
 		)
 		(property "Value" "+3.3V"
-			(at 190.5 123.19 0)
+			(at 196.85 118.11 0)
 			(show_name no)
 			(do_not_autoplace no)
@@
 		)
 		(property "Footprint" ""
-			(at 190.5 128.27 0)
+			(at 196.85 123.19 0)
 			(hide yes)
 			(show_name no)
@@
 		)
 		(property "Datasheet" ""
-			(at 190.5 128.27 0)
+			(at 196.85 123.19 0)
 			(hide yes)
 			(show_name no)
@@
 		)
 		(property "Description" "Power symbol creates a global label with name \"+3.3V\""
-			(at 190.5 128.27 0)
+			(at 196.85 123.19 0)
 			(hide yes)
 			(show_name no)
@@
 	(symbol
 		(lib_id "Device:R")
-		(at 190.5 137.16 0)
+		(at 196.85 132.08 0)
 		(unit 1)
 		(body_style 1)
@@
 		(dnp no)
 		(property "Reference" "R34"
-			(at 185.42 137.16 0)
+			(at 191.77 132.08 0)
 			(show_name no)
 			(do_not_autoplace no)
@@
 		)
 		(property "Value" "10k"
-			(at 184.15 139.7 0)
+			(at 190.5 134.62 0)
 			(show_name no)
 			(do_not_autoplace no)
@@
 		)
 		(property "Footprint" "Resistor_SMD:R_0402_1005Metric"
-			(at 188.722 137.16 0)
+			(at 195.072 132.08 0)
 			(hide yes)
 			(show_name no)
@@
 		)
 		(property "Datasheet" ""
-			(at 190.5 137.16 0)
+			(at 196.85 132.08 0)
 			(hide yes)
 			(show_name no)
@@
 		)
 		(property "Description" "Resistor"
-			(at 190.5 137.16 0)
+			(at 196.85 132.08 0)
 			(hide yes)
 			(show_name no)
