File: poweroutput.kicad_sch (KiCad schematic)
At the start: 0 parts

Commit message: v2
Parts:
- added J4: DG142R-5.08-02P-14-00AH, DG142R-5.08-02P-14-00AH:DG142R-5.08-02P-14-00AH, symbol DG142R-5.08-02P-14-00AH:DG142R-5.08-02P-14-00AH
- added J5: BANANA_POS, symbol Connector_Generic:Conn_01x01
- added J6: BANANA_LOW1, symbol Connector_Generic:Conn_01x01
- added J7: BANANA_LOW2, symbol Connector_Generic:Conn_01x01
