File: usb_pd_controller.kicad_sch (KiCad schematic)
At the start: 28 parts, among them Q1 BSS138, Q2 BSS138, Q3 IRF7855TRPBF, Q4 IRF7855TRPBF, U1 AP33772SDKZ-13-FA02

Commit message: KiCad schematic updates - 2026-09-07
Parts:
- C1, C2, C3, C4, C8, R14, R8, R9: footprint (none) -> Capacitor_SMD:C_01005_0402Metric
- R12, R4, R5, R6, R7: footprint (none) -> Resistor_SMD:R_01005_0402Metric
Changed lines of the file:
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@@
 			)
 		)
-		(property "Footprint" ""
+		(property "Footprint" "Resistor_SMD:R_01005_0402Metric"
 			(at 230.632 71.12 90)
 			(hide yes)
@@
 			)
 		)
-		(property "Footprint" ""
+		(property "Footprint" "Capacitor_SMD:C_01005_0402Metric"
 			(at 167.64 88.138 90)
 			(hide yes)
@@
 			)
 		)
-		(property "Footprint" ""
+		(property "Footprint" "Capacitor_SMD:C_01005_0402Metric"
 			(at 102.5652 109.22 0)
 			(hide yes)
@@
 			)
 		)
-		(property "Footprint" ""
+		(property "Footprint" "Capacitor_SMD:C_01005_0402Metric"
 			(at 170.942 93.98 90)
 			(hide yes)
@@
 			)
 		)
-		(property "Footprint" ""
+		(property "Footprint" "Capacitor_SMD:C_01005_0402Metric"
 			(at 140.97 98.298 90)
 			(hide yes)
@@
 			)
 		)
-		(property "Footprint" ""
+		(property "Footprint" "Capacitor_SMD:C_01005_0402Metric"
 			(at 139.7 57.4548 0)
 			(hide yes)
@@
 			)
 		)
-		(property "Footprint" ""
+		(property "Footprint" "Capacitor_SMD:C_01005_0402Metric"
 			(at 114.6048 45.72 0)
 			(hide yes)
@@
 			)
 		)
-		(property "Footprint" ""
+		(property "Footprint" "Resistor_SMD:R_01005_0402Metric"
 			(at 140.97 70.358 90)
 			(hide yes)
@@
 			)
 		)
-		(property "Footprint" ""
+		(property "Footprint" "Resistor_SMD:R_01005_0402Metric"
 			(at 268.732 71.12 90)
 			(hide yes)
@@
 			)
 		)
-		(property "Footprint" ""
+		(property "Footprint" "Resistor_SMD:R_01005_0402Metric"
 			(at 268.732 134.62 90)
 			(hide yes)
@@
 			)
 		)
-		(property "Footprint" ""
+		(property "Footprint" "Capacitor_SMD:C_01005_0402Metric"
 			(at 144.4752 109.22 0)
 			(hide yes)
@@
 			)
 		)
-		(property "Footprint" ""
+		(property "Footprint" "Capacitor_SMD:C_01005_0402Metric"
 			(at 133.0452 181.61 0)
 			(hide yes)
@@
 			)
 		)
-		(property "Footprint" ""
+		(property "Footprint" "Resistor_SMD:R_01005_0402Metric"
 			(at 234.188 135.89 90)
 			(hide yes)

Commit message: 08/09/26
Connections:
- net TYPE-C KONNEKTÖRÜ: now also U1.1 (ISENP)
- net MCU_3V3 renamed +3.3V
- net USB_VBUS: no longer names the net of R11.1
- net USB_VBUS: no longer U1.1 (ISENP)
Other:
- moved on the sheet: C8, Q3, Q4, R11

Commit message: 10/09/26
Parts:
- R14, R8, R9: footprint Capacitor_SMD:C_01005_0402Metric -> Resistor_SMD:R_0603_1608Metric
Connections:
- net TYPE-C KONNEKTÖRÜ is gone; now on net USB_VBUS: U1.1 (ISENP)
- net GND: now also D1.1 (K); no longer D1.2 (A)
- net PD_5V: now also C4.1, TP4.1, U1.20 (V5V)
- net PD_GATE: now also TP5.1
- net PD_I2C_SCL_3V3: now also R4.1
- net PD_I2C_SCL_5V: now also R5.2
- net PD_I2C_SDA_3V3: now also R7.2
- net PD_I2C_SDA_5V: now also R6.2
- net PD_INT_3V3: now also R9.1
- net PD_INT_5V: now also R8.1, U1.9 (INT)
- net PD_VBUS_SENSED: now also C3.1, TP2.1, U1.24 (VCC)
- net PD_VOUT: now also TP3.1
- net USB_CC1: now also U1.17 (CC1)
- net USB_CC2: now also U1.16 (CC2)
- net USB_VBUS: now reaches TP1.1
- net USB_VBUS: now also R11.1
- net at R14.2: now also D1.2 (A); no longer D1.1 (K)
Other:
- moved on the sheet: C1, C2, C3, C4, C8, D1, Q1, Q2, Q3, Q4, R11, R12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

Commit message: v2
Parts:
- C3: value 1 uF -> 1uF / 50V; footprint Capacitor_SMD:C_01005_0402Metric -> Capacitor_SMD:C_0805_2012Metric
- C4: value 1uF -> 1uF / 10V; footprint Capacitor_SMD:C_01005_0402Metric -> Capacitor_SMD:C_0603_1608Metric
- C8: value 10uF -> 10uF / 50V; footprint Capacitor_SMD:C_01005_0402Metric -> Capacitor_SMD:C_1210_3225Metric
- Q3, Q4: footprint (none) -> Package_SO:SOIC-8_3.9x4.9mm_P1.27mm; symbol Transistor_FET:Q_NMOS_GSD -> Power_Supply_Custom:IRF7855_SO8
- R11: value 5mR -> 5mR / 1W; footprint (none) -> Resistor_SMD:R_2512_6332Metric
Connections:
- net PD_GATE: now also Q3.4 (G), Q4.4 (G); no longer Q3.1 (G), Q4.1 (G)
- net PD_I2C_SCL_3V3: no longer R4.1
- net PD_I2C_SCL_5V: no longer R5.2
- net PD_I2C_SDA_3V3: no longer R7.2
- net PD_I2C_SDA_5V: no longer R6.2
- net PD_INT_5V: no longer R8.1
- net PD_VBUS_SENSED: now also Q4.5 (D), Q4.6 (D), Q4.7 (D), Q4.8 (D); no longer Q4.3 (D)
- net PD_VOUT: now also Q3.5 (D), Q3.6 (D), Q3.7 (D), Q3.8 (D); no longer Q3.3 (D)
- net USB_VBUS: no longer R11.1
- net at Q3.2 (S), Q4.2 (S): now also Q3.1 (S), Q3.3 (S), Q4.1 (S), Q4.3 (S)
Other:
- moved on the sheet: R11, R5, R8, R9, TP1, TP2, TP3

Commit message: 11 Eylül
Parts:
- C1, C2: footprint Capacitor_SMD:C_01005_0402Metric -> Capacitor_SMD:C_0402_1005Metric
- C4: footprint Capacitor_SMD:C_0603_1608Metric -> Capacitor_SMD:C_0402_1005Metric
- D1: footprint (none) -> LED_SMD:LED_0402_1005Metric
- R12, R4, R5, R6, R7: footprint Resistor_SMD:R_01005_0402Metric -> Resistor_SMD:R_0402_1005Metric
- R13, R21: footprint (none) -> Resistor_SMD:R_0402_1005Metric
- R14, R8, R9: footprint Resistor_SMD:R_0603_1608Metric -> Resistor_SMD:R_0402_1005Metric
- TH1: value NCP03XH103 / 10k NTC -> TSM0B103F3381RZ / 10k NTC; footprint (none) -> Resistor_SMD:R_0402_1005Metric
- TP1, TP2, TP3, TP4, TP5: footprint (none) -> TestPoint:TestPoint_Pad_D1.0mm
Connections:
- net PD_I2C_SCL_3V3: now also R4.1
- net PD_I2C_SCL_5V: now also R5.2
- net PD_I2C_SDA_3V3: now also R7.2
- net PD_I2C_SDA_5V: now also R6.2
- net PD_INT_5V: now also R8.1
- net USB_VBUS: now also R11.1
Other:
- moved on the sheet: D1, Q1, Q2, Q3, Q4, R11, R4, R5, R6, R7, R8, TP2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
