File: .codex-encoder/userinterface.before.kicad_sch (KiCad schematic)
At the start: 12 parts, among them J3 Conn_01x40, Q6 Q_NMOS_GSD, SW3 L-KLS4-EC12-012424-W

Commit message: 10/09/26
Parts:
- removed R34, R35, R36: 10k, Resistor_SMD:R_0603_1608Metric, symbol Device:R
- renumbered SW3 to SW
Connections:
- net BL_SINK: no longer Q6.3 (D)
- net GND: no longer SW.2 (C), SW.5 (S2)
- net ENCODER_A: no longer names the net of SW.1 (A)
- net ENCODER_B: no longer names the net of SW.3 (B)
- net ENCODER_SW: no longer names the net of SW.4 (S1)
Other:
- note removed: "ENCODER: A=GPIO22, B=GPIO23, SW=GPIO21 3.3V pull-ups; contacts close to GND. Firmware: quadrature state decoding and switch debounce required."
Changed lines of the file:
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@@
 		(dnp no)
 		(fields_autoplaced yes)
-		(property "Reference" "SW3"
+		(property "Reference" "SW"
 			(at 227.965 86.36 0)
 			(show_name no)
@@
 			(project "masaüstü güç kaynağı"
 				(path "/a43081a6-9aa2-4898-9347-bbcb5849dafd/f0e4530d-2b12-46bf-98ff-bd44498f317b"
-					(reference "SW3")
+					(reference "SW")
 					(unit 1)
 				)
@@
 		)
 	)
-(wire (pts (xy 216.535 93.345) (xy 203.2 93.345)) (stroke (width 0) (type default)))
-(global_label "ENCODER_A" (shape passive) (at 203.2 93.345 180) (effects (font (size 1.27 1.27)) (justify right)))
-(wire (pts (xy 216.535 103.505) (xy 203.2 103.505)) (stroke (width 0) (type default)))
-(global_label "ENCODER_B" (shape passive) (at 203.2 103.505 180) (effects (font (size 1.27 1.27)) (justify right)))
-(global_label "GND" (shape passive) (at 216.535 98.425 180) (effects (font (size 1.27 1.27)) (justify right)))
-(wire (pts (xy 239.395 97.155) (xy 250.19 97.155)) (stroke (width 0) (type default)))
-(global_label "ENCODER_SW" (shape passive) (at 250.19 97.155 0) (effects (font (size 1.27 1.27)) (justify left)))
-(wire (pts (xy 239.395 99.695) (xy 246.38 99.695)) (stroke (width 0) (type default)))
-(wire (pts (xy 246.38 99.695) (xy 246.38 110.49)) (stroke (width 0) (type default)))
-(global_label "GND" (shape passive) (at 246.38 110.49 0) (effects (font (size 1.27 1.27)) (justify left)))
-(symbol (lib_id "Device:R") (at 190.5 137.16 0) (unit 1) (body_style 1) (exclude_from_sim no) (in_bom yes) (on_board yes) (in_pos_files yes) (dnp no) (property "Reference" "R34" (at 185.42 137.16 0) (show_name no) (do_not_autoplace no) (effects (font (size 1.27 1.27)) (justify left))) (property "Value" "10k" (at 184.14999999999998 139.7 0) (show_name no) (do_not_autoplace no) (effects (font (size 1.27 1.27)) (justify left))) (property "Footprint" "Resistor_SMD:R_0603_1608Metric" (at 188.72199999999998 137.16 0) (hide yes) (show_name no) (do_not_autoplace no) (effects (font (size 1.27 1.27)))) (property "Datasheet" "" (at 190.5 137.16 0) (hide yes) (show_name no) (do_not_autoplace no) (effects (font (size 1.27 1.27)))) (property "Description" "Resistor" (at 190.5 137.16 0) (hide yes) (show_name no) (do_not_autoplace no) (effects (font (size 1.27 1.27)))) (pin "1") (pin "2") (instances (project "masaüstü güç kaynağı" (path "/a43081a6-9aa2-4898-9347-bbcb5849dafd/f0e4530d-2b12-46bf-98ff-bd44498f317b" (reference "R34") (unit 1)))))
-(wire (pts (xy 190.5 133.35) (xy 190.5 128.26999999999998)) (stroke (width 0) (type default)))
-(global_label "+3.3V" (shape passive) (at 190.5 128.26999999999998 0) (effects (font (size 1.27 1.27)) (justify left)))
-(wire (pts (xy 190.5 140.97) (xy 190.5 146.05)) (stroke (width 0) (type default)))
-(global_label "ENCODER_A" (shape passive) (at 190.5 146.05 0) (effects (font (size 1.27 1.27)) (justify left)))
-(symbol (lib_id "Device:R") (at 223.52 137.16 0) (unit 1) (body_style 1) (exclude_from_sim no) (in_bom yes) (on_board yes) (in_pos_files yes) (dnp no) (property "Reference" "R35" (at 218.44 137.16 0) (show_name no) (do_not_autoplace no) (effects (font (size 1.27 1.27)) (justify left))) (property "Value" "10k" (at 217.17000000000002 139.7 0) (show_name no) (do_not_autoplace no) (effects (font (size 1.27 1.27)) (justify left))) (property "Footprint" "Resistor_SMD:R_0603_1608Metric" (at 221.74200000000002 137.16 0) (hide yes) (show_name no) (do_not_autoplace no) (effects (font (size 1.27 1.27)))) (property "Datasheet" "" (at 223.52 137.16 0) (hide yes) (show_name no) (do_not_autoplace no) (effects (font (size 1.27 1.27)))) (property "Description" "Resistor" (at 223.52 137.16 0) (hide yes) (show_name no) (do_not_autoplace no) (effects (font (size 1.27 1.27)))) (pin "1") (pin "2") (instances (project "masaüstü güç kaynağı" (path "/a43081a6-9aa2-4898-9347-bbcb5849dafd/f0e4530d-2b12-46bf-98ff-bd44498f317b" (reference "R35") (unit 1)))))
-(wire (pts (xy 223.52 133.35) (xy 223.52 128.26999999999998)) (stroke (width 0) (type default)))
-(global_label "+3.3V" (shape passive) (at 223.52 128.26999999999998 0) (effects (font (size 1.27 1.27)) (justify left)))
-(wire (pts (xy 223.52 140.97) (xy 223.52 146.05)) (stroke (width 0) (type default)))
-(global_label "ENCODER_B" (shape passive) (at 223.52 146.05 0) (effects (font (size 1.27 1.27)) (justify left)))
-(symbol (lib_id "Device:R") (at 256.54 137.16 0) (unit 1) (body_style 1) (exclude_from_sim no) (in_bom yes) (on_board yes) (in_pos_files yes) (dnp no) (property "Reference" "R36" (at 251.46 137.16 0) (show_name no) (do_not_autoplace no) (effects (font (size 1.27 1.27)) (justify left))) (property "Value" "10k" (at 250.19 139.7 0) (show_name no) (do_not_autoplace no) (effects (font (size 1.27 1.27)) (justify left))) (property "Footprint" "Resistor_SMD:R_0603_1608Metric" (at 254.762 137.16 0) (hide yes) (show_name no) (do_not_autoplace no) (effects (font (size 1.27 1.27)))) (property "Datasheet" "" (at 256.54 137.16 0) (hide yes) (show_name no) (do_not_autoplace no) (effects (font (size 1.27 1.27)))) (property "Description" "Resistor" (at 256.54 137.16 0) (hide yes) (show_name no) (do_not_autoplace no) (effects (font (size 1.27 1.27)))) (pin "1") (pin "2") (instances (project "masaüstü güç kaynağı" (path "/a43081a6-9aa2-4898-9347-bbcb5849dafd/f0e4530d-2b12-46bf-98ff-bd44498f317b" (reference "R36") (unit 1)))))
-(wire (pts (xy 256.54 133.35) (xy 256.54 128.26999999999998)) (stroke (width 0) (type default)))
-(global_label "+3.3V" (shape passive) (at 256.54 128.26999999999998 0) (effects (font (size 1.27 1.27)) (justify left)))
-(wire (pts (xy 256.54 140.97) (xy 256.54 146.05)) (stroke (width 0) (type default)))
-(global_label "ENCODER_SW" (shape passive) (at 256.54 146.05 0) (effects (font (size 1.27 1.27)) (justify left)))
-(text "ENCODER: A=GPIO22, B=GPIO23, SW=GPIO21\n3.3V pull-ups; contacts close to GND.\nFirmware: quadrature state decoding and switch debounce required." (at 182.88 158.75 0) (effects (font (size 1.27 1.27)) (justify left top)))
-(wire (pts (xy 57.785 156.845) (xy 67.945 156.845)) (stroke (width 0) (type default)))
 )
