File: reports/fixes-20260909/before/masaüstü güç kaynağı.kicad_sch (KiCad schematic)
At the start: 0 parts

Commit message: 10/09/26
Other:
- sheet USB_PD_CONTROLLER ports: added USB_CC1, USB_CC2, USB_VBUS; removed none
Changed lines of the file:
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@@
 		)
 	)
-	(sheet (at 83.82 40.64) (size 36.83 38.1) (exclude_from_sim no) (in_bom yes) (on_board yes) (dnp no) (fields_autoplaced yes) (stroke (width 0.1524) (type solid) (color 228 64 255 1)) (fill (color 227 90 255 1)) (property "Sheetname" "USB_PD_CONTROLLER" (at 83.82 39.9284 0) (show_name no) (do_not_autoplace no) (effects (font (size 1.27 1.27)) (justify left bottom))) (property "Sheetfile" "usb_pd_controller.kicad_sch" (at 83.82 79.3246 0) (show_name no) (do_not_autoplace no) (effects (font (size 1.27 1.27)) (justify left top))) (instances (project "masaüstü güç kaynağı" (path "/a43081a6-9aa2-4898-9347-bbcb5849dafd" (page "2")))))
+	(sheet
+		(at 83.82 40.64)
+		(size 36.83 38.1)
+		(exclude_from_sim no)
+		(in_bom yes)
+		(on_board yes)
+		(dnp no)
+		(fields_autoplaced yes)
+		(stroke
+			(width 0.1524)
+			(type solid)
+			(color 228 64 255 1)
+		)
+		(fill
+			(color 227 90 255 1)
+		)
+		(property "Sheetname" "USB_PD_CONTROLLER"
+			(at 83.82 39.9284 0)
+			(show_name no)
+			(do_not_autoplace no)
+			(effects
+				(font
+					(size 1.27 1.27)
+				)
+				(justify left bottom)
+			)
+		)
+		(property "Sheetfile" "usb_pd_controller.kicad_sch"
+			(at 83.82 79.3246 0)
+			(show_name no)
+			(do_not_autoplace no)
+			(effects
+				(font
+					(size 1.27 1.27)
+				)
+				(justify left top)
+			)
+		)
+		(pin "USB_CC1" input
+			(at 120.65 49.53 0)
+			(effects
+				(font
+					(size 1.27 1.27)
+				)
+				(justify right)
+			)
+		)
+		(pin "USB_CC2" input
+			(at 120.65 53.34 0)
+			(effects
+				(font
+					(size 1.27 1.27)
+				)
+				(justify right)
+			)
+		)
+		(pin "USB_VBUS" input
+			(at 120.65 44.45 0)
+			(effects
+				(font
+					(size 1.27 1.27)
+				)
+				(justify right)
+			)
+		)
+		(instances
+			(project "masaüstü güç kaynağı"
+				(path "/a43081a6-9aa2-4898-9347-bbcb5849dafd"
+					(page "2")
+				)
+			)
+		)
+	)
 	(sheet
 		(at 219.71 39.37)
