File: reports/fixes-20260909/before/mcu.kicad_sch (KiCad schematic)
At the start: 28 parts, among them J2 DS1021-1X3SF11-B, SW1 BOOT, SW2 RESET, U2 ESP32-C6-WROOM-1, U4 RV-3028-C7

Commit message: 10/09/26
Parts:
- removed R37: 10kR, Resistor_SMD:R_0603_1608Metric, symbol Device:R
- C5: footprint Capacitor_SMD:C_0805_2012Metric -> Capacitor_SMD:C_01005_0402Metric
- J1: renamed from J2; footprint CONNFLY_DS1021-1X3SF11-B:CONNFLY_DS1021-1X3SF11-B -> DS1021-1X3SF11-B:CONNFLY_DS1021-1X3SF11-B
Connections:
- net RTC_SCL: no longer R25.2, U4.3 (SCL)
- new net: R25.2, U4.3 (SCL)
