File: reports/fixes-20260909/before/userinterface.kicad_sch (KiCad schematic)
At the start: 12 parts, among them J3 Conn_01x40, Q6 Q_NMOS_GSD, SW3 L-KLS4-EC12-012424-W

Commit message: 10/09/26
Connections:
- net BL_SINK: no longer Q6.3 (D)
Changed lines of the file:
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@@
 (global_label "ENCODER_SW" (shape passive) (at 256.54 146.05 0) (effects (font (size 1.27 1.27)) (justify left)))
 (text "ENCODER: A=GPIO22, B=GPIO23, SW=GPIO21\n3.3V pull-ups; contacts close to GND.\nFirmware: quadrature state decoding and switch debounce required." (at 182.88 158.75 0) (effects (font (size 1.27 1.27)) (justify left top)))
-(wire (pts (xy 57.785 156.845) (xy 67.945 156.845)) (stroke (width 0) (type default)))
 )
