File: reports/review-20260910/before/powergeneration.kicad_sch (KiCad schematic)
At the start: 18 parts, among them U5 AOZ1284PI, U6 TL431BIDBZR

Commit message: v2
Parts:
- removed R43: 1kR / 2W, Resistor_SMD:R_2512_6332Metric, symbol Device:R
- removed U6: TL431BIDBZR, Package_TO_SOT_SMD:SOT-23, symbol Reference_Voltage:TL431DBZ
- C15, C16: DesignNote X7R; bank effective Cout >=44uF at 3.3V. Confirm exact MPN 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 -> X7R; bank effective Cout >=44uF at 3.3V; actual C/ESR UNRES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
- C19: value 18nF / 16V -> UNRESOLVED
- R41: value 12.7kR 1% -> UNRESOLVED
Other:
- note added: "L/D MPN + footprints: UNRESOLVED Isat >=2A normal load; fault capability unverified Cout effective >=44uF; DC bias must be checked"
- note added: "VIN = EXPOSED PAD 9: PD_VOUT, NOT GND. EN requires independent 1.2..5V bias. DO NOT connect to PD_VOUT. COMP values UNRESOLVED: datasheet GEA / Cc equations conflict. RF=100k: table 500kHz; equation 476.19kHz. Actual range UNRESOLVED."
- note removed: "L/D exact MPN and footprints require selection. L: Isat >=2A normal load, Irms >=1.5A. Cout effective >=44uF; check DC-bias curves."
- note removed: "VIN = EXPOSED PAD 9: PD_VOUT, NOT GND. EN: 2.495V shunt bias; R43 dissipation 0.65W at 28V. COMP: Rc=12.7k, Cc=18nF; fc about 8.5..10kHz at Cout_eff=44uF. RF=100k: table 500kHz; equation 476.19kHz. Verify on prototype."
