File: reports/review-20260910/before/powersensing.kicad_sch (KiCad schematic)
At the start: 4 parts, among them U3 INA228

Commit message: v2
Parts:
- RShunt: value 5mR / 1W -> 5m; footprint Resistor_SMD:R_2512_6332Metric -> Resistor_SMD:R_01005_0402Metric
Changed lines of the file:
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@@
 		(dnp no)
 		(property "Reference" "U3"
-			(at 132.588 85.598 0)
+			(at 133.35 90.17 0)
 			(show_name no)
 			(do_not_autoplace no)
@@
 		)
 		(property "Value" "INA228"
-			(at 130.81 87.884 0)
+			(at 141.605 90.17 0)
 			(show_name no)
 			(do_not_autoplace no)
@@
 			)
 		)
-		(property "Value" "5mR / 1W"
+		(property "Value" "5m"
 			(at 85.725 114.3 90)
 			(show_name no)
@@
 			)
 		)
-		(property "Footprint" "Resistor_SMD:R_2512_6332Metric"
+		(property "Footprint" "Resistor_SMD:R_01005_0402Metric"
 			(at 85.725 119.888 90)
 			(hide yes)
