File: reports/review-20260910/before/usb_pd_controller.kicad_sch (KiCad schematic)
At the start: 28 parts, among them J2 DS1021-1X3SF11-B, SW1 BOOT, SW2 RESET, U2 ESP32-C6-WROOM-1, U4 RV-3028-C7

Commit message: v2
Parts:
- removed BT1: Battery_Cell, symbol Device:Battery_Cell
- removed C10, C9: 100nF, symbol Device:C
- removed C5: 22uF, Capacitor_SMD:C_0805_2012Metric, symbol Device:C
- removed C6: 100nF, Capacitor_SMD:C_01005_0402Metric, symbol Device:C
- removed C7: 1uF, Capacitor_SMD:C_01005_0402Metric, symbol Device:C
- removed J2: DS1021-1X3SF11-B, CONNFLY_DS1021-1X3SF11-B:CONNFLY_DS1021-1X3SF11-B, symbol DS1021-1X3SF11-B:DS1021-1X3SF11-B
- removed R1: 10 kΩ, Resistor_SMD:R_01005_0402Metric, symbol Device:R
- removed R10, R23: 10k, symbol Device:R
- removed R15: 22 R, symbol Device:R
- removed R16: 22R, symbol Device:R
- removed R2, R3: 22Ω, symbol Device:R
- removed R22: 1K, Resistor_SMD:R_01005_0402Metric, symbol Device:R
- removed R24: 4,7k, symbol Device:R
- removed R25: 4.7k, Resistor_SMD:R_01005_0402Metric, symbol Device:R
- removed R26: 4.7K, Resistor_SMD:R_01005_0402Metric, symbol Device:R
- removed R37: 10kR, Resistor_SMD:R_0603_1608Metric, symbol Device:R
- removed SW1: BOOT, symbol Switch:SW_Push
- removed SW2: RESET, symbol Switch:SW_Push
- removed TP10, TP6, TP7, TP8, TP9: TestPoint, symbol Connector:TestPoint
- removed U2: ESP32-C6-WROOM-1, PCM_Espressif:ESP32-C6-WROOM-1, symbol PCM_Espressif:ESP32-C6-WROOM-1
- removed U4: RV-3028-C7, Package_SON:MicroCrystal_C7_SON-8_1.5x3.2mm_P0.9mm, symbol Timer_RTC:RV-3028-C7
- added C1, C2: 100 nF, Capacitor_SMD:C_01005_0402Metric, symbol Device:C
- added C3: 1 uF, Capacitor_SMD:C_01005_0402Metric, symbol Device:C
- added C4: 1uF, Capacitor_SMD:C_01005_0402Metric, symbol Device:C
- added C8: 10uF, Capacitor_SMD:C_01005_0402Metric, symbol Device:C
- added D1: LED, symbol Device:LED
- added Q1, Q2: BSS138, Package_TO_SOT_SMD:SOT-23, symbol Transistor_FET:BSS138
- added Q3, Q4: IRF7855TRPBF, symbol Transistor_FET:Q_NMOS_GSD
- added R11: 5mR, symbol Device:R
- added R12: 6.2k, Resistor_SMD:R_01005_0402Metric, symbol Device:R
- added R13: 100R, symbol Device:R
- added R14: 2.2k, Resistor_SMD:R_0603_1608Metric, symbol Device:R
- added R21: 100K, symbol Device:R
- added R4: 4.7 kΩ, Resistor_SMD:R_01005_0402Metric, symbol Device:R
- added R5: 4.7kΩ, Resistor_SMD:R_01005_0402Metric, symbol Device:R
- added R6: 4.7 k, Resistor_SMD:R_01005_0402Metric, symbol Device:R
- added R7: 4.7k, Resistor_SMD:R_01005_0402Metric, symbol Device:R
- added R8: 12k, Resistor_SMD:R_0603_1608Metric, symbol Device:R
- added R9: 20k, Resistor_SMD:R_0603_1608Metric, symbol Device:R
- added TH1: NCP03XH103 / 10k NTC, symbol Device:Thermistor_NTC
- added TP1, TP2, TP3, TP4, TP5: TestPoint, symbol Connector:TestPoint
- added U1: AP33772SDKZ-13-FA02, Package_DFN_QFN:Texas_RTW_WQFN-24-1EP_4x4mm_P0.5mm_EP2.7x2.7mm, symbol Interface_USB:AP33772SDKZ-xx-FA02
Connections:
- net +3.3V: now also Q1.1 (G), Q2.1 (G), R4.2, R7.1
- net GND: now also C1.2, C2.2, C3.2, C4.2, C8.2, D1.1 (K), R21.1, R9.2, TH1.1, U1.25 (GND), U1.3 (GND)
- net PD_I2C_SCL_3V3: now also Q1.2 (S)
- net PD_I2C_SDA_3V3: now also Q2.2 (S)
- net PD_INT_3V3: now also R8.2, R9.1
- new net: C2.1, U1.15 (IFB)
- new net: Q3.2 (S), Q4.2 (S)
- new net: R14.1, U1.8 (LED)
- new net: D1.2 (A), R14.2
- new net: R21.2, U1.11 (VSEL)
- new net: C1.1, U1.12 (V18)
- new net: TH1.2, U1.13 (OTP)
- new net: R13.1, U1.22 (VOUT)
- new net: R12.1, U1.23 (PWR_EN)
- new net PD_5V: C4.1, R5.1, R6.1, TP4.1, U1.20 (V5V)
- new net PD_GATE: Q3.1 (G), Q4.1 (G), R12.2, TP5.1
- new net PD_I2C_SCL_5V: Q1.3 (D), U1.5 (SCL)
- new net PD_I2C_SDA_5V: Q2.3 (D), U1.4 (SDA)
- new net PD_INT_5V: U1.9 (INT)
- new net PD_VBUS_SENSED: C3.1, Q4.3 (D), R11.2, TP2.1, U1.24 (VCC)
- new net PD_VOUT: C8.1, Q3.3 (D), R13.2, TP3.1
- new net USB_CC1: U1.17 (CC1)
- new net USB_CC2: U1.16 (CC2)
- new net USB_VBUS: TP1.1, U1.1 (ISENP)
- no-connect marks 1 -> 4
Other:
- removed sheet CALC_MCU
- added sheet CALC_USB_PD_CONTROLLER (calc_usb_pd_controller.kicad_sch)
- note removed: "Boşta kalan pinlere 22R sonrası bir test point koyarak daha sonra kullanılabilir halde tasarım yapalım."
- note removed: "ESP32 decoupling kapasiteleri pin ile bağlantılı gösterilmesi layout çiziminde bunların pine yakın konumlandırılması gerektiğini hatırlatır."
- note removed: "ESP32'yi nasıl programlayacağız? Uart pinlerini bağlamamız gerekiyor mu?"
- note removed: "Encoder seçimi yapılarak uygun şekilde bağlantısı yapılmalı!"
- note removed: "PORT tanımlamaları yatay konumlandırılmalı ve giriş, çıkış gibi gösterimleri doğru yapılmalı."
- note removed: "Pin ataması ESP32'nin uygunlupu kontrol edilerek birbirine yakın pinler ile bağlanmalı. Bu layout çizimini kolaylaştırır."
- note removed: "RTC pil konusu netleştirilecek."
