File: reports/review-20260910/before/userinterface.kicad_sch (KiCad schematic)
At the start: 12 parts, among them J3 Conn_01x40, Q5 AO3400A, SW3 L-KLS4-EC12-012424-W

Commit message: v2
Parts:
- removed Q5: AO3400A, AO3400A:SOT95P280X125-3N, symbol AO3400A:AO3400A
- added Q6: Q_NMOS_GSD, symbol Transistor_FET:Q_NMOS_GSD
Connections:
- net GND: now also Q6.2 (S)
- net at R28.2, R29.1: now also Q6.1 (G)
Other:
- moved on the sheet: R28, R29
