File: reports/layout-20260911/backups/before-gnd-routing-correction-20260913.kicad_pcb (KiCad board)
At the start: 4 copper layers, 90 x 55 mm, 100 parts, among them J1 DX07B024JJ1R1500, J2 DS1021-1X3SF11-B, J3 NHD-2.4-240320AF-CSXP, J4 DG142R-5.08-02P-14-00AH, Q1 BSS138, Q2 BSS138, Q3 IRF7855TRPBF, Q4 IRF7855TRPBF, SW1 BOOT / PTS810, SW2 RESET / PTS810, SW3 L-KLS4-EC12-012424-W, U1 AP33772SDKZ-13-FA02, U2 ESP32-C6-WROOM-1, U3 INA228, U4 RV-3028-C7, U5 AOZ1284PI, U6 TL431BIDBZR, U7 TPS61023DRLR, U8 CAT4104V-GT3, U9 TPD4E05U06QDQARQ1

Commit message: 12/09/26
Routing:
- net GND: track 17.8 -> 358.8 mm, vias 48 -> 13
- removed copper zone on F.Cu, net GND
