File: reports/layout-20260911/backups/masaüstü güç kaynağı_before_lower_placement_20260912_194621.kicad_pcb (KiCad board)
At the start: 4 copper layers, 90 x 55 mm, 100 parts, among them J1 DX07B024JJ1R1500, J2 DS1021-1X3SF11-B, J3 NHD-2.4-240320AF-CSXP, J4 DG142R-5.08-02P-14-00AH, Q1 BSS138, Q2 BSS138, Q3 IRF7855TRPBF, Q4 IRF7855TRPBF, SW1 BOOT / PTS810, SW2 RESET / PTS810, SW3 L-KLS4-EC12-012424-W, U1 AP33772SDKZ-13-FA02, U2 ESP32-C6-WROOM-1, U3 INA228, U4 RV-3028-C7, U5 AOZ1284PI, U6 TL431BIDBZR, U7 TPS61023DRLR, U8 CAT4104V-GT3, U9 TPD4E05U06QDQARQ1

Commit message: 12/09/26
Parts:
- moved C15 33.4 mm to (73.5, 40.0), turned to 0 degrees
- moved C17 23.7 mm to (77.2, 40.0), turned to 0 degrees
- moved D2 22.0 mm to (75.0, 53.5), turned to 90 degrees
- moved L1 21.5 mm to (69.0, 47.0), turned to 0 degrees
- moved R46 18.7 mm to (62.5, 64.2)
- moved R38 16.3 mm to (69.0, 40.8), turned to 0 degrees
- moved R43 16.0 mm to (51.0, 48.2), turned to 0 degrees
- moved R40 15.2 mm to (77.2, 41.5)
- moved R28 13.7 mm to (59.5, 57.5), turned to 0 degrees
- moved R44 12.9 mm to (56.5, 63.5)
- moved C16 12.1 mm to (51.0, 43.8), turned to 0 degrees
- moved C20 11.5 mm to (66.2, 57.5)
- moved C14 10.8 mm to (60.0, 40.0)
- moved C19 10.6 mm to (66.0, 40.8)
- moved R29 10.1 mm to (62.5, 57.5), turned to 0 degrees
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Routing:
- net PD_VOUT: track 59.8 -> 0.00 mm, vias 5 -> 0
- net +3.3V: track 36.9 -> 0.00 mm, vias 2 -> 0
- net OUT_POS: track 29.4 -> 0.00 mm, vias 2 -> 0
- net USB_VBUS: track 26.0 -> 0.00 mm
- net /POWER GENERATION/EN_CTRL: track 20.8 -> 0.00 mm
- net GND: track 17.8 -> 0.00 mm, vias 48 -> 0
- net PD_VBUS_SENSED: track 12.3 -> 0.00 mm
- net Net-(Q3-S-Pad1): track 11.0 -> 0.00 mm
- net /POWER GENERATION/LX_SW: track 10.3 -> 0.00 mm
- net /POWER GENERATION/FB_3V3: track 4.13 -> 0.00 mm
- net /POWER GENERATION/COMP_NODE: track 3.45 -> 0.00 mm
- net Net-(U5-BST): track 2.72 -> 0.00 mm
- net /POWER GENERATION/SS_RAMP: track 2.52 -> 0.00 mm
- net /POWER GENERATION/FSW_SET: track 1.79 -> 0.00 mm
- net Net-(C19-Pad1): track 1.51 -> 0.00 mm
- removed copper zone on F.Cu, net GND
