File: REV_B_20260914/usb_c_input.kicad_sch (KiCad schematic)
At the start: 5 parts, among them J1 DX07B024JJ1R1500, U9 TPD4E05U06QDQARQ1

Commit message: connector
Parts:
- removed D4, D5: AQ3130E-01ETG (bidirectional), Diode_SMD:D_SOD-882, symbol Device:D_TVS
- added J7: USB_C_Receptacle_USB2.0_16P, Connector_USB:USB_C_Receptacle_GCT_USB4105-xx-A_16P_TopMnt_Horizontal, symbol Connector:USB_C_Receptacle_USB2.0_16P
- added U10: TPD4EUSB30, Package_SON:USON-10_2.5x1.0mm_P0.5mm, symbol Power_Protection:TPD4EUSB30
Connections:
- net GND: now also J7.A1 (GND), J7.A12 (GND), J7.B1 (GND), J7.B12 (GND), J7.SH (SHIELD); no longer J1.A1 (GND), J1.A12 (GND), J1.B1 (GND), J1.B12 (GND), J1.SH (SHIELD)
- net USB_CC1: now also J7.A5 (CC1); no longer J1.A5 (CC1)
- net USB_CC2: now also J7.B5 (CC2); no longer J1.B5 (CC2)
- net USB_DM: now also J7.A7 (D-), J7.B7 (D-); no longer J1.A7 (D-), J1.B7 (D-)
- net USB_DP: now also J7.A6 (D+), J7.B6 (D+); no longer J1.A6 (D+), J1.B6 (D+)
- net USB_VBUS: now also J7.A4 (VBUS), J7.A9 (VBUS), J7.B4 (VBUS), J7.B9 (VBUS); no longer J1.A4 (VBUS), J1.A9 (VBUS), J1.B4 (VBUS), J1.B9 (VBUS)
- new net: U10.3 (GND), U10.8 (GND)
- new net: J1.A1 (GND), J1.A12 (GND), J1.B1 (GND), J1.B12 (GND)
- new net: J1.A4 (VBUS), J1.A9 (VBUS), J1.B4 (VBUS), J1.B9 (VBUS)
- no-connect marks 16 -> 17
