File: hardware/gopo.kicad_pcb (KiCad board)
At the start: 4 copper layers, 60 x 40 mm, 0 parts

Commit message: pcb dosyası lokalden projeye taşındı
Parts:
- added BT1: CR2032 holder, Power_Output_Custom:KLS_CR2032_05, B.Cu at (44.0, 119.1)
- added C1: 100 nF, Capacitor_SMD:C_0402_1005Metric, B.Cu at (57.2, 104.8)
- added C10: 100nF, Capacitor_SMD:C_0402_1005Metric, B.Cu at (74.1, 121.6)
- added C11: 100nF, Capacitor_SMD:C_0402_1005Metric, B.Cu at (79.0, 90.0)
- added C12: 10uF, Capacitor_SMD:C_0402_1005Metric, F.Cu at (31.5, 101.4)
- added C13: 10uF, Capacitor_SMD:C_0402_1005Metric, F.Cu at (35.2, 101.5)
- added C14: 100nF, Capacitor_SMD:C_0402_1005Metric, F.Cu at (36.3, 101.5)
- added C15: 47uF, Capacitor_SMD:C_0402_1005Metric, F.Cu at (28.9, 102.2)
- added C16: 47uF, Capacitor_SMD:C_0402_1005Metric, F.Cu at (30.4, 101.5)
- added C17: 100nF / 16V, Capacitor_SMD:C_0402_1005Metric, F.Cu at (28.9, 103.5)
- added C18: 10nF, Capacitor_SMD:C_0402_1005Metric, F.Cu at (38.9, 104.9)
- added C19: 18nF / 16V, Capacitor_SMD:C_0402_1005Metric, F.Cu at (39.1, 109.4)
- added C2: 100 nF, Capacitor_SMD:C_0402_1005Metric, B.Cu at (53.6, 106.6)
- added C20: 22uF, Capacitor_SMD:C_0402_1005Metric, F.Cu at (45.8, 112.1)
- added C21: 22uF, Capacitor_SMD:C_0402_1005Metric, F.Cu at (50.7, 110.3)
- added C22: 100nF / 16V, Capacitor_SMD:C_0402_1005Metric, F.Cu at (52.2, 105.0)
- added C3: 1uF / 50V, Capacitor_SMD:C_0402_1005Metric, B.Cu at (49.6, 101.7)
- added C4: 1uF / 10V, Capacitor_SMD:C_0402_1005Metric, B.Cu at (49.7, 107.5)
- added C5: 22uF, Capacitor_SMD:C_0402_1005Metric, B.Cu at (80.7, 118.7)
- added C6: 100nF, Capacitor_SMD:C_0402_1005Metric, B.Cu at (80.7, 119.7)
- added C7: 1uF, Capacitor_SMD:C_0402_1005Metric, B.Cu at (77.3, 119.1)
- added C8: 10uF / 50V, Capacitor_SMD:C_0402_1005Metric, F.Cu at (33.9, 109.4)
- added C9: 100nF, Capacitor_SMD:C_0402_1005Metric, B.Cu at (76.2, 121.6)
- added D1: LED, LED_SMD:LED_0402_1005Metric, B.Cu at (59.3, 101.4)
- added D2: SS2060FL_R1_00001, Diode_SMD:D_SOD-123F, F.Cu at (27.4, 105.4)
- added D3: AQ3130E-01ETG (bidirectional), Diode_SMD:D_SOD-882, F.Cu at (35.0, 118.6)
- added J2: DS1021-1X3SF11-B, CONNFLY_DS1021-1X3SF11-B:CONNFLY_DS1021-1X3SF11-B, F.Cu at (107.6, 69.3)
- added J3: NHD-2.4-240320AF-CSXP, Molex_541324062:CON_541324062_MOL, F.Cu at (58.3, 114.0)
- added J4: DG142R-5.08-02P-14-00AH, DG142R-5.08-02P-14-00AH:DG142R-5.08-02P-14-00AH, B.Cu at (36.8, 94.0)
- added J7: USB_C_Receptacle_USB2.0_16P, Connector_USB:USB_C_Receptacle_GCT_USB4105-xx-A_16P_TopMnt_Horizontal, F.Cu at (28.3, 121.7)
- added L1: SRI0704-220M, Inductor_SMD:L_7.3x7.3_H4.5, F.Cu at (33.4, 96.0)
- added L2: 2.2uH, Inductor_SMD:L_Wuerth_MAPI-4030, F.Cu at (51.9, 113.2)
- added Q1: BSS138, Package_TO_SOT_SMD:SOT-23, B.Cu at (56.3, 97.6)
- added Q2: BSS138, Package_TO_SOT_SMD:SOT-23, B.Cu at (52.6, 97.6)
- added Q3: IRF7855TRPBF, Package_SO:SOIC-8_3.9x4.9mm_P1.27mm, B.Cu at (43.4, 104.1)
- added Q4: IRF7855TRPBF, Package_SO:SOIC-8_3.9x4.9mm_P1.27mm, B.Cu at (44.5, 93.8)
- added R1: 10 kΩ, Resistor_SMD:R_0402_1005Metric, B.Cu at (78.6, 119.1)
- added R10: 10k, Resistor_SMD:R_0402_1005Metric, B.Cu at (64.4, 90.4)
- added R11: 5mR / 1W, Resistor_SMD:R_0402_1005Metric, B.Cu at (46.4, 99.0)
- added R12: 6.2k, Resistor_SMD:R_0402_1005Metric, B.Cu at (49.6, 103.9)
- added R13: 100R, Resistor_SMD:R_0402_1005Metric, B.Cu at (49.6, 102.8)
- added R14: 2.2k, Resistor_SMD:R_0402_1005Metric, B.Cu at (57.2, 101.4)
- added R15: 22 R, Resistor_SMD:R_0402_1005Metric, B.Cu at (70.1, 119.8)
- added R16: 22R, Resistor_SMD:R_0402_1005Metric, B.Cu at (72.4, 119.8)
- added R2: 22Ω, Resistor_SMD:R_0402_1005Metric, B.Cu at (64.7, 119.7)
- added R21: 100K, Resistor_SMD:R_0402_1005Metric, B.Cu at (57.2, 103.7)
- added R22: 1K, Resistor_SMD:R_0402_1005Metric, B.Cu at (75.2, 121.6)
- added R23: 10k, Resistor_SMD:R_0402_1005Metric, B.Cu at (77.3, 121.6)
- added R24: 4,7k, Resistor_SMD:R_0402_1005Metric, B.Cu at (71.0, 125.2)
- added R25: 4.7k, Resistor_SMD:R_0402_1005Metric, B.Cu at (72.3, 125.2)
- added R26: 4.7K, Resistor_SMD:R_0402_1005Metric, B.Cu at (73.5, 125.2)
- added R27: 10K, Resistor_SMD:R_0402_1005Metric, B.Cu at (78.2, 96.0)
- added R28: 100R, Resistor_SMD:R_0402_1005Metric, F.Cu at (52.2, 107.6)
- added R29: 100kR, Resistor_SMD:R_0402_1005Metric, F.Cu at (52.2, 106.2)
- added R3: 22Ω, Resistor_SMD:R_0402_1005Metric, B.Cu at (66.3, 119.7)
- added R34: 10k, Resistor_SMD:R_0402_1005Metric, B.Cu at (104.6, 84.8)
- added R35: 10k, Resistor_SMD:R_0402_1005Metric, B.Cu at (99.5, 84.8)
- added R36: 10k, Resistor_SMD:R_0402_1005Metric, B.Cu at (104.9, 63.6)
- added R37: 10kR, Resistor_SMD:R_0402_1005Metric, B.Cu at (68.8, 119.8)
- added R38: 100kR 1%, Resistor_SMD:R_0402_1005Metric, F.Cu at (28.8, 107.3)
- added R39: 10kR 0.1%, Resistor_SMD:R_0402_1005Metric, F.Cu at (38.9, 106.2)
- added R4: 4.7 kΩ, Resistor_SMD:R_0402_1005Metric, B.Cu at (57.3, 94.3)
- added R40: 3.20kR 0.1%, Resistor_SMD:R_0402_1005Metric, F.Cu at (38.9, 107.4)
- added R41: 12.7kR 1%, Resistor_SMD:R_0402_1005Metric, F.Cu at (37.8, 109.4)
- added R42: 100kR, Resistor_SMD:R_0402_1005Metric, F.Cu at (38.9, 103.5)
- added R43: 1kR / 2W, Resistor_SMD:R_0402_1005Metric, F.Cu at (37.5, 101.5)
- added R44: 604kR 0.1%, Resistor_SMD:R_0402_1005Metric, F.Cu at (48.3, 109.7)
- added R45: 100kR 0.1%, Resistor_SMD:R_0402_1005Metric, F.Cu at (45.8, 110.8)
- added R46: 3.24kR 0.1%, Resistor_SMD:R_0402_1005Metric, F.Cu at (52.1, 103.6)
- added R5: 4.7kΩ, Resistor_SMD:R_0402_1005Metric, B.Cu at (55.3, 94.4)
- added R6: 4.7 k, Resistor_SMD:R_0402_1005Metric, B.Cu at (51.6, 94.4)
- added R7: 4.7k, Resistor_SMD:R_0402_1005Metric, B.Cu at (53.5, 94.4)
- added R8: 12k, Resistor_SMD:R_0402_1005Metric, B.Cu at (57.2, 102.5)
- added R9: 20k, Resistor_SMD:R_0402_1005Metric, B.Cu at (59.4, 102.5)
- added RShunt1: 5mR / 1W, Resistor_SMD:R_0402_1005Metric, B.Cu at (81.8, 89.9)
- added SW1: BOOT / PTS810, Button_Switch_SMD:SW_SPST_PTS810, B.Cu at (63.1, 94.6)
- added SW2: RESET / PTS810, Button_Switch_SMD:SW_SPST_PTS810, B.Cu at (80.2, 123.2)
- added SW3: L-KLS4-EC1121S-E5A-F12.5, L-KLS4-EC1121S-E5A-F12.5:L-KLS4-EC1121S-E5A-F12.5, B.Cu at (104.6, 81.9)
- added TH1: TSM0B103F3381RZ / 10k NTC, Resistor_SMD:R_0402_1005Metric, B.Cu at (54.7, 106.6)
- added TP1: TestPoint, TestPoint:TestPoint_Pad_D1.0mm, B.Cu at (49.8, 97.8)
- added TP10: TestPoint, TestPoint:TestPoint_Pad_D1.0mm, B.Cu at (65.4, 123.0)
- added TP2: TestPoint, TestPoint:TestPoint_Pad_D1.0mm, B.Cu at (49.7, 100.0)
- added TP3: TestPoint, TestPoint:TestPoint_Pad_D1.0mm, B.Cu at (47.4, 103.6)
- added TP4: TestPoint, TestPoint:TestPoint_Pad_D1.0mm, B.Cu at (49.6, 105.8)
- added TP5: TestPoint, TestPoint:TestPoint_Pad_D1.0mm, B.Cu at (47.3, 101.4)
- added TP6: TestPoint, TestPoint:TestPoint_Pad_D1.0mm, B.Cu at (66.2, 96.8)
- added TP7: TestPoint, TestPoint:TestPoint_Pad_D1.0mm, B.Cu at (67.8, 95.4)
- added TP8: TestPoint, TestPoint:TestPoint_Pad_D1.0mm, B.Cu at (69.3, 96.9)
- added TP9: TestPoint, TestPoint:TestPoint_Pad_D1.0mm, B.Cu at (70.0, 122.9)
- added U1: AP33772SDKZ-13-FA02, Package_DFN_QFN:Texas_RTW_WQFN-24-1EP_4x4mm_P0.5mm_EP2.7x2.7mm, B.Cu at (53.4, 102.9)
- added U10: TPD4EUSB30, Package_SON:USON-10_2.5x1.0mm_P0.5mm, F.Cu at (35.1, 124.8)
- added U2: ESP32-C6-WROOM-1, PCM_Espressif:ESP32-C6-WROOM-1, B.Cu at (73.8, 107.9)
- added U3: INA228, Package_SO:TSSOP-10_3x3mm_P0.5mm, B.Cu at (80.7, 93.8)
- added U4: RV-3028-C7, Package_SON:MicroCrystal_C7_SON-8_1.5x3.2mm_P0.9mm, B.Cu at (76.2, 124.3)
- added U5: AOZ1284PI, Package_SO:SOIC-8-1EP_3.9x4.9mm_P1.27mm_EP2.71x3.7mm, F.Cu at (33.8, 105.4)
- added U6: TL431BIDBZR, Package_TO_SOT_SMD:SOT-23, F.Cu at (47.1, 114.7)
- added U7: TPS61023DRLR, Power_Management_Custom:TPS61023_DRL0006A, F.Cu at (48.2, 111.4)
- added U8: CAT4104V-GT3, Package_SO:SOIC-8_3.9x4.9mm_P1.27mm, F.Cu at (47.0, 105.5)
- added U9: TPD4E05U06QDQARQ1, USB_ESD:antmicro_tpd4e05u06qdqarq1, F.Cu at (35.0, 121.4)
Routing:
- net Net-(U2-GPIO13/USB_D+): track 0.00 -> 2.83 mm
- net Net-(U2-GPIO12/USB_D-): track 0.00 -> 2.73 mm
- net Net-(BT1-+): track 0.00 -> 0.72 mm
Other:
- board size 60 x 40 mm -> 65.9 x 40.6 mm
