File: hardware/gopo.kicad_pcb (KiCad board)
At the start: 4 copper layers, 99.4 x 61 mm, 143 parts, among them J3 TFT032B018, J4 SolderWire-1.5sqmm, J7 USB_C_Receptacle_USB2.0_16P, J8 2-CH UART TO ETH, J9 ENCODER CABLE, Q1 BSS138P, Q2 BSS138P, Q3 SQJB60EP, Q4 BSS138P, Q5 SQJB60EP, Q6 BSS138P, Q7 IRLML6344, Q8 TSM3443CX6, SW1 BOOT / PTS810, SW2 RESET / PTS810, U1 AP33772SDKZ-13-FA02, U10 USBLC6-2SC6, U11 TPS55340PWPR, U12 LM74801-Q1, U13 74LVC1G08, U2 ESP32-C6-MINI-1-H4, U3 INA226, U4 BQ32000, U5 AOZ1284PI, U6 TLV431BQDBZT, Y1 32.768kHz

Commit message: PCB tasarım güncellemeleri
Parts:
- added MECH_ENC: PANEL EC1121S; J9 cable, , F.Cu at (54.3, 112.4)
- C5, C6, C7, D3, D8, D9, J7, R1, R10, R15, R16, R2, R3, R37, R62, R63, TP10, TP9, U10, U2: moved to F.Cu
- moved TP8 144.0 mm to (80.0, 72.0), turned to 0 degrees
- moved TP7 143.9 mm to (77.0, 72.0), turned to 0 degrees
- moved TP6 143.8 mm to (74.0, 72.0), turned to 0 degrees
- moved Q1 109.7 mm to (105.8, 74.0)
- moved Q2 109.7 mm to (110.2, 74.0)
- moved R4 109.7 mm to (105.8, 70.5)
- moved R5 109.7 mm to (105.8, 77.5)
- moved R6 109.7 mm to (110.2, 77.5)
- moved R7 109.7 mm to (110.2, 70.5)
- moved J8 96.4 mm to (102.5, 79.6), turned to 0 degrees
- moved C6 94.0 mm to (71.0, 83.0)
- moved C33 93.5 mm to (114.5, 81.0)
- moved D10 93.0 mm to (124.0, 117.5)
- moved Q4 93.0 mm to (120.0, 122.5)
- moved Q6 93.0 mm to (119.5, 117.5)
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Other:
- outline, holes or cut-outs redrawn

Commit message: 28/09/26
Parts:
- R34, R35, R36: moved to F.Cu
- TP10, TP9: moved to B.Cu
- moved R36 101.5 mm to (69.6, 96.0), turned to 0 degrees
- moved R35 97.9 mm to (67.5, 96.0), turned to 0 degrees
- moved R34 94.3 mm to (65.4, 96.0), turned to 0 degrees
- moved TP1 89.3 mm to (71.5, 101.3)
- moved R11 81.0 mm to (76.5, 103.0)
- moved C3 79.2 mm to (72.5, 107.0)
- moved TP3 78.9 mm to (90.8, 103.6)
- moved TP2 76.7 mm to (82.0, 102.5)
- moved TP4 74.2 mm to (70.0, 125.0)
- moved TH1 74.1 mm to (73.5, 111.0)
- moved Q3 72.1 mm to (78.5, 110.0)
- moved C1 70.9 mm to (73.5, 124.3), turned to 180 degrees
- moved R21 70.7 mm to (75.6, 124.3)
- moved R8 70.5 mm to (77.6, 124.3)
- moved R14 70.4 mm to (80.8, 120.5)
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