File: hardware/powersensing.kicad_sch (KiCad schematic)
At the start: 4 parts, among them U3 INA228

Commit message: usb_pd_controller: VBUS dağıtımını tek sayfada topla (A2)
AP33772S bloğu ile VBUS şönt / PD çıkış anahtarı tek çerçevede birleşti:
USB_VBUS -> TP1 -> R11 şönt -> PD_VBUS_SENSED rayı -> Q4/Q3 -> PD_VOUT,
rayın devamı doğrudan AP74502Q bloğuna gidiyor. ISENP, VCC, PWR_EN->R12
kapı sürüşü ve VOUT geri beslemesi artık gerçek tellerle bağlı.

poweroutput'taki AP74502Q çıkış anahtarı ve powersensing'teki INA228
ölçüm bloğu bu sayfaya taşındı; SW_OUT ve PD_VBUS_SENSED sayfa içi yerel
etiket oldu (global etiketler kaldırıldı). poweroutput yalnızca panel
konnektörlerini tutuyor ve A4'e döndü; powersensing boşaldı.

Bağlantılar isimden bağımsız karşılaştırmayla doğrulandı: kayıp/yeni net
yok, yalnızca sayfa kapsamı değişen 5 net yeniden adlandı
(GATE_DRV, OV_SENSE, SRC_COMMON, PD_VBUS_SENSED, SW_OUT).
ERC değişmedi (0 hata, 2 eski uyarı).

Co-Authored-By: Claude Opus 5 <noreply@anthropic.com>
Parts:
- removed C11: 100nF, Capacitor_SMD:C_0402_1005Metric, symbol Device:C
- removed R27: 10K, Resistor_SMD:R_0402_1005Metric, symbol Device:R
- removed RShunt1: 5mR / 1W, Resistor_SMD:R_2512_6332Metric, symbol Device:R
- removed U3: INA228, Package_SO:TSSOP-10_3x3mm_P0.5mm, symbol Sensor_Energy:INA228
Other:
- note removed: "INA228 CIKIS AKIM / VOLTAJ OLCUMU"
- note removed: "Kelvin: Vin+/Vin- sontun pad uclarindan ayri izle alinir."
