File: hardware/gopo.kicad_sch (KiCad schematic)
At the start: 0 parts

Commit message: usb_pd_controller: tüm güç zincirini tek A3 sayfasında topla
powergeneration (TPS55340 ön-boost + AOZ1284 buck) ve poweroutput (panel
konnektörleri) blokları bu sayfaya taşındı. Sayfa A2'den A3'e indirildi;
bloklar altı slota yeniden çizildi:
  satır 1: PD kontrolcü + VBUS şönt/anahtar | AP74502Q çıkış anahtarı |
           INA228 ölçüm + panel çıkışı (TVS ve boşaltma direnci dahil)
  satır 2: TPS55340 ön-boost | AOZ1284 buck | I2C seviye dönüştürücü

Okunurluk için: buck bloğu iki satıra bölünüp sütun aralıkları 12.7 mm'ye
çıkarıldı, PD kontrolcüde V5V rayı kapı hattının üstüne alındı, INA228 ile
panel konnektörleri tek blokta birleşti, V_PRE artık ön-boost çıkışından
buck girişine gerçek telle gidiyor.

Boş kalan sayfalar silindi: powergeneration, poweroutput, powersensing,
calc_usb_pd_controller, CALC_MCU, CALC_USB_C_INPUT (sayfa sembolleri ve
gopo.kicad_pro kayıtları dahil). Şematik 12 sayfadan 6 sayfaya indi.

Bağlantılar isimden bağımsız karşılaştırmayla doğrulandı: kayıp/yeni net
yok; yalnızca sayfa kapsamı değişen 9 net yeniden adlandı
(/POWER GENERATION/* -> /USB_PD_CONTROLLER/*). ERC değişmedi
(0 hata, 2 eski uyarı), lint temiz.

Co-Authored-By: Claude Opus 5 <noreply@anthropic.com>
Other:
- removed sheet POWER GENERATION
- removed sheet POWER OUTPUT
- removed sheet POWER SENSING
Changed lines of the file:
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@@
-	)
-	(sheet
-		(at 106.68 109.22)
-		(size 40.64 44.45)
-		(exclude_from_sim no)
-		(in_bom yes)
-		(on_board yes)
-		(dnp no)
-		(fields_autoplaced yes)
-		(stroke
-			(width 0.1524)
-			(type solid)
-		)
-		(fill
-			(color 227 90 255 1)
-		)
-		(property "Sheetname" "POWER SENSING"
-			(at 106.68 108.5084 0)
-			(show_name no)
-			(do_not_autoplace no)
-			(effects
-				(font
-					(size 1.27 1.27)
-				)
-				(justify left bottom)
-			)
-		)
-		(property "Sheetfile" "powersensing.kicad_sch"
-			(at 106.68 154.2546 0)
-			(show_name no)
-			(do_not_autoplace no)
-			(effects
-				(font
-					(size 1.27 1.27)
-				)
-				(justify left top)
-			)
-		)
-		(instances
-			(project "gopo"
-				(path "/a43081a6-9aa2-4898-9347-bbcb5849dafd"
-					(page "4")
-				)
-			)
-		)
-	)
-	(sheet
-		(at 38.1 109.22)
-		(size 39.37 43.18)
-		(exclude_from_sim no)
-		(in_bom yes)
-		(on_board yes)
-		(dnp no)
-		(fields_autoplaced yes)
-		(stroke
-			(width 0.1524)
-			(type solid)
-		)
-		(fill
-			(color 227 90 255 1)
-		)
-		(property "Sheetname" "POWER GENERATION"
-			(at 38.1 108.5084 0)
-			(show_name no)
-			(do_not_autoplace no)
-			(effects
-				(font
-					(size 1.27 1.27)
-				)
-				(justify left bottom)
-			)
-		)
-		(property "Sheetfile" "powergeneration.kicad_sch"
-			(at 38.1 152.9846 0)
-			(show_name no)
-			(do_not_autoplace no)
-			(effects
-				(font
-					(size 1.27 1.27)
-				)
-				(justify left top)
-			)
-		)
-		(instances
-			(project "gopo"
-				(path "/a43081a6-9aa2-4898-9347-bbcb5849dafd"
-					(page "5")
-				)
-			)
-		)
 	)
 	(sheet
@@
 				)
 			)
-		)
-	)
-	(sheet
-		(at 191.77 109.22)
-		(size 45.72 43.18)
-		(exclude_from_sim no)
-		(in_bom yes)
-		(on_board yes)
-		(dnp no)
-		(fields_autoplaced yes)
-		(stroke
-			(width 0.1524)
-			(type solid)
-		)
-		(fill
-			(color 227 90 255 1)
-		)
-		(property "Sheetname" "POWER OUTPUT"
-			(at 191.77 108.5084 0)
-			(show_name no)
-			(do_not_autoplace no)
-			(effects
-				(font
-					(size 1.27 1.27)
-				)
-				(justify left bottom)
-			)
-		)
-		(property "Sheetfile" "poweroutput.kicad_sch"
-			(at 191.77 152.9846 0)
-			(show_name no)
-			(do_not_autoplace no)
-			(effects
-				(font
-					(size 1.27 1.27)
-				)
-				(justify left top)
-			)
-		)
-		(instances
-			(project "gopo"
-				(path "/a43081a6-9aa2-4898-9347-bbcb5849dafd"
-					(page "6")
-				)
-			)
