File: hardware/usb_pd_controller.kicad_sch (KiCad schematic)
At the start: 28 parts, among them Q1 BSS138, Q2 BSS138, Q3 IRF7855TRPBF, Q4 IRF7855TRPBF, U1 AP33772SDKZ-13-FA02

Commit message: usb_pd_controller: VBUS dağıtımını tek sayfada topla (A2)
AP33772S bloğu ile VBUS şönt / PD çıkış anahtarı tek çerçevede birleşti:
USB_VBUS -> TP1 -> R11 şönt -> PD_VBUS_SENSED rayı -> Q4/Q3 -> PD_VOUT,
rayın devamı doğrudan AP74502Q bloğuna gidiyor. ISENP, VCC, PWR_EN->R12
kapı sürüşü ve VOUT geri beslemesi artık gerçek tellerle bağlı.

poweroutput'taki AP74502Q çıkış anahtarı ve powersensing'teki INA228
ölçüm bloğu bu sayfaya taşındı; SW_OUT ve PD_VBUS_SENSED sayfa içi yerel
etiket oldu (global etiketler kaldırıldı). poweroutput yalnızca panel
konnektörlerini tutuyor ve A4'e döndü; powersensing boşaldı.

Bağlantılar isimden bağımsız karşılaştırmayla doğrulandı: kayıp/yeni net
yok, yalnızca sayfa kapsamı değişen 5 net yeniden adlandı
(GATE_DRV, OV_SENSE, SRC_COMMON, PD_VBUS_SENSED, SW_OUT).
ERC değişmedi (0 hata, 2 eski uyarı).

Co-Authored-By: Claude Opus 5 <noreply@anthropic.com>
Parts:
- added C11: 100nF, Capacitor_SMD:C_0402_1005Metric, symbol Device:C
- added C30: 22nF 50V, Capacitor_SMD:C_0402_1005Metric, symbol Device:C
- added C31: 220nF 25V, Capacitor_SMD:C_0402_1005Metric, symbol Device:C
- added C32: 100nF 50V, Capacitor_SMD:C_0402_1005Metric, symbol Device:C
- added D6: BZT52C12, Diode_SMD:D_SOD-123, symbol Device:D_Zener
- added D7: SMBJ30A, Diode_SMD:D_SMB, symbol Power_Path_Custom:SMBJ30A
- added Q5, Q6: 60V 4mR TBD, symbol Transistor_FET:Q_NMOS_GSD
- added R27: 10K, Resistor_SMD:R_0402_1005Metric, symbol Device:R
- added R54: 1kR, Resistor_SMD:R_0402_1005Metric, symbol Device:R_Small_US
- added R55: 232kR, Resistor_SMD:R_0402_1005Metric, symbol Device:R_Small_US
- added R56, R57: 10kR, Resistor_SMD:R_0402_1005Metric, symbol Device:R_Small_US
- added R58: 100kR, Resistor_SMD:R_0402_1005Metric, symbol Device:R_Small_US
- added R59: 10kR 0.25W, Resistor_SMD:R_0402_1005Metric, symbol Device:R_Small_US
- added RShunt1: 5mR / 1W, Resistor_SMD:R_2512_6332Metric, symbol Device:R
- added U12: AP74502Q, Package_TO_SOT_SMD:TSOT-23-8_HandSoldering, symbol Power_Path_Custom:AP74502Q
- added U3: INA228, Package_SO:TSSOP-10_3x3mm_P0.5mm, symbol Sensor_Energy:INA228
Connections:
- net +3.3V: now also C11.1, R27.1, U3.6 (VS)
- net GND: now also C11.2, C30.2, C32.2, D7.2 (A2), R56.2, R58.2, R59.2, U12.2 (GND), U3.1 (A1), U3.2 (A0), U3.7 (GND)
- net PD_I2C_SCL_3V3: now also U3.5 (SCL)
- net PD_I2C_SDA_3V3: now also U3.4 (SDA)
- net PD_VBUS_SENSED: now also Q5.3 (D), R55.1
- new net: C31.2, U12.4 (VCAP)
- new net: C30.1, R54.2
- new net GATE_DRV: D6.1 (K), Q5.1 (G), Q6.1 (G), R54.1, U12.6 (GATE)
- new net INA_ALERT: R27.2, R57.2, R58.1, U12.1 (EN/UVLO), U3.3 (~{Alert})
- new net OUT_EN: R57.1
- new net OUT_POS: D7.1 (A1), R59.1, RShunt1.2, U3.8 (Vbus), U3.9 (Vin-)
- new net OV_SENSE: R55.2, R56.1, U12.7 (OV)
- new net SRC_COMMON: D6.2 (A), Q5.2 (S), Q6.2 (S), U12.8 (SRC)
- new net SW_OUT: Q6.3 (D), RShunt1.1, U3.10 (Vin+)
- new net V_PRE: C31.1, C32.1, U12.5 (VS)
- no-connect marks 4 -> 5
Other:
- note added: "AP33772S PD KONTROLCU + VBUS SONT / ANAHTAR"
- note added: "AP74502Q CIKIS ANAHTARI"
- note added: "INA228 CIKIS AKIM / VOLTAJ OLCUMU"
- note added: "Kelvin: Vin+/Vin- sontun pad uclarindan ayri izle alinir."
- note removed: "AP33772S USB PD KONTROLCU"
- note removed: "VBUS SONT + PD CIKIS ANAHTARI"
- moved on the sheet: C1, C2, C3, C4, C8, D1, Q1, Q2, Q3, Q4, R11, R12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

Commit message: usb_pd_controller: tüm güç zincirini tek A3 sayfasında topla
powergeneration (TPS55340 ön-boost + AOZ1284 buck) ve poweroutput (panel
konnektörleri) blokları bu sayfaya taşındı. Sayfa A2'den A3'e indirildi;
bloklar altı slota yeniden çizildi:
  satır 1: PD kontrolcü + VBUS şönt/anahtar | AP74502Q çıkış anahtarı |
           INA228 ölçüm + panel çıkışı (TVS ve boşaltma direnci dahil)
  satır 2: TPS55340 ön-boost | AOZ1284 buck | I2C seviye dönüştürücü

Okunurluk için: buck bloğu iki satıra bölünüp sütun aralıkları 12.7 mm'ye
çıkarıldı, PD kontrolcüde V5V rayı kapı hattının üstüne alındı, INA228 ile
panel konnektörleri tek blokta birleşti, V_PRE artık ön-boost çıkışından
buck girişine gerçek telle gidiyor.

Boş kalan sayfalar silindi: powergeneration, poweroutput, powersensing,
calc_usb_pd_controller, CALC_MCU, CALC_USB_C_INPUT (sayfa sembolleri ve
gopo.kicad_pro kayıtları dahil). Şematik 12 sayfadan 6 sayfaya indi.

Bağlantılar isimden bağımsız karşılaştırmayla doğrulandı: kayıp/yeni net
yok; yalnızca sayfa kapsamı değişen 9 net yeniden adlandı
(/POWER GENERATION/* -> /USB_PD_CONTROLLER/*). ERC değişmedi
(0 hata, 2 eski uyarı), lint temiz.

Co-Authored-By: Claude Opus 5 <noreply@anthropic.com>
Parts:
- added C12, C13: 10uF, Capacitor_SMD:C_1210_3225Metric, symbol Device:C
- added C14, C24: 100nF, Capacitor_SMD:C_0402_1005Metric, symbol Device:C
- added C15: 47uF, Capacitor_SMD:C_0402_1005Metric, symbol Device:C
- added C16: 47uF, Capacitor_SMD:C_1210_3225Metric, symbol Device:C
- added C17: 100nF / 16V, Capacitor_SMD:C_0402_1005Metric, symbol Device:C
- added C18: 10nF, Capacitor_SMD:C_0402_1005Metric, symbol Device:C
- added C19: 18nF / 16V, Capacitor_SMD:C_0402_1005Metric, symbol Device:C
- added C23: 47nF, Capacitor_SMD:C_0402_1005Metric, symbol Device:C
- added C25, C27, C28: 10uF 50V, Capacitor_SMD:C_1210_3225Metric, symbol Device:C
- added C26: 100nF 50V, Capacitor_SMD:C_0402_1005Metric, symbol Device:C
- added C29: 47uF 50V, Capacitor_SMD:C_1210_3225Metric, symbol Device:C
- added D2: SS2060FL_R1_00001, Diode_SMD:D_SOD-123F, symbol Device:D_Schottky
- added D4: SS34 TBD, Diode_SMD:D_SMA, symbol Device:D_Schottky
- added D5: BAT54, Diode_SMD:D_SOD-123, symbol Device:D_Schottky
- added J4: DG142R-5.08-02P-14-00AH, DG142R-5.08-02P-14-00AH:DG142R-5.08-02P-14-00AH, symbol DG142R-5.08-02P-14-00AH:DG142R-5.08-02P-14-00AH
- added J5: 108-0902-001, Power_Output_Custom:Cinch_108-0902-001_Panel, symbol Connector_Generic:Conn_01x01
- added J6: 108-0903-001, Power_Output_Custom:Cinch_108-0903-001_Panel, symbol Connector_Generic:Conn_01x01
- added L1: SRI0704-220M, Inductor_SMD:L_7.3x7.3_H4.5, symbol Device:L
- added L3: 6.8uH TBD, Inductor_SMD:L_1210_3225Metric, symbol Device:L
- added R38: 100kR 1%, Resistor_SMD:R_0402_1005Metric, symbol Device:R_Small_US
- added R39: 10kR 0.1%, Resistor_SMD:R_0402_1005Metric, symbol Device:R_Small_US
- added R40: 3.20kR 0.1%, Resistor_SMD:R_0402_1005Metric, symbol Device:R_Small_US
- added R41: 12.7kR 1%, Resistor_SMD:R_0402_1005Metric, symbol Device:R_Small_US
- added R42, R53: 100kR, Resistor_SMD:R_0402_1005Metric, symbol Device:R_Small_US
- added R43: 1kR / 2W, Resistor_SMD:R_2512_6332Metric, symbol Device:R_Small_US
- added R47: 78.7kR, Resistor_SMD:R_0402_1005Metric, symbol Device:R_Small_US
- added R48: 30.1kR, Resistor_SMD:R_0402_1005Metric, symbol Device:R_Small_US
- added R49: 9.76kR, Resistor_SMD:R_0402_1005Metric, symbol Device:R_Small_US
- added R50: 820R, Resistor_SMD:R_0402_1005Metric, symbol Device:R_Small_US
- added R51: 1kR, Resistor_SMD:R_0402_1005Metric, symbol Device:R_Small_US
- added R52: 2kR, Resistor_SMD:R_0402_1005Metric, symbol Device:R_Small_US
- added U11: TPS55340PWPR, Package_SO:Texas_HTSSOP-14-1EP_4.4x5mm_P0.65mm_EP3.4x5mm_Mask3.155x3.255mm_ThermalVias, symbol Power_Path_Custom:TPS55340PWPR
- added U5: AOZ1284PI, Package_SO:SOIC-8-1EP_3.9x4.9mm_P1.27mm_EP2.71x3.7mm, symbol Regulator_Switching:AOZ1284PI
- added U6: TL431BIDBZR, Package_TO_SOT_SMD:SOT-23, symbol Reference_Voltage:TL431DBZ
Connections:
- net +3.3V: now also C15.1, C16.1, L1.2, R39.1, R50.1
- net GND: now also C12.2, C13.2, C14.2, C15.2, C16.2, C18.2, C19.2, C23.2, C24.2, C25.2, C26.2, C27.2, C28.2, C29.2, D2.2 (A), J4.2 (GND), J6.1 (Pin_1), R38.2, R40.2, R42.2, R47.2, R49.2, R51.2, U11.11 (NC), U11.12 (PGND), U11.13 (PGND), U11.14 (PGND), U11.15 (PowerPAD), U11.6 (SYNC), U11.7 (AGND), U5.3 (GND), U6.3 (A)
- net OUT_POS: now also J4.1 (OUT_POS), J5.1 (Pin_1)
- net PD_VOUT: now also C25.1, C26.1, C29.1, L3.2, R53.1, U11.3 (VIN)
- net V_PRE: now also C12.1, C13.1, C14.1, C27.1, C28.1, D4.1 (K), R43.1, R48.1, U5.9 (VIN)
- new net: C19.1, R41.2
- new net: C23.1, U11.5 (SS)
- new net: R47.1, U11.10 (FREQ)
- new net: R53.2, U11.4 (EN)
- new net: R52.1, U11.8 (COMP)
- new net: C24.1, R52.2
- new net: C17.1, U5.2 (BST)
- new net BOOST_FB: D5.2 (A), R48.2, R49.1, U11.9 (FB)
- new net BOOST_SW: D4.2 (A), L3.1, U11.1 (SW), U11.2 (SW)
- new net COMP_NODE: R41.1, U5.5 (COMP)
- new net EN_CTRL: R42.1, R43.2, U5.8 (EN), U6.1 (K), U6.2 (REF)
- new net FB_3V3: R39.2, R40.1, U5.6 (FB)
- new net FSW_SET: R38.1, U5.4 (FSW)
- new net LX_SW: C17.2, D2.1 (K), L1.1, U5.1 (LX)
- new net SS_RAMP: C18.1, U5.7 (SS)
- new net V_CL: D5.1 (K), R50.2, R51.1
Other:
- removed sheet CALC_USB_PD_CONTROLLER
- note added: "AOZ1284 3.3V BUCK"
- note added: "Cin: 50V X7R; effective bank >=10uF @28V"
- note added: "Cout: 10V X7R; effective bank >=44uF @3.3V"
- note added: "INA228 OLCUM + PANEL CIKISI"
- note added: "INTERNAL 3.3V BUCK — 5..28V INPUT / 1A DESIGN LOAD"
- note added: "L/D exact MPN and footprints require selection. L: Isat >=2A normal load, Irms >=1.5A. Cout effective >=44uF; check DC-bias curves."
- note added: "PANEL: J5 red (+), J6 black (GND). J4.1 = OUT_POS; J4.2 = GND. Panel-mount jacks: wire to PCB terminal."
- note added: "TPS55340 PRE-BOOST"
- note added: "VIN = EXPOSED PAD 9: V_PRE, NOT GND. EN: 2.495V shunt bias; R43 dissipation 0.65W at 28V. COMP: Rc=12.7k, Cc=18nF; fc about 8.5..10kHz at Cout_eff=44uF. RF=100k: table 500kHz; equation 476.19kHz. Verify on prototype."
- note added: "V_PRE = 5.02 V (pass-through > 5.5 V)"
- note removed: "INA228 CIKIS AKIM / VOLTAJ OLCUMU"
- moved on the sheet: C1, C11, C2, C3, C30, C31, C32, C4, C8, D1, D6, D7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

Commit message: hardware: komponent alanlarını standarda oturt, yalnız Value+Reference göster
134 komponentin alan seti design_decisions/standards/komponent-field-standardi.csv
uyarınca yeniden kuruldu (3.144 alan). Her komponent grup koduna atandı ve ALL +
gruba özel alanlar standarttaki sırayla yazıldı; CSV'de koşullu işaretli alanlar
(Sadece Zener / Sadece ADC / Sadece RTC) yalnız ilgili parçaya kondu.

Eski alan adları standarda birleşti: Manufacturer Part Number ve DisplayMPN ->
MPN, Voltage -> VoltageRating, Field5 -> DesignNote / TerminationStyle,
Supplier + Battery -> SelectionNote / DesignNote. Sim.* alanları korundu.

Value IEC 60062 koduna çevrildi (10 kΩ/4,7k/100K/10kR karışıktı -> 10k/4k7/100k).
Value'dan çıkan gerilim, güç, tolerans ve dielektrik kendi alanlarına taşındı.
L1 ve D2'de Value MPN'di; parametrik değere çevrilip sipariş kodu MPN'e alındı.

Görünürlük tek kurala indi: yalnız Reference + Value. Description 119 sembolde
açıktı, kapandı. Güç sembolleri depo kuralına oturdu (Reference gizli, GND ve
PWR_FLAG değeri gizli, +3.3V görünür).

Parça verisi gerektiren 1.755 alan TBD bırakıldı; yalnız depodan (footprint,
lib_id, BOM_PRELIMINARY, tasarım notları) doğrulanabilen değerler yazıldı,
MPN veya datasheet parametresi uydurulmadı.

Okunabilirlik: C3 değeri PD_VBUS_SENSED telinin üstündeydi, TP5 referansı
PD_GATE etiketiyle çakışıyordu; ikisinin de yalnız metin konumu kaydırıldı.

gopo.kicad_pro'ya 10 çekirdek alanın Field Name Templates kaydı eklendi.

Bu commit ayrıca KiCad 10'un kendi kaydını taşır: güç sembollerinden
(fields_autoplaced no) düştü ve C4/TP4 elle boş alana taşındı.

Doğrulama: netlist farkı YOK, ERC 2 uyarı (değişmedi), lint 6/1/0/0 (değişmedi),
field_geometry farkı yalnız C3 ve TP5.

Co-Authored-By: Claude Opus 5 <noreply@anthropic.com>
Parts:
- C1, C2: value 100 nF -> 100n; AssemblyNote (none) -> TBD; Category (none) -> Capacitors; DesignNote (none) -> TBD; Dielectric (none) -> TBD; EffectiveCapacitance (none) -> TBD; Height (none) -> TBD; Lifecycle (none) -> TBD; MPN (none) -> TBD; Manufacturer (none) -> TBD; MountingType (none) -> Surface Mount; OperatingTemp (none) -> TBD; Package (none) -> 0402 (1005 Metric); RoHS (none) -> TBD; SelectionNote (none) -> TBD; Subcategory (none) -> Ceramic Capacitors; Tolerance (none) -> TBD; VoltageRating (none) -> TBD
- C11, C24: value 100nF -> 100n; AssemblyNote (none) -> TBD; Category (none) -> Capacitors; DesignNote (none) -> TBD; Dielectric (none) -> TBD; EffectiveCapacitance (none) -> TBD; Height (none) -> TBD; Lifecycle (none) -> TBD; MPN (none) -> TBD; Manufacturer (none) -> TBD; MountingType (none) -> Surface Mount; OperatingTemp (none) -> TBD; Package (none) -> 0402 (1005 Metric); RoHS (none) -> TBD; SelectionNote (none) -> TBD; Subcategory (none) -> Ceramic Capacitors; Tolerance (none) -> TBD; VoltageRating (none) -> TBD
- C12, C13: value 10uF -> 10u; AssemblyNote (none) -> TBD; Category (none) -> Capacitors; DesignNote X7R; C12+C13 effective capacitance >=10uF at 28V; verify ac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 -> X7R; C12+C13 efektif kapasite 28V'ta >=10uF olmali, MPN dog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; Dielectric (none) -> X7R; EffectiveCapacitance (none) -> TBD; Height (none) -> TBD; Lifecycle (none) -> TBD; MPN (none) -> TBD; Manufacturer (none) -> TBD; MountingType (none) -> Surface Mount; OperatingTemp (none) -> TBD; Package (none) -> 1210 (3225 Metric); RoHS (none) -> TBD; SelectionNote (none) -> TBD; Subcategory (none) -> Ceramic Capacitors; Tolerance (none) -> TBD; Voltage 50V -> (none); VoltageRating (none) -> 50V
- C14: value 100nF -> 100n; AssemblyNote (none) -> TBD; Category (none) -> Capacitors; DesignNote X7R; C12+C13 effective capacitance >=10uF at 28V; verify ac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 -> X7R.; Dielectric (none) -> X7R; EffectiveCapacitance (none) -> TBD; Height (none) -> TBD; Lifecycle (none) -> TBD; MPN (none) -> TBD; Manufacturer (none) -> TBD; MountingType (none) -> Surface Mount; OperatingTemp (none) -> TBD; Package (none) -> 0402 (1005 Metric); RoHS (none) -> TBD; SelectionNote (none) -> TBD; Subcategory (none) -> Ceramic Capacitors; Tolerance (none) -> TBD; Voltage 50V -> (none); VoltageRating (none) -> 50V
- C15: value 47uF -> 47u; AssemblyNote (none) -> TBD; Category (none) -> Capacitors; DesignNote X7R; bank effective Cout >=44uF at 3.3V. Confirm exact MPN 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 -> X7R; banka efektif Cout 3.3V'ta >=44uF olmali, MPN dogrulan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; Dielectric (none) -> X7R; EffectiveCapacitance (none) -> TBD; Height (none) -> TBD; Lifecycle (none) -> TBD; MPN (none) -> TBD; Manufacturer (none) -> TBD; MountingType (none) -> Surface Mount; OperatingTemp (none) -> TBD; Package (none) -> 0402 (1005 Metric); RoHS (none) -> TBD; SelectionNote (none) -> TBD; Subcategory (none) -> Ceramic Capacitors; Tolerance (none) -> TBD; Voltage 10V -> (none); VoltageRating (none) -> 10V
- C16: value 47uF -> 47u; AssemblyNote (none) -> TBD; Category (none) -> Capacitors; DesignNote X7R; bank effective Cout >=44uF at 3.3V. Confirm exact MPN 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 -> X7R; banka efektif Cout 3.3V'ta >=44uF olmali, MPN dogrulan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; Dielectric (none) -> X7R; EffectiveCapacitance (none) -> TBD; Height (none) -> TBD; Lifecycle (none) -> TBD; MPN (none) -> TBD; Manufacturer (none) -> TBD; MountingType (none) -> Surface Mount; OperatingTemp (none) -> TBD; Package (none) -> 1210 (3225 Metric); RoHS (none) -> TBD; SelectionNote (none) -> TBD; Subcategory (none) -> Ceramic Capacitors; Tolerance (none) -> TBD; Voltage 10V -> (none); VoltageRating (none) -> 10V
- C17: value 100nF / 16V -> 100n; AssemblyNote (none) -> TBD; Category (none) -> Capacitors; DesignNote (none) -> TBD; Dielectric (none) -> TBD; EffectiveCapacitance (none) -> TBD; Height (none) -> TBD; Lifecycle (none) -> TBD; MPN (none) -> TBD; Manufacturer (none) -> TBD; MountingType (none) -> Surface Mount; OperatingTemp (none) -> TBD; Package (none) -> 0402 (1005 Metric); RoHS (none) -> TBD; SelectionNote (none) -> TBD; Subcategory (none) -> Ceramic Capacitors; Tolerance (none) -> TBD; Voltage 16V -> (none); VoltageRating (none) -> 16V
- C18: value 10nF -> 10n; AssemblyNote (none) -> TBD; Category (none) -> Capacitors; DesignNote (none) -> TBD; Dielectric (none) -> TBD; EffectiveCapacitance (none) -> TBD; Height (none) -> TBD; Lifecycle (none) -> TBD; MPN (none) -> TBD; Manufacturer (none) -> TBD; MountingType (none) -> Surface Mount; OperatingTemp (none) -> TBD; Package (none) -> 0402 (1005 Metric); RoHS (none) -> TBD; SelectionNote (none) -> TBD; Subcategory (none) -> Ceramic Capacitors; Tolerance (none) -> TBD; Voltage 10V -> (none); VoltageRating (none) -> 10V
- C19: value 18nF / 16V -> 18n; AssemblyNote (none) -> TBD; Category (none) -> Capacitors; DesignNote (none) -> TBD; Dielectric (none) -> TBD; EffectiveCapacitance (none) -> TBD; Height (none) -> TBD; Lifecycle (none) -> TBD; MPN (none) -> TBD; Manufacturer (none) -> TBD; MountingType (none) -> Surface Mount; OperatingTemp (none) -> TBD; Package (none) -> 0402 (1005 Metric); RoHS (none) -> TBD; SelectionNote (none) -> TBD; Subcategory (none) -> Ceramic Capacitors; Tolerance (none) -> TBD; VoltageRating (none) -> 16V
- C23: value 47nF -> 47n; AssemblyNote (none) -> TBD; Category (none) -> Capacitors; DesignNote (none) -> TBD; Dielectric (none) -> TBD; EffectiveCapacitance (none) -> TBD; Height (none) -> TBD; Lifecycle (none) -> TBD; MPN (none) -> TBD; Manufacturer (none) -> TBD; MountingType (none) -> Surface Mount; OperatingTemp (none) -> TBD; Package (none) -> 0402 (1005 Metric); RoHS (none) -> TBD; SelectionNote (none) -> TBD; Subcategory (none) -> Ceramic Capacitors; Tolerance (none) -> TBD; VoltageRating (none) -> TBD
- C25, C27, C28: value 10uF 50V -> 10u; AssemblyNote (none) -> TBD; Category (none) -> Capacitors; DesignNote (none) -> TBD; Dielectric (none) -> TBD; EffectiveCapacitance (none) -> TBD; Height (none) -> TBD; Lifecycle (none) -> TBD; MPN (none) -> TBD; Manufacturer (none) -> TBD; MountingType (none) -> Surface Mount; OperatingTemp (none) -> TBD; Package (none) -> 1210 (3225 Metric); RoHS (none) -> TBD; SelectionNote (none) -> TBD; Subcategory (none) -> Ceramic Capacitors; Tolerance (none) -> TBD; VoltageRating (none) -> 50V
- C26, C32: value 100nF 50V -> 100n; AssemblyNote (none) -> TBD; Category (none) -> Capacitors; DesignNote (none) -> TBD; Dielectric (none) -> TBD; EffectiveCapacitance (none) -> TBD; Height (none) -> TBD; Lifecycle (none) -> TBD; MPN (none) -> TBD; Manufacturer (none) -> TBD; MountingType (none) -> Surface Mount; OperatingTemp (none) -> TBD; Package (none) -> 0402 (1005 Metric); RoHS (none) -> TBD; SelectionNote (none) -> TBD; Subcategory (none) -> Ceramic Capacitors; Tolerance (none) -> TBD; VoltageRating (none) -> 50V
- C29: value 47uF 50V -> 47u; AssemblyNote (none) -> TBD; Category (none) -> Capacitors; DesignNote (none) -> TBD; Dielectric (none) -> TBD; EffectiveCapacitance (none) -> TBD; Height (none) -> TBD; Lifecycle (none) -> TBD; MPN (none) -> TBD; Manufacturer (none) -> TBD; MountingType (none) -> Surface Mount; OperatingTemp (none) -> TBD; Package (none) -> 1210 (3225 Metric); RoHS (none) -> TBD; SelectionNote (none) -> TBD; Subcategory (none) -> Ceramic Capacitors; Tolerance (none) -> TBD; VoltageRating (none) -> 50V
- C3: value 2.2uF / 50V X7R -> 2u2; AssemblyNote (none) -> TBD; Category (none) -> Capacitors; DesignNote (none) -> TBD; Dielectric (none) -> X7R; EffectiveCapacitance (none) -> TBD; Height (none) -> TBD; Lifecycle (none) -> TBD; MPN (none) -> TBD; Manufacturer (none) -> TBD; MountingType (none) -> Surface Mount; OperatingTemp (none) -> TBD; Package (none) -> 0805 (2012 Metric); RoHS (none) -> TBD; SelectionNote (none) -> TBD; Subcategory (none) -> Ceramic Capacitors; Tolerance (none) -> TBD; VoltageRating (none) -> 50V
- C30: value 22nF 50V -> 22n; AssemblyNote (none) -> TBD; Category (none) -> Capacitors; DesignNote (none) -> TBD; Dielectric (none) -> TBD; EffectiveCapacitance (none) -> TBD; Height (none) -> TBD; Lifecycle (none) -> TBD; MPN (none) -> TBD; Manufacturer (none) -> TBD; MountingType (none) -> Surface Mount; OperatingTemp (none) -> TBD; Package (none) -> 0402 (1005 Metric); RoHS (none) -> TBD; SelectionNote (none) -> TBD; Subcategory (none) -> Ceramic Capacitors; Tolerance (none) -> TBD; VoltageRating (none) -> 50V
- C31: value 220nF 25V -> 220n; AssemblyNote (none) -> TBD; Category (none) -> Capacitors; DesignNote (none) -> TBD; Dielectric (none) -> TBD; EffectiveCapacitance (none) -> TBD; Height (none) -> TBD; Lifecycle (none) -> TBD; MPN (none) -> TBD; Manufacturer (none) -> TBD; MountingType (none) -> Surface Mount; OperatingTemp (none) -> TBD; Package (none) -> 0402 (1005 Metric); RoHS (none) -> TBD; SelectionNote (none) -> TBD; Subcategory (none) -> Ceramic Capacitors; Tolerance (none) -> TBD; VoltageRating (none) -> 25V
- C4: value 1uF / 10V -> 1u0; AssemblyNote (none) -> TBD; Category (none) -> Capacitors; DesignNote (none) -> TBD; Dielectric (none) -> TBD; EffectiveCapacitance (none) -> TBD; Height (none) -> TBD; Lifecycle (none) -> TBD; MPN (none) -> TBD; Manufacturer (none) -> TBD; MountingType (none) -> Surface Mount; OperatingTemp (none) -> TBD; Package (none) -> 0402 (1005 Metric); RoHS (none) -> TBD; SelectionNote (none) -> TBD; Subcategory (none) -> Ceramic Capacitors; Tolerance (none) -> TBD; VoltageRating (none) -> 10V
- C8: value 10uF / 50V -> 10u; AssemblyNote (none) -> TBD; Category (none) -> Capacitors; DesignNote (none) -> TBD; Dielectric (none) -> TBD; EffectiveCapacitance (none) -> TBD; Height (none) -> TBD; Lifecycle (none) -> TBD; MPN (none) -> TBD; Manufacturer (none) -> TBD; MountingType (none) -> Surface Mount; OperatingTemp (none) -> TBD; Package (none) -> 0402 (1005 Metric); RoHS (none) -> TBD; SelectionNote (none) -> TBD; Subcategory (none) -> Ceramic Capacitors; Tolerance (none) -> TBD; VoltageRating (none) -> 50V
- D1: AssemblyNote (none) -> TBD; Category (none) -> Optoelectronics; Color (none) -> TBD; DesignNote (none) -> TBD; ForwardCurrent (none) -> TBD; ForwardVoltage (none) -> TBD; Height (none) -> TBD; LensType (none) -> TBD; Lifecycle (none) -> TBD; LuminousIntensity (none) -> TBD; MPN (none) -> TBD; Manufacturer (none) -> TBD; MountingType (none) -> Surface Mount; OperatingTemp (none) -> TBD; Package (none) -> 0402 (1005 Metric); RoHS (none) -> TBD; SelectionNote (none) -> TBD; Subcategory (none) -> LED Indication - Discrete; ViewingAngle (none) -> TBD; Wavelength (none) -> TBD
- D2: value SS2060FL_R1_00001 -> SS2060FL; AssemblyNote (none) -> TBD; Category (none) -> Discrete Semiconductor Products; DesignNote PANJIT 60V 2A Schottky, SOD-123FL; cathode LX, anode GND; O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 -> Katot LX, anot GND. Tedarik: Ozdisan.; DiodeType (none) -> Schottky; ForwardCurrent (none) -> 2A; ForwardVoltage (none) -> TBD; Height (none) -> TBD; Lifecycle (none) -> TBD; MountingType (none) -> Surface Mount; OperatingTemp (none) -> TBD; Package (none) -> SOD-123F; ReverseCurrent (none) -> TBD; ReverseVoltage (none) -> 60V; RoHS (none) -> TBD; SelectionNote (none) -> TBD; Subcategory (none) -> Diodes
- D4: AssemblyNote (none) -> TBD; Category (none) -> Discrete Semiconductor Products; DesignNote (none) -> SS34 hedefi; kesin MPN secilmedi.; DiodeType (none) -> Schottky; ForwardCurrent (none) -> TBD; ForwardVoltage (none) -> TBD; Height (none) -> TBD; Lifecycle (none) -> TBD; MPN (none) -> TBD; Manufacturer (none) -> TBD; MountingType (none) -> Surface Mount; OperatingTemp (none) -> TBD; Package (none) -> SMA (DO-214AC); ReverseCurrent (none) -> TBD; ReverseVoltage (none) -> TBD; RoHS (none) -> TBD; SelectionNote (none) -> TBD; Subcategory (none) -> Diodes
- D5: AssemblyNote (none) -> TBD; Category (none) -> Discrete Semiconductor Products; DesignNote (none) -> TBD; DiodeType (none) -> Schottky; ForwardCurrent (none) -> TBD; ForwardVoltage (none) -> TBD; Height (none) -> TBD; Lifecycle (none) -> TBD; MPN (none) -> BAT54; Manufacturer (none) -> TBD; MountingType (none) -> Surface Mount; OperatingTemp (none) -> TBD; Package (none) -> SOD-123; ReverseCurrent (none) -> TBD; ReverseVoltage (none) -> TBD; RoHS (none) -> TBD; SelectionNote (none) -> TBD; Subcategory (none) -> Diodes
- D6: AssemblyNote (none) -> TBD; Category (none) -> Discrete Semiconductor Products; DesignNote (none) -> TBD; DiodeType (none) -> Zener; ForwardCurrent (none) -> TBD; ForwardVoltage (none) -> TBD; Height (none) -> TBD; Lifecycle (none) -> TBD; MPN (none) -> BZT52C12; Manufacturer (none) -> TBD; MountingType (none) -> Surface Mount; OperatingTemp (none) -> TBD; Package (none) -> SOD-123; PowerDissipation (none) -> TBD; ReverseCurrent (none) -> TBD; ReverseRecoveryTime (none) -> TBD; ReverseVoltage (none) -> TBD; RoHS (none) -> TBD; SelectionNote (none) -> TBD; Subcategory (none) -> Diodes; TestCurrent (none) -> TBD; ZenerTolerance (none) -> TBD; ZenerVoltage (none) -> 12V
- D7: AssemblyNote (none) -> TBD; BreakdownVoltage (none) -> TBD; Capacitance (none) -> TBD; Category (none) -> Circuit Protection; ChannelCount (none) -> 1; ClampingVoltage (none) -> TBD; DesignNote (none) -> TBD; Height (none) -> TBD; Lifecycle (none) -> TBD; MPN (none) -> SMBJ30A; Manufacturer (none) -> TBD; MountingType (none) -> Surface Mount; OperatingTemp (none) -> TBD; Package (none) -> SMB (DO-214AA); PeakPulseCurrent (none) -> TBD; Polarity (none) -> Unidirectional; RoHS (none) -> TBD; SelectionNote (none) -> TBD; StandoffVoltage (none) -> 30V; Subcategory (none) -> TVS Diodes
- J4: AssemblyNote (none) -> TBD; Category (none) -> Connectors, Interconnects; ConnectorType (none) -> Terminal Block; ContactPlating (none) -> TBD; CurrentRating (none) -> TBD; DesignNote (none) -> 2 kutuplu 5.08 mm klemens; cikis terminali.; Height (none) -> TBD; Lifecycle (none) -> TBD; MatingCycles (none) -> TBD; MountingType (none) -> Through Hole; OperatingTemp (none) -> TBD; Orientation (none) -> TBD; Package (none) -> 5.08mm 2-pos THT; Pitch (none) -> 5.08mm; PositionCount (none) -> 2; RoHS (none) -> TBD; RowCount (none) -> 1; SelectionNote (none) -> TBD; Series (none) -> TBD; Shielding (none) -> TBD; Subcategory (none) -> Terminal Blocks; TorqueRating (none) -> TBD; VoltageRating (none) -> TBD; WireGauge (none) -> TBD; WireTermination (none) -> TBD
- J5, J6: Category (none) -> Connectors, Interconnects; ConnectorType (none) -> Terminal; ContactPlating (none) -> TBD; CurrentRating (none) -> TBD; DesignNote (none) -> PANEL MOUNT; J4'e kablo ile gider, kart uzerinde yalniz mek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; Height (none) -> TBD; Lifecycle (none) -> TBD; MatingCycles (none) -> TBD; MountingType (none) -> Mechanical; OperatingTemp (none) -> TBD; Orientation (none) -> TBD; Package (none) -> Panel Mount Binding Post; Pitch (none) -> TBD; PositionCount (none) -> 1; RoHS (none) -> TBD; RowCount (none) -> 1; SelectionNote (none) -> TBD; Series (none) -> TBD; Shielding (none) -> TBD; Subcategory (none) -> -; VoltageRating (none) -> TBD
- L1: value SRI0704-220M -> 22u; AssemblyNote (none) -> TBD; Category (none) -> Inductors, Coils, Chokes; CurrentRMS (none) -> 1.95A; CurrentSaturation (none) -> 1.95A (L -17%, 18.2uH); DCR (none) -> 110mOhm; DesignNote CORE MASTER 22uH, 1.95A rated, 0.11ohm max; 18.2uH at 1.95A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 -> 22uH, 1.95A, 0.11ohm max; 1.95A'de 18.2uH (L -17%).; Height (none) -> TBD; Lifecycle (none) -> TBD; MountingType (none) -> Surface Mount; OperatingTemp (none) -> TBD; Package (none) -> 7.3x7.3x4.5mm; RoHS (none) -> TBD; SRF (none) -> TBD; SelectionNote (none) -> TBD; Shielding (none) -> Shielded; Subcategory (none) -> Fixed Inductors; Tolerance (none) -> TBD
- L3: value 6.8uH TBD -> 6u8; AssemblyNote (none) -> TBD; Category (none) -> Inductors, Coils, Chokes; CurrentRMS (none) -> TBD; CurrentSaturation (none) -> TBD; DCR (none) -> TBD; DesignNote (none) -> TBD; Height (none) -> TBD; Lifecycle (none) -> TBD; MPN (none) -> TBD; Manufacturer (none) -> TBD; MountingType (none) -> Surface Mount; OperatingTemp (none) -> TBD; Package (none) -> 1210 (3225 Metric); RoHS (none) -> TBD; SRF (none) -> TBD; SelectionNote (none) -> TBD; Shielding (none) -> TBD; Subcategory (none) -> Fixed Inductors; Tolerance (none) -> TBD
- Q1, Q2: AssemblyNote (none) -> TBD; Category (none) -> Discrete Semiconductor Products; ChannelType (none) -> N-Channel; CurrentID (none) -> TBD; DesignNote (none) -> TBD; GateCharge (none) -> TBD; Height (none) -> TBD; Lifecycle (none) -> TBD; MountingType (none) -> Surface Mount; OperatingTemp (none) -> TBD; Package (none) -> SOT-23; RdsOn (none) -> TBD; RoHS (none) -> TBD; SelectionNote (none) -> TBD; Subcategory (none) -> FETs, MOSFETs - Single; ThermalResistance (none) -> TBD; VgsThreshold (none) -> TBD; VoltageDS (none) -> TBD
- Q3, Q4: AssemblyNote (none) -> TBD; Category (none) -> Discrete Semiconductor Products; ChannelType (none) -> N-Channel; CurrentID (none) -> TBD; DesignNote (none) -> Prototip secimi; AP33772S kapi seviyesiyle kayip/SOA acik.; Field5 SELECTED_FOR_PROTOTYPE -> (none); GateCharge (none) -> TBD; Height (none) -> TBD; Lifecycle (none) -> TBD; MountingType (none) -> Surface Mount; OperatingTemp (none) -> TBD; Package (none) -> SOIC-8; RdsOn (none) -> TBD; RoHS (none) -> TBD; SelectionNote (none) -> TBD; Subcategory (none) -> FETs, MOSFETs - Single; ThermalResistance (none) -> TBD; VgsThreshold (none) -> TBD; VoltageDS (none) -> TBD
- Q5, Q6: AssemblyNote (none) -> TBD; Category (none) -> Discrete Semiconductor Products; ChannelType (none) -> N-Channel; CurrentID (none) -> TBD; DesignNote (none) -> Parca secilmedi; 60V / 4mOhm hedefi ile aranacak.; GateCharge (none) -> TBD; Height (none) -> TBD; Lifecycle (none) -> TBD; MPN (none) -> TBD; Manufacturer (none) -> TBD; MountingType (none) -> TBD; OperatingTemp (none) -> TBD; Package (none) -> TBD; RdsOn (none) -> 4mOhm; RoHS (none) -> TBD; SelectionNote (none) -> TBD; Subcategory (none) -> FETs, MOSFETs - Single; ThermalResistance (none) -> TBD; VgsThreshold (none) -> TBD; VoltageDS (none) -> 60V
- R11: value 5mR / 1W -> 5m0; AssemblyNote (none) -> TBD; Category (none) -> Resistors; Composition (none) -> TBD; DesignNote (none) -> TBD; Field5 KELVIN_4_TERMINAL -> (none); Height (none) -> TBD; Lifecycle (none) -> TBD; MPN (none) -> TBD; Manufacturer (none) -> TBD; MountingType (none) -> Surface Mount; OperatingTemp (none) -> TBD; Package (none) -> 2512 (6332 Metric); PowerRating (none) -> 1W; RoHS (none) -> TBD; SelectionNote (none) -> TBD; Subcategory (none) -> Current Sense Resistors; TempCoefficient (none) -> TBD; TerminationStyle (none) -> 4-Terminal (Kelvin); Tolerance (none) -> TBD
- R12: value 6.2k -> 6k2; AssemblyNote (none) -> TBD; Category (none) -> Resistors; Composition (none) -> TBD; DesignNote (none) -> TBD; Height (none) -> TBD; Lifecycle (none) -> TBD; MPN (none) -> TBD; Manufacturer (none) -> TBD; MountingType (none) -> Surface Mount; OperatingTemp (none) -> TBD; Package (none) -> 0402 (1005 Metric); PowerRating (none) -> TBD; RoHS (none) -> TBD; SelectionNote (none) -> TBD; Subcategory (none) -> Chip Resistor - Surface Mount; TempCoefficient (none) -> TBD; Tolerance (none) -> TBD; VoltageRating (none) -> TBD
- R13, R50, R8, R9: AssemblyNote (none) -> TBD; Category (none) -> Resistors; Composition (none) -> TBD; DesignNote (none) -> TBD; Height (none) -> TBD; Lifecycle (none) -> TBD; MPN (none) -> TBD; Manufacturer (none) -> TBD; MountingType (none) -> Surface Mount; OperatingTemp (none) -> TBD; Package (none) -> 0402 (1005 Metric); PowerRating (none) -> TBD; RoHS (none) -> TBD; SelectionNote (none) -> TBD; Subcategory (none) -> Chip Resistor - Surface Mount; TempCoefficient (none) -> TBD; Tolerance (none) -> TBD; VoltageRating (none) -> TBD
- R14: value 2.2k -> 2k2; AssemblyNote (none) -> TBD; Category (none) -> Resistors; Composition (none) -> TBD; DesignNote (none) -> TBD; Height (none) -> TBD; Lifecycle (none) -> TBD; MPN (none) -> TBD; Manufacturer (none) -> TBD; MountingType (none) -> Surface Mount; OperatingTemp (none) -> TBD; Package (none) -> 0402 (1005 Metric); PowerRating (none) -> TBD; RoHS (none) -> TBD; SelectionNote (none) -> TBD; Subcategory (none) -> Chip Resistor - Surface Mount; TempCoefficient (none) -> TBD; Tolerance (none) -> TBD; VoltageRating (none) -> TBD
- R21: value 100K -> 100k; AssemblyNote (none) -> TBD; Category (none) -> Resistors; Composition (none) -> TBD; DesignNote (none) -> TBD; Height (none) -> TBD; Lifecycle (none) -> TBD; MPN (none) -> TBD; Manufacturer (none) -> TBD; MountingType (none) -> Surface Mount; OperatingTemp (none) -> TBD; Package (none) -> 0402 (1005 Metric); PowerRating (none) -> TBD; RoHS (none) -> TBD; SelectionNote (none) -> TBD; Subcategory (none) -> Chip Resistor - Surface Mount; TempCoefficient (none) -> TBD; Tolerance (none) -> TBD; VoltageRating (none) -> TBD
- R27: value 10K -> 10k; AssemblyNote (none) -> TBD; Category (none) -> Resistors; Composition (none) -> TBD; DesignNote (none) -> TBD; Height (none) -> TBD; Lifecycle (none) -> TBD; MPN (none) -> TBD; Manufacturer (none) -> TBD; MountingType (none) -> Surface Mount; OperatingTemp (none) -> TBD; Package (none) -> 0402 (1005 Metric); PowerRating (none) -> TBD; RoHS (none) -> TBD; SelectionNote (none) -> TBD; Subcategory (none) -> Chip Resistor - Surface Mount; TempCoefficient (none) -> TBD; Tolerance (none) -> TBD; VoltageRating (none) -> TBD
- R38: value 100kR 1% -> 100k; AssemblyNote (none) -> TBD; Category (none) -> Resistors; Composition (none) -> TBD; DesignNote (none) -> TBD; Height (none) -> TBD; Lifecycle (none) -> TBD; MPN (none) -> TBD; Manufacturer (none) -> TBD; MountingType (none) -> Surface Mount; OperatingTemp (none) -> TBD; Package (none) -> 0402 (1005 Metric); PowerRating (none) -> TBD; RoHS (none) -> TBD; SelectionNote (none) -> TBD; Subcategory (none) -> Chip Resistor - Surface Mount; TempCoefficient (none) -> TBD; Tolerance (none) -> +/-1%; VoltageRating (none) -> TBD
- R39: value 10kR 0.1% -> 10k; AssemblyNote (none) -> TBD; Category (none) -> Resistors; Composition (none) -> TBD; DesignNote (none) -> TBD; Height (none) -> TBD; Lifecycle (none) -> TBD; MPN (none) -> TBD; Manufacturer (none) -> TBD; MountingType (none) -> Surface Mount; OperatingTemp (none) -> TBD; Package (none) -> 0402 (1005 Metric); PowerRating (none) -> TBD; RoHS (none) -> TBD; SelectionNote (none) -> TBD; Subcategory (none) -> Chip Resistor - Surface Mount; TempCoefficient (none) -> TBD; Tolerance (none) -> +/-0.1%; VoltageRating (none) -> TBD
- R4: value 4.7 kΩ -> 4k7; AssemblyNote (none) -> TBD; Category (none) -> Resistors; Composition (none) -> TBD; DesignNote (none) -> TBD; Height (none) -> TBD; Lifecycle (none) -> TBD; MPN (none) -> TBD; Manufacturer (none) -> TBD; MountingType (none) -> Surface Mount; OperatingTemp (none) -> TBD; Package (none) -> 0402 (1005 Metric); PowerRating (none) -> TBD; RoHS (none) -> TBD; SelectionNote (none) -> TBD; Subcategory (none) -> Chip Resistor - Surface Mount; TempCoefficient (none) -> TBD; Tolerance (none) -> TBD; VoltageRating (none) -> TBD
- R40: value 3.20kR 0.1% -> 3k20; AssemblyNote (none) -> TBD; Category (none) -> Resistors; Composition (none) -> TBD; DesignNote (none) -> TBD; Height (none) -> TBD; Lifecycle (none) -> TBD; MPN (none) -> TBD; Manufacturer (none) -> TBD; MountingType (none) -> Surface Mount; OperatingTemp (none) -> TBD; Package (none) -> 0402 (1005 Metric); PowerRating (none) -> TBD; RoHS (none) -> TBD; SelectionNote (none) -> TBD; Subcategory (none) -> Chip Resistor - Surface Mount; TempCoefficient (none) -> TBD; Tolerance (none) -> +/-0.1%; VoltageRating (none) -> TBD
- R41: value 12.7kR 1% -> 12k7; AssemblyNote (none) -> TBD; Category (none) -> Resistors; Composition (none) -> TBD; DesignNote (none) -> TBD; Height (none) -> TBD; Lifecycle (none) -> TBD; MPN (none) -> TBD; Manufacturer (none) -> TBD; MountingType (none) -> Surface Mount; OperatingTemp (none) -> TBD; Package (none) -> 0402 (1005 Metric); PowerRating (none) -> TBD; RoHS (none) -> TBD; SelectionNote (none) -> TBD; Subcategory (none) -> Chip Resistor - Surface Mount; TempCoefficient (none) -> TBD; Tolerance (none) -> +/-1%; VoltageRating (none) -> TBD
- R42, R53, R58: value 100kR -> 100k; AssemblyNote (none) -> TBD; Category (none) -> Resistors; Composition (none) -> TBD; DesignNote (none) -> TBD; Height (none) -> TBD; Lifecycle (none) -> TBD; MPN (none) -> TBD; Manufacturer (none) -> TBD; MountingType (none) -> Surface Mount; OperatingTemp (none) -> TBD; Package (none) -> 0402 (1005 Metric); PowerRating (none) -> TBD; RoHS (none) -> TBD; SelectionNote (none) -> TBD; Subcategory (none) -> Chip Resistor - Surface Mount; TempCoefficient (none) -> TBD; Tolerance (none) -> TBD; VoltageRating (none) -> TBD
- R43: value 1kR / 2W -> 1k0; AssemblyNote (none) -> TBD; Category (none) -> Resistors; Composition (none) -> TBD; DesignNote Shunt feed: 0.651W at 28V. Select actual 2W-rated part; foo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 -> Sont besleme: 28V'ta 0.651W. Gercek 2W parca secilecek; aya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; Height (none) -> TBD; Lifecycle (none) -> TBD; MPN (none) -> TBD; Manufacturer (none) -> TBD; MountingType (none) -> Surface Mount; OperatingTemp (none) -> TBD; Package (none) -> 2512 (6332 Metric); PowerRating (none) -> 2W; RoHS (none) -> TBD; SelectionNote (none) -> TBD; Subcategory (none) -> Chip Resistor - Surface Mount; TempCoefficient (none) -> TBD; Tolerance (none) -> TBD; VoltageRating (none) -> TBD
- R47: value 78.7kR -> 78k7; AssemblyNote (none) -> TBD; Category (none) -> Resistors; Composition (none) -> TBD; DesignNote (none) -> TBD; Height (none) -> TBD; Lifecycle (none) -> TBD; MPN (none) -> TBD; Manufacturer (none) -> TBD; MountingType (none) -> Surface Mount; OperatingTemp (none) -> TBD; Package (none) -> 0402 (1005 Metric); PowerRating (none) -> TBD; RoHS (none) -> TBD; SelectionNote (none) -> TBD; Subcategory (none) -> Chip Resistor - Surface Mount; TempCoefficient (none) -> TBD; Tolerance (none) -> TBD; VoltageRating (none) -> TBD
- R48: value 30.1kR -> 30k1; AssemblyNote (none) -> TBD; Category (none) -> Resistors; Composition (none) -> TBD; DesignNote (none) -> TBD; Height (none) -> TBD; Lifecycle (none) -> TBD; MPN (none) -> TBD; Manufacturer (none) -> TBD; MountingType (none) -> Surface Mount; OperatingTemp (none) -> TBD; Package (none) -> 0402 (1005 Metric); PowerRating (none) -> TBD; RoHS (none) -> TBD; SelectionNote (none) -> TBD; Subcategory (none) -> Chip Resistor - Surface Mount; TempCoefficient (none) -> TBD; Tolerance (none) -> TBD; VoltageRating (none) -> TBD
- R49: value 9.76kR -> 9k76; AssemblyNote (none) -> TBD; Category (none) -> Resistors; Composition (none) -> TBD; DesignNote (none) -> TBD; Height (none) -> TBD; Lifecycle (none) -> TBD; MPN (none) -> TBD; Manufacturer (none) -> TBD; MountingType (none) -> Surface Mount; OperatingTemp (none) -> TBD; Package (none) -> 0402 (1005 Metric); PowerRating (none) -> TBD; RoHS (none) -> TBD; SelectionNote (none) -> TBD; Subcategory (none) -> Chip Resistor - Surface Mount; TempCoefficient (none) -> TBD; Tolerance (none) -> TBD; VoltageRating (none) -> TBD
- R5: value 4.7kΩ -> 4k7; AssemblyNote (none) -> TBD; Category (none) -> Resistors; Composition (none) -> TBD; DesignNote (none) -> TBD; Height (none) -> TBD; Lifecycle (none) -> TBD; MPN (none) -> TBD; Manufacturer (none) -> TBD; MountingType (none) -> Surface Mount; OperatingTemp (none) -> TBD; Package (none) -> 0402 (1005 Metric); PowerRating (none) -> TBD; RoHS (none) -> TBD; SelectionNote (none) -> TBD; Subcategory (none) -> Chip Resistor - Surface Mount; TempCoefficient (none) -> TBD; Tolerance (none) -> TBD; VoltageRating (none) -> TBD
- R51, R54: value 1kR -> 1k0; AssemblyNote (none) -> TBD; Category (none) -> Resistors; Composition (none) -> TBD; DesignNote (none) -> TBD; Height (none) -> TBD; Lifecycle (none) -> TBD; MPN (none) -> TBD; Manufacturer (none) -> TBD; MountingType (none) -> Surface Mount; OperatingTemp (none) -> TBD; Package (none) -> 0402 (1005 Metric); PowerRating (none) -> TBD; RoHS (none) -> TBD; SelectionNote (none) -> TBD; Subcategory (none) -> Chip Resistor - Surface Mount; TempCoefficient (none) -> TBD; Tolerance (none) -> TBD; VoltageRating (none) -> TBD
- R52: value 2kR -> 2k0; AssemblyNote (none) -> TBD; Category (none) -> Resistors; Composition (none) -> TBD; DesignNote (none) -> TBD; Height (none) -> TBD; Lifecycle (none) -> TBD; MPN (none) -> TBD; Manufacturer (none) -> TBD; MountingType (none) -> Surface Mount; OperatingTemp (none) -> TBD; Package (none) -> 0402 (1005 Metric); PowerRating (none) -> TBD; RoHS (none) -> TBD; SelectionNote (none) -> TBD; Subcategory (none) -> Chip Resistor - Surface Mount; TempCoefficient (none) -> TBD; Tolerance (none) -> TBD; VoltageRating (none) -> TBD
- R55: value 232kR -> 232k; AssemblyNote (none) -> TBD; Category (none) -> Resistors; Composition (none) -> TBD; DesignNote (none) -> TBD; Height (none) -> TBD; Lifecycle (none) -> TBD; MPN (none) -> TBD; Manufacturer (none) -> TBD; MountingType (none) -> Surface Mount; OperatingTemp (none) -> TBD; Package (none) -> 0402 (1005 Metric); PowerRating (none) -> TBD; RoHS (none) -> TBD; SelectionNote (none) -> TBD; Subcategory (none) -> Chip Resistor - Surface Mount; TempCoefficient (none) -> TBD; Tolerance (none) -> TBD; VoltageRating (none) -> TBD
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Other:
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