File: hardware/usb_pd_controller.kicad_sch (KiCad schematic)
At the start: 85 parts, among them J4 DG142R-5.08-02P-14-00AH, J5 108-0902-001, J6 108-0903-001, Q1 BSS138, Q2 BSS138, Q3 IRF7855TRPBF, Q4 IRF7855TRPBF, Q5 60V 4mR TBD, Q6 60V 4mR TBD, U1 AP33772SDKZ-13-FA02, U11 TPS55340PWPR, U12 AP74502Q, U3 INA228, U5 AOZ1284PI, U6 TL431BIDBZR

Commit message: hardware: RTC'yi BQ32000 + süper kapasitöre geçir, Özdisan BOM'unu şemaya aktar
RTC (mcu):
- U4 RV-3028-C7 -> BQ32000DR (SOIC-8, I2C 0x68, open-drain IRQ, dahili
  trickle charger). Y1 ABS25-32.768KHZ-T (CL 12,5 pF, harici yük C yok),
  C33 Korchip DCL5R5155HF 1,5 F/5,5 V (H-tipi yatay coin, ~22 gün yedek).
- BT1 (CR2032), R22, R23, C10 kaldırıldı; C9 100n -> 1u0 (datasheet >= 1 uF).
- Yeni footprint: Power_Output_Custom:Korchip_DCL_H-Type_D19.0mm_P20.00mm_Horizontal
  (Korchip DCL datasheet çiziminden; numune ile doğrulanmalı).
- Beklenen netlist farkı yalnız RTC netleri: RTC_SCL/SDA/INT U4 pin
  numaraları, Net-(U4-OSCI/OSCO/VBACK) yeni; Net-(BT1-+), Net-(U4-EVI),
  Net-(U4-VBACKUP), U4 CLKOUT kalktı. ERC değişmedi (0 hata, 2 eski uyarı).

Özdisan BOM aktarımı (tüm sayfalar):
- MPN, Manufacturer, parametrik alanlar ve SelectionNote (Özdisan kodu,
  stok 21.09.2026, durum) BOM_OZDISAN_REV_C_20260921.xlsx'ten yazıldı.
- Onaylı değişiklikler: C5/C20/C21 0805; C8/C12/C13/C25/C27/C28 4u7 50V
  X7R 1210; C15/C29 47u 35V hibrit (Device:C_Polarized, CP_Elec_6.3x5.8);
  C31 0603 25V; R59 0805 1/3W; R40 3k24 + R39 10k2 (VOUT 3,3185 V);
  U6 TL431AIDBZR; D4 SX36.
- Stokta olmayan parçalarda (U1, U2, U7, U8, U10, U12, L1, L2, C19) MPN
  korundu, öneri SelectionNote ve todo.txt'de. Alan geometrisi ve
  görünürlük değişmedi. PCB şemadan henüz güncellenmedi.

Aynı commit'te önceden commit edilmemiş çalışma: Q3/Q5 SQJB60EP ve U3
INA226 entegrasyonu, raporları ve datasheet'leri.

Co-Authored-By: Claude Opus 5 <noreply@anthropic.com>
Parts:
- C1, C11, C2, C24: Dielectric TBD -> X7R; MPN TBD -> CC0402KRX7R9BB104; Manufacturer TBD -> Yageo; SelectionNote TBD -> Özdisan 609906; stok 117450 (21.09.2026); Uygun. Tek MPN: C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; Tolerance TBD -> +/-10%; VoltageRating TBD -> 50V
- C12, C13: value 10u -> 4u7; DesignNote X7R; C12+C13 efektif kapasite 28V'ta >=10uF olmali, MPN dog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 -> Ortak secim 4u7 50V X7R 1210 (1210 10u 50V stokta yok). V_P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; MPN TBD -> CL32B475KBJNNNE; Manufacturer TBD -> Samsung Electro-Mechanics; SelectionNote TBD -> Özdisan 1206577; stok 37121 (21.09.2026); Muadil. 21.09 üçü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; Tolerance TBD -> +/-10%
- C14: MPN TBD -> CC0402KRX7R9BB104; Manufacturer TBD -> Yageo; SelectionNote TBD -> Özdisan 609906; stok 117450 (21.09.2026); Uygun. Tek MPN: C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; Tolerance TBD -> +/-10%
- C15: footprint Capacitor_SMD:C_0402_1005Metric -> Capacitor_SMD:CP_Elec_6.3x5.8; symbol Device:C -> Device:C_Polarized; CapacitorType (none) -> Hybrid Polymer Aluminum; DesignNote X7R; banka efektif Cout 3.3V'ta >=44uF olmali, MPN dogrulan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 -> 47uF 35V hibrit; AOZ1284 cikisinda ~56kHz ESR sifiri, R41/C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; Dielectric X7R -> (none); ESR (none) -> 60mOhm @100kHz; EffectiveCapacitance TBD -> (none); Height TBD -> 5.8mm; Lifetime (none) -> 10000h @105C; MPN TBD -> EEHZA1V470P; Manufacturer TBD -> Panasonic; OperatingTemp TBD -> -55C to 105C; Package 0402 (1005 Metric) -> 6.3x5.8mm SMD Can; RippleCurrent (none) -> 1.3A @100kHz; SelectionNote TBD -> Özdisan 1098034; stok 840 (21.09.2026); Uygun. 21.09 üçüncü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; Subcategory Ceramic Capacitors -> Aluminum - Polymer Capacitors; Tolerance TBD -> +/-20%; VoltageRating 10V -> 35V
- C16: Dielectric X7R -> X5R; MPN TBD -> CL32A476KOJNNNE; Manufacturer TBD -> Samsung Electro-Mechanics; SelectionNote TBD -> Özdisan 423179; stok 53829 (21.09.2026); Uygun. +3.3V; 16V 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; Tolerance TBD -> +/-10%; VoltageRating 10V -> 16V
- C17: Dielectric TBD -> X7R; MPN TBD -> CC0402KRX7R9BB104; Manufacturer TBD -> Yageo; SelectionNote TBD -> Özdisan 609906; stok 117450 (21.09.2026); Uygun. Tek MPN: C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; Tolerance TBD -> +/-10%; VoltageRating 16V -> 50V
- C18: Dielectric TBD -> X7R; MPN TBD -> CL05B103KA5NNNC; Manufacturer TBD -> Samsung Electro-Mechanics; SelectionNote TBD -> Özdisan 446224; stok 43984 (21.09.2026); Uygun.; Tolerance TBD -> +/-10%; VoltageRating 10V -> 25V
- C19: SelectionNote TBD -> Özdisan 446224 / 521982; stok 43984 (21.09.2026); Muadil. 2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
- C23: Dielectric TBD -> X7R; MPN TBD -> CL05B473KO5NNNC; Manufacturer TBD -> Samsung Electro-Mechanics; SelectionNote TBD -> Özdisan 443226; stok 48227 (21.09.2026); Uygun.; Tolerance TBD -> +/-10%; VoltageRating TBD -> 16V
- C25, C27, C28: value 10u -> 4u7; DesignNote TBD -> Ortak secim 4u7 50V X7R 1210 (1210 10u 50V stokta yok). V_P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; Dielectric TBD -> X7R; MPN TBD -> CL32B475KBJNNNE; Manufacturer TBD -> Samsung Electro-Mechanics; SelectionNote TBD -> Özdisan 1206577; stok 37121 (21.09.2026); Muadil. 21.09 üçü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; Tolerance TBD -> +/-10%
- C26, C32: Dielectric TBD -> X7R; MPN TBD -> CC0402KRX7R9BB104; Manufacturer TBD -> Yageo; SelectionNote TBD -> Özdisan 609906; stok 117450 (21.09.2026); Uygun. Tek MPN: C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; Tolerance TBD -> +/-10%
- C29: footprint Capacitor_SMD:C_1210_3225Metric -> Capacitor_SMD:CP_Elec_6.3x5.8; symbol Device:C -> Device:C_Polarized; CapacitorType (none) -> Hybrid Polymer Aluminum; DesignNote TBD -> PD_VOUT sonumleme (C_DAMP): 47uF, 35-50V, ESR 50-100mOhm; s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; Dielectric TBD -> (none); ESR (none) -> 60mOhm @100kHz; EffectiveCapacitance TBD -> (none); Height TBD -> 5.8mm; Lifetime (none) -> 10000h @105C; MPN TBD -> EEHZA1V470P; Manufacturer TBD -> Panasonic; OperatingTemp TBD -> -55C to 105C; Package 1210 (3225 Metric) -> 6.3x5.8mm SMD Can; RippleCurrent (none) -> 1.3A @100kHz; SelectionNote TBD -> Özdisan 1098034; stok 840 (21.09.2026); Uygun. 21.09 üçüncü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; Subcategory Ceramic Capacitors -> Aluminum - Polymer Capacitors; Tolerance TBD -> +/-20%; VoltageRating 50V -> 35V
- C3: Dielectric X7R -> X5R; MPN TBD -> CL21A225KB9LNNC; Manufacturer TBD -> Samsung Electro-Mechanics; SelectionNote TBD -> Özdisan 522705; stok 52721 (21.09.2026); Uygun. 21.09 üçünc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; Tolerance TBD -> +/-10%
- C30: Dielectric TBD -> X7R; MPN TBD -> CC0402KRX7R9BB223; Manufacturer TBD -> Yageo; SelectionNote TBD -> Özdisan 746989; stok 413880 (21.09.2026); Uygun.; Tolerance TBD -> +/-10%
- C31: footprint Capacitor_SMD:C_0402_1005Metric -> Capacitor_SMD:C_0603_1608Metric; DesignNote TBD -> AP74502Q VCAP-VIN arasi; VCAP-VSRC max 13.9V, VCAP-VIN abs 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; Dielectric TBD -> X7R; MPN TBD -> CL10B224KA8NNNC; Manufacturer TBD -> Samsung Electro-Mechanics; Package 0402 (1005 Metric) -> 0603 (1608 Metric); SelectionNote TBD -> Özdisan 15507; stok 664332 (21.09.2026); Uygun. 21.09 üçünc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; Tolerance TBD -> +/-10%
- C4: Dielectric TBD -> X5R; MPN TBD -> EMK105BJ105KVHF; Manufacturer TBD -> Taiyo Yuden; SelectionNote TBD -> Özdisan 623573; stok 5005 (21.09.2026); Uygun. C4 (PD_5V) i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; Tolerance TBD -> +/-10%; VoltageRating 10V -> 16V
- C8: value 10u -> 4u7; footprint Capacitor_SMD:C_0402_1005Metric -> Capacitor_SMD:C_1210_3225Metric; DesignNote TBD -> Ortak secim 4u7 50V X7R 1210 (1210 10u 50V stokta yok). V_P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; Dielectric TBD -> X7R; MPN TBD -> CL32B475KBJNNNE; Manufacturer TBD -> Samsung Electro-Mechanics; Package 0402 (1005 Metric) -> 1210 (3225 Metric); SelectionNote TBD -> Özdisan 1206577; stok 37121 (21.09.2026); Muadil. 21.09 üçü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; Tolerance TBD -> +/-10%
- D1: MPN TBD -> APHHS1005SURCK; Manufacturer TBD -> Kingbright; SelectionNote TBD -> Özdisan 708179; stok 272 (21.09.2026); Uygun. 21.09 ikinci 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
- D2: SelectionNote TBD -> Özdisan 574723; stok 51111 (21.09.2026); Uygun.
- D4: value SS34 TBD -> SX36; MPN TBD -> SX36_R1_00001; Manufacturer TBD -> PANJIT; SelectionNote TBD -> Özdisan 574842; stok 437 (21.09.2026); Uygun. SS34 Özdisan'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
- D5: MPN BAT54 -> BAT54T1G; Manufacturer TBD -> onsemi; SelectionNote TBD -> Özdisan 614028; stok 595 (21.09.2026); Uygun. Otomatik MPN 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
- D6: MPN BZT52C12 -> BZT52-C12_R1_00001; Manufacturer TBD -> PANJIT; SelectionNote TBD -> Özdisan 560765; stok 4720 (21.09.2026); Uygun.
- D7: MPN SMBJ30A -> SMBJ30A-E3/52; Manufacturer TBD -> Vishay; SelectionNote TBD -> Özdisan 507320; stok 15956 (21.09.2026); Uygun. Şema açıkla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
- J4: SelectionNote TBD -> Özdisan 695538; stok 1624 (21.09.2026); Uygun. 21.09 ikinci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
- J5, J6: SelectionNote TBD -> Özdisan (21.09.2026): İndekste yok. 21.09 ikinci kontrol: b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
- L1: SelectionNote TBD -> Özdisan (21.09.2026): Stokta yok. 11.09 raporunda Özdisan s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
- L3: MPN TBD -> B82422H1682K000; Manufacturer TBD -> TDK (EPCOS); SelectionNote TBD -> Özdisan 489001; stok 10 (21.09.2026); Uyarı. Footprint'e uy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
- Q1, Q2: MPN BSS138 -> BSS138P,215; Manufacturer onsemi -> Nexperia; SelectionNote TBD -> Özdisan 737689; stok 73553 (21.09.2026); Uygun. Jenerik BSS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
- Q3: renamed from Q4; value IRF7855TRPBF -> SQJB60EP; footprint Package_SO:SOIC-8_3.9x4.9mm_P1.27mm -> (none); symbol Power_Supply_Custom:IRF7855_SO8 -> Power_Supply_Custom:SQJB60EP; AssemblyNote TBD -> Leadless paket; elle lehimleme onerilmiyor (datasheet not e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; CurrentID TBD -> 30A; DesignNote Prototip secimi; AP33772S kapi seviyesiyle kayip/SOA acik. -> Footprint dogrulanmadi: PowerPAK SO-8L DUAL land pattern Ki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; GateCharge TBD -> 18nC; Height TBD -> 1.14mm max; MPN IRF7855TRPBF -> SQJB60EP-T1_GE3; Manufacturer Infineon Technologies -> Vishay Siliconix; OperatingTemp TBD -> -55C...+175C; Package SOIC-8 -> PowerPAK SO-8L Dual; RdsOn TBD -> 12mOhm; SelectionNote TBD -> Özdisan 700940; stok 107664 (21.09.2026); Uygun. Seçim rapo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; Subcategory FETs, MOSFETs - Single -> FETs, MOSFETs - Arrays; ThermalResistance TBD -> RthJA 85C/W, RthJC 3.1C/W; VgsThreshold TBD -> 1.5-2.5V; VoltageDS TBD -> 60V
- Q3: value IRF7855TRPBF -> SQJB60EP; footprint Package_SO:SOIC-8_3.9x4.9mm_P1.27mm -> (none); symbol Power_Supply_Custom:IRF7855_SO8 -> Power_Supply_Custom:SQJB60EP; AssemblyNote TBD -> Leadless paket; elle lehimleme onerilmiyor (datasheet not e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; CurrentID TBD -> 30A; DesignNote Prototip secimi; AP33772S kapi seviyesiyle kayip/SOA acik. -> Footprint dogrulanmadi: PowerPAK SO-8L DUAL land pattern Ki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; GateCharge TBD -> 18nC; Height TBD -> 1.14mm max; MPN IRF7855TRPBF -> SQJB60EP-T1_GE3; Manufacturer Infineon Technologies -> Vishay Siliconix; OperatingTemp TBD -> -55C...+175C; Package SOIC-8 -> PowerPAK SO-8L Dual; RdsOn TBD -> 12mOhm; SelectionNote TBD -> Özdisan 700940; stok 107664 (21.09.2026); Uygun. Seçim rapo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; Subcategory FETs, MOSFETs - Single -> FETs, MOSFETs - Arrays; ThermalResistance TBD -> RthJA 85C/W, RthJC 3.1C/W; VgsThreshold TBD -> 1.5-2.5V; VoltageDS TBD -> 60V
- Q5: value 60V 4mR TBD -> SQJB60EP; symbol Transistor_FET:Q_NMOS_GSD -> Power_Supply_Custom:SQJB60EP; AssemblyNote TBD -> Leadless paket; elle lehimleme onerilmiyor (datasheet not e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; CurrentID TBD -> 30A; DesignNote Parca secilmedi; 60V / 4mOhm hedefi ile aranacak. -> Footprint dogrulanmadi: PowerPAK SO-8L DUAL land pattern Ki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; GateCharge TBD -> 18nC; Height TBD -> 1.14mm max; MPN TBD -> SQJB60EP-T1_GE3; Manufacturer TBD -> Vishay Siliconix; MountingType TBD -> Surface Mount; OperatingTemp TBD -> -55C...+175C; Package TBD -> PowerPAK SO-8L Dual; RdsOn 4mOhm -> 12mOhm; SelectionNote TBD -> Özdisan 700940; stok 107664 (21.09.2026); Uygun. Seçim rapo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; Subcategory FETs, MOSFETs - Single -> FETs, MOSFETs - Arrays; ThermalResistance TBD -> RthJA 85C/W, RthJC 3.1C/W; VgsThreshold TBD -> 1.5-2.5V
- Q5: renamed from Q6; value 60V 4mR TBD -> SQJB60EP; symbol Transistor_FET:Q_NMOS_GSD -> Power_Supply_Custom:SQJB60EP; AssemblyNote TBD -> Leadless paket; elle lehimleme onerilmiyor (datasheet not e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; CurrentID TBD -> 30A; DesignNote Parca secilmedi; 60V / 4mOhm hedefi ile aranacak. -> Footprint dogrulanmadi: PowerPAK SO-8L DUAL land pattern Ki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; GateCharge TBD -> 18nC; Height TBD -> 1.14mm max; MPN TBD -> SQJB60EP-T1_GE3; Manufacturer TBD -> Vishay Siliconix; MountingType TBD -> Surface Mount; OperatingTemp TBD -> -55C...+175C; Package TBD -> PowerPAK SO-8L Dual; RdsOn 4mOhm -> 12mOhm; SelectionNote TBD -> Özdisan 700940; stok 107664 (21.09.2026); Uygun. Seçim rapo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; Subcategory FETs, MOSFETs - Single -> FETs, MOSFETs - Arrays; ThermalResistance TBD -> RthJA 85C/W, RthJC 3.1C/W; VgsThreshold TBD -> 1.5-2.5V
- R11, RShunt1: Composition TBD -> Metal Element (Isaohm); MPN TBD -> BVT-I-R005-1.0; Manufacturer TBD -> Isabellenhütte; PowerRating 1W -> 2.5W @70C / 1.5W @100C; SelectionNote TBD -> Özdisan 536256; stok 774 (21.09.2026); Uygun. 21.09 dördünc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; TempCoefficient TBD -> 0+/-50ppm/C; Tolerance TBD -> +/-1%; VoltageRating (none) -> N/A
- R12: Composition TBD -> Thick Film; MPN TBD -> 0402WGF6201TCE; Manufacturer TBD -> Royalohm; PowerRating TBD -> 0.0625W; SelectionNote TBD -> Özdisan 359873; stok 19300 (21.09.2026); Uygun.; TempCoefficient TBD -> +/-100ppm/C; Tolerance TBD -> +/-1%; VoltageRating TBD -> 50V
- R13: Composition TBD -> Thin Film; MPN TBD -> TC0250B1000TCC; Manufacturer TBD -> Royalohm; PowerRating TBD -> 0.0625W; SelectionNote TBD -> Özdisan 569711; stok 7445 (21.09.2026); Uygun.; TempCoefficient TBD -> +/-50ppm/C; Tolerance TBD -> +/-0.1%; VoltageRating TBD -> 25V
- R14: Composition TBD -> Precision Thick Film; MPN TBD -> ERJ2RKF2201X; Manufacturer TBD -> Panasonic; PowerRating TBD -> 0.1W; SelectionNote TBD -> Özdisan 494655; stok 67988 (21.09.2026); Uygun.; TempCoefficient TBD -> +/-100ppm/C; Tolerance TBD -> +/-1%; VoltageRating TBD -> 50V
- R21: Composition TBD -> Thick Film; MPN TBD -> CQ02WGF1003TCE; Manufacturer TBD -> Royalohm; PowerRating TBD -> 0.0625W; SelectionNote TBD -> Özdisan 587906; stok 99900 (21.09.2026); Satın alınmaz. DNP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; TempCoefficient TBD -> +/-100ppm/C; Tolerance TBD -> +/-1%; VoltageRating TBD -> 50V
- R27, R56, R57: Composition TBD -> Thin Film; MPN TBD -> TC0250B1002TCC; Manufacturer TBD -> Royalohm; PowerRating TBD -> 0.0625W; SelectionNote TBD -> Özdisan 569744; stok 4220 (21.09.2026); Uygun. Özdisan'da 0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; TempCoefficient TBD -> +/-50ppm/C; Tolerance TBD -> +/-0.1%; VoltageRating TBD -> 25V
- R38: Composition TBD -> Thick Film; MPN TBD -> CQ02WGF1003TCE; Manufacturer TBD -> Royalohm; PowerRating TBD -> 0.0625W; SelectionNote TBD -> Özdisan 587906; stok 99900 (21.09.2026); Uygun.; TempCoefficient TBD -> +/-100ppm/C; VoltageRating TBD -> 50V
- R39: value 10k -> 10k2; Composition TBD -> Thick Film; DesignNote TBD -> AOZ1284 FB ust direnci. R40=3k24 ile VOUT=0.8*(1+10.2/3.24)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; MPN TBD -> RC1005F1022CS; Manufacturer TBD -> Samsung Electro-Mechanics; PowerRating TBD -> 0.0625W; SelectionNote TBD -> Özdisan 695131; stok 5865 (21.09.2026); Muadil. 21.09 üçünc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; TempCoefficient TBD -> +/-100ppm/C; Tolerance +/-0.1% -> +/-1%; VoltageRating TBD -> 50V
- R4, R5, R6, R7: Composition TBD -> High Power Thick Film; MPN TBD -> HP02WAF4701TCE; Manufacturer TBD -> Royalohm; PowerRating TBD -> 0.1W; SelectionNote TBD -> Özdisan 603918; stok 9400 (21.09.2026); Uygun.; TempCoefficient TBD -> +/-100ppm/C; Tolerance TBD -> +/-1%; VoltageRating TBD -> 50V
- R40: value 3k20 -> 3k24; Composition TBD -> Precision Thick Film; DesignNote TBD -> AOZ1284 FB alt direnci. %1 serisinde 3k20 yok; R39=10k2 ile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; MPN TBD -> ERJ2RKF3241X; Manufacturer TBD -> Panasonic; PowerRating TBD -> 0.1W; SelectionNote TBD -> Özdisan 494659; stok 76745 (21.09.2026); Muadil. 21.09 üçün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; TempCoefficient TBD -> +/-100ppm/C; Tolerance +/-0.1% -> +/-1%; VoltageRating TBD -> 50V
- R41: Composition TBD -> Thick Film; MPN TBD -> 0402WGF1272TCE; Manufacturer TBD -> Royalohm; PowerRating TBD -> 0.0625W; SelectionNote TBD -> Özdisan 506317; stok 18380 (21.09.2026); Uygun.; TempCoefficient TBD -> +/-100ppm/C; VoltageRating TBD -> 50V
- R42, R53, R58: Composition TBD -> Thick Film; MPN TBD -> CQ02WGF1003TCE; Manufacturer TBD -> Royalohm; PowerRating TBD -> 0.0625W; SelectionNote TBD -> Özdisan 587906; stok 99900 (21.09.2026); Uygun.; TempCoefficient TBD -> +/-100ppm/C; Tolerance TBD -> +/-1%; VoltageRating TBD -> 50V
- R43: Composition TBD -> Anti-Surge Thick Film; MPN TBD -> PS122WF1001T4E; Manufacturer TBD -> Royalohm; SelectionNote TBD -> Özdisan 746122; stok 93571 (21.09.2026); Uygun. 2W şartı (2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; TempCoefficient TBD -> +/-100ppm/C; Tolerance TBD -> +/-1%; VoltageRating TBD -> 500V
- R47: Composition TBD -> Thick Film; MPN TBD -> 0402WGF7872TCE; Manufacturer TBD -> Royalohm; PowerRating TBD -> 0.0625W; SelectionNote TBD -> Özdisan 506387; stok 7070 (21.09.2026); Uygun.; TempCoefficient TBD -> +/-100ppm/C; Tolerance TBD -> +/-1%; VoltageRating TBD -> 50V
- R48: Composition TBD -> Thick Film; MPN TBD -> 0402WGF3012TCE; Manufacturer TBD -> Royalohm; PowerRating TBD -> 0.0625W; SelectionNote TBD -> Özdisan 506349; stok 10680 (21.09.2026); Uygun.; TempCoefficient TBD -> +/-100ppm/C; Tolerance TBD -> +/-1%; VoltageRating TBD -> 50V
- R49: Composition TBD -> Thick Film; MPN TBD -> 0402WGF9761TCE; Manufacturer TBD -> Royalohm; PowerRating TBD -> 0.0625W; SelectionNote TBD -> Özdisan 506310; stok 17170 (21.09.2026); Uygun.; TempCoefficient TBD -> +/-100ppm/C; Tolerance TBD -> +/-1%; VoltageRating TBD -> 50V
- R50: Composition TBD -> Thick Film; MPN TBD -> RC0402JR-07820RL; Manufacturer TBD -> Yageo; PowerRating TBD -> 0.0625W; SelectionNote TBD -> Özdisan 423409; stok 92000 (21.09.2026); Uygun. 0402 820R y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; TempCoefficient TBD -> +/-100ppm/C; Tolerance TBD -> +/-5%; VoltageRating TBD -> 50V
- R51, R54: Composition TBD -> Thin Film; MPN TBD -> RT0402BRD071KL; Manufacturer TBD -> Yageo; PowerRating TBD -> 0.0625W; SelectionNote TBD -> Özdisan 1212342; stok 37995 (21.09.2026); Uygun. 0402 1k %1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; TempCoefficient TBD -> +/-25ppm/C; Tolerance TBD -> +/-0.1%; VoltageRating TBD -> 50V
- R52: Composition TBD -> Precision Thick Film; MPN TBD -> ERJ2RKF2001X; Manufacturer TBD -> Panasonic; PowerRating TBD -> 0.1W; SelectionNote TBD -> Özdisan 518487; stok 34590 (21.09.2026); Uygun.; TempCoefficient TBD -> +/-100ppm/C; Tolerance TBD -> +/-1%; VoltageRating TBD -> 50V
- R55: Composition TBD -> Thick Film; MPN TBD -> 0402WGF2323TCE; Manufacturer TBD -> Royalohm; PowerRating TBD -> 0.0625W; SelectionNote TBD -> Özdisan 506426; stok 6600 (21.09.2026); Uygun.; TempCoefficient TBD -> +/-100ppm/C; Tolerance TBD -> +/-1%; VoltageRating TBD -> 50V
- R59: footprint Resistor_SMD:R_0402_1005Metric -> Resistor_SMD:R_0805_2012Metric; Composition TBD -> High Power Thick Film; DesignNote TBD -> OUT_POS bleed. 30V OVLO esiginde 90mW; %50 azaltma ile >=0.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; MPN TBD -> HP05W3F1002T5E; Manufacturer TBD -> Royalohm; Package 0402 (1005 Metric) -> 0805 (2012 Metric); PowerRating 0.25W -> 0.333W; SelectionNote TBD -> Özdisan 604238; stok 710 (21.09.2026); Uygun. 21.09 üçüncü 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; TempCoefficient TBD -> +/-100ppm/C; Tolerance TBD -> +/-1%; VoltageRating TBD -> 150V
- R8: Composition TBD -> Thick Film; MPN TBD -> CRCW040212K0FKED; Manufacturer TBD -> Vishay; PowerRating TBD -> 0.0625W; SelectionNote TBD -> Özdisan 519356; stok 6761 (21.09.2026); Uygun.; TempCoefficient TBD -> +/-100ppm/C; Tolerance TBD -> +/-1%; VoltageRating TBD -> 50V
- R9: Composition TBD -> Thin Film; MPN TBD -> TC0250B2002TCC; Manufacturer TBD -> Royalohm; PowerRating TBD -> 0.0625W; SelectionNote TBD -> Özdisan 570296; stok 3225 (21.09.2026); Uygun. 0402 20k %1 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; TempCoefficient TBD -> +/-50ppm/C; Tolerance TBD -> +/-0.1%; VoltageRating TBD -> 25V
- TH1: Manufacturer THINKING -> Thinking Electronic; SelectionNote TBD -> Özdisan 509291; stok 8430 (21.09.2026); Uygun.
- TP1, TP2, TP3, TP4, TP5: SelectionNote TBD -> Özdisan (21.09.2026): Satın alınmaz. Kart üzerindeki pad; s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
- U1: SelectionNote TBD -> Özdisan (21.09.2026): Stokta yok. Özdisan indeksinde (stoks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
- U11: SelectionNote TBD -> Özdisan 645605; stok 449 (21.09.2026); Uygun.
- U12: SelectionNote TBD -> Özdisan (21.09.2026): Stokta yok. İdeal diyot kategorisi in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
- U3: value INA228 -> INA226; symbol Sensor_Energy:INA228 -> Sensor_Energy:INA226; MPN INA228AIDGSR -> INA226AIDGSR; SelectionNote TBD -> Özdisan 640350; stok 9865 (21.09.2026); Uygun. Seçim raporu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
- U5: SelectionNote TBD -> Özdisan 594873; stok 6659 (21.09.2026); Uygun. Şemada 'Teda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
- U6: value TL431BIDBZR -> TL431AIDBZR; MPN TL431BIDBZR -> TL431AIDBZR; SelectionNote TBD -> Özdisan 341981; stok 2428 (21.09.2026); Muadil. B sınıfı (%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
Connections:
- net GATE_DRV: now also Q5.2 (G), Q5.4 (G); no longer Q5.1 (G), Q5.1 (G)
- net PD_GATE: now also Q3.2 (G); no longer Q3.4 (G)
- net PD_VBUS_SENSED: now also Q5.7 (D), Q5.8 (D); no longer Q3.5 (D), Q3.6 (D), Q5.3 (D)
- net PD_VOUT: no longer Q3.7 (D), Q3.8 (D)
- net SRC_COMMON: now also Q5.1 (S), Q5.3 (S); no longer Q5.2 (S), Q5.2 (S)
- net SW_OUT: now also Q5.5 (D), Q5.6 (D); no longer Q5.3 (D)
- new net: Q3.1 (S), Q3.3 (S)
Other:
- note added: "INA226 OLCUM + PANEL CIKISI"
- note removed: "INA228 OLCUM + PANEL CIKISI"

Commit message: hardware: ekranı TFT032B018'e geçir, todo'yu güncelle, Imax 3 A kararını kaydet
TFT032B018 (userinterface):
- J3 Conn_01x40 (Molex 54132-4062) -> Conn_01x30, KLS L-KLS1-242I-2.0-30-R;
  yeni footprint Connector_FPC_Custom:KLS_L-KLS1-242I-2.0-30_1x30-2MP_P0.50mm_Horizontal
  (fp-lib-table'a eklendi). SPI: 16=DC, 17=SCLK, 18=CS, 19=MOSI, 20=RST;
  21 IM=3.3V; DB0..7, RDX GND; TE ve dokunmatik pinleri boş. C34 1u0 dekuplaj.
- Backlight: TPS61023 boost (U7, L2, C20, C21, R44, R45) ve CAT4104 (U8,
  C22, R46) kalktı; +3.3V -> R60 5R6 -> BL_A, BL_K -> Q7 IRLML6344
  (R28/R29 ile TFT_BL_PWM).
- Beklenen netlist farkı: BACKLIGHT_4V2, BL_BOOST_*, BL_K1..4, Net-(U8-*)
  kalktı; BL_A, BL_K, Net-(Q7-G) eklendi; TFT_* netleri J3'ün yeni pin
  numaralarına geçti. ERC değişmedi (0 hata, 2 eski uyarı).
- Özdisan alanları (J3, Q7, R60, C34) ve BOM tablosu güncellendi; ekran modülü
  şema dışı satır olarak BOM'da (stok 5).
- mcu/userinterface: kullanılmayan lib_symbols tanımları silindi
  (Device:Battery_Cell, AO3400A); netlist farkı YOK.

Kayıtlar:
- todo.txt: tamamlanan şema maddeleri
  design_decisions/output/SEMA_TAMAMLANAN_TODO_REV_C_20260922.md'ye taşındı;
  AP74502Q sembolü Diodes datasheet'iyle doğrulandı (datasheet eklendi),
  U12 paket (SOT28) kontrolü ve SMBJ30A PCB maddesi güncellendi.
- Maksimum çıkış akımı 3 A: design_decisions/output/CIKIS_AKIMI_3A_KARARI_20260922.md.
  "Imax kesinleştir" ve "3.3 V adaptör başlığı" maddeleri kapandı; prototip ve
  INA226 firmware değerleri 3 A'e göre güncellendi, RShunt1 5 mOhm'da kaldı.

Co-Authored-By: Claude Opus 5 <noreply@anthropic.com>
Parts:
- C4: SelectionNote Özdisan 623573; stok 5005 (21.09.2026); Uygun. C4 (PD_5V) için ≥10V şartını karşılar. C9: BQ32000 VCC dekuplajı, datasheet ≥1 µF istiyor (100n → 1u0). -> Özdisan 623573; stok 5005 (21.09.2026); Uygun. C4 (PD_5V) için ≥10V şartını karşılar. C9: BQ32000 VCC dekuplajı, datasheet ≥1 µF istiyor (100n → 1u0). C34: TFT032B018 VCI/IOVCC dekuplajı (J3 yanında).
Changed lines of the file:
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@@
 			)
 		)
-		(property "SelectionNote" "Özdisan 623573; stok 5005 (21.09.2026); Uygun. C4 (PD_5V) için ≥10V şartını karşılar. C9: BQ32000 VCC dekuplajı, datasheet ≥1 µF istiyor (100n → 1u0)."
+		(property "SelectionNote" "Özdisan 623573; stok 5005 (21.09.2026); Uygun. C4 (PD_5V) için ≥10V şartını karşılar. C9: BQ32000 VCC dekuplajı, datasheet ≥1 µF istiyor (100n → 1u0). C34: TFT032B018 VCI/IOVCC dekuplajı (J3 yanında)."
 			(at 85.09 67.31 0)
 			(hide yes)

Commit message: hardware: çıkış anahtarını LM74801'e geçir, USB-C korumasını ve OUT_EN'i düzelt
Çıkış anahtarı / ters akım (usb_pd_controller):
- U12 AP74502Q -> LM74801-Q1 (LM74801QDRRRQ1, WSON-12, EP boşta). AP74502Q
  ideal diyot değil; çıkış açıkken ters akım doğrudan adaptör VBUS'ına
  gidiyordu. Ortak-source Q5: HGATE -> Q5A (GATE_DRV, R54/C30, D6),
  DGATE -> Q5B (yeni net), A/OUT = SRC_COMMON, C = SW_OUT, VS/VSNS/SW = V_PRE.
- R55 232k -> 237k: LM74801 OV 30.4 V (29.5-31.3 V), 28 V EPR +%5 üstünde.
- OUT_EN kapatamıyordu (EN ~1.57 V > 1.32 V): R57 kalktı, U13 74LVC1G08
  (SN74LVC1G08DBVR) EN = OUT_EN AND ~ALERT; R61 4k7 OUT_EN pull-down, C35.
- AOZ1284 kompanzasyonu: R41 12k7 -> 51k, C19 18n -> 15n (fC ~5 -> ~20 kHz).
- Q3/Q5 footprint: yeni Package_SO_Custom:Vishay_PowerPAK_SO-8L_Dual
  (Vishay doc 63817'den ölçüldü; 6/8 yalnız bakır eş drain pedleri).
- TL431DBZ önbelleği KiCad 10 kütüphanesinden yenilendi (pin uçları aynı).

MCU:
- RTC (BQ32000) PD/INA226 I2C bus'ına alındı, R25/R26 kalktı; OUT_EN = GPIO6
  (MTCK), GPIO7 boş.

USB-C girişi (usb_c_input):
- CC1/CC2'ye Rd 5k1 (R62/R63) eklendi; AP33772S Figure 1 harici Rd istiyor,
  şemada hiç yoktu.
- CC1/CC2 5.5 V'luk U10'dan ayrıldı (AP33772S CC 34 V'a dayanır, U10 28 V
  kısa devrede yanardı); D8/D9 SMF30A CC ESD opsiyonu DNP.
- U10 TPD4EUSB30 -> USBLC6-2SC6 (yalnız D+/D-, jumper_pin_groups ile
  flow-through, VBUS pini +3.3V). D3 SMBJ30A yer için sağa taşındı.

Doğrulama: her adımda beklenen netlist farkı; son durum ERC 0 hata / 0 uyarı,
101 net. Parçalar Özdisan stoğundan (SelectionNote alanlarında).

Kayıtlar:
- todo.txt açık kalanlara göre yeniden düzenlendi.
- design_decisions/output/SEMA_TAMAMLANAN_TODO_REV_C_20260922.md: bu
  maddelerin gerekçe ve hesapları.
- design_decisions/output/CIKIS_GERILIMI_28V_TAVANI_20260922.md: 28 V tavanı.
- Datasheet'ler: LM7480-Q1, SMF (Thinking), USBLC6-2.

Co-Authored-By: Claude Opus 5 <noreply@anthropic.com>
Parts:
- removed R57: 10k, Resistor_SMD:R_0402_1005Metric, symbol Device:R_Small_US
- added C35: 100n, Capacitor_SMD:C_0402_1005Metric, symbol Device:C
- added R61: 4k7, Resistor_SMD:R_0402_1005Metric, symbol Device:R_Small_US
- added U13: 74LVC1G08, Package_TO_SOT_SMD:SOT-23-5, symbol Power_Path_Custom:74LVC1G08
- C19: value 18n -> 15n; DesignNote TBD -> AOZ1284 CC: sifir 1/(2pi 51k 15n) = 208 Hz < fC/5.; Dielectric TBD -> X7R; MPN TBD -> CL05B153KO5NNNC; Manufacturer TBD -> Samsung; SelectionNote Özdisan 446224 / 521982; stok 43984 (21.09.2026); Muadil. 2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 -> Özdisan 521922; stok 5150 (22.09.2026); Uygun. 12n stokta y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; Tolerance TBD -> +/-10%
- Q3, Q5: footprint (none) -> Package_SO_Custom:Vishay_PowerPAK_SO-8L_Dual
- R41: value 12k7 -> 51k; DesignNote TBD -> AOZ1284 RC: fC ~20 kHz (CO ~89 uF: C15 hibrit + C16).; MPN 0402WGF1272TCE -> 0402WGF5102TCE; SelectionNote Özdisan 506317; stok 18380 (21.09.2026); Uygun. -> Özdisan 359892; stok 29800 (22.09.2026); Uygun.
- R55: value 232k -> 237k; DesignNote TBD -> OV = 1.231 V x (1 + 237k/10k) = 30.4 V (29.5-31.3 V); 28 V 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; MPN 0402WGF2323TCE -> 0402WGF2373TCE; SelectionNote Özdisan 506426; stok 6600 (21.09.2026); Uygun. -> Özdisan 506427; stok 18600 (22.09.2026); Uygun.
- U12: value AP74502Q -> LM74801-Q1; footprint Package_TO_SOT_SMD:TSOT-23-8_HandSoldering -> Package_SON:WSON-12-1EP_3x3mm_P0.5mm_EP1.5x2.5mm; symbol Power_Path_Custom:AP74502Q -> Power_Path_Custom:LM74801-Q1; DesignNote TBD -> Ortak-source: HGATE->Q5A (giris, R54/C30 yavas acilis, D6 k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; MPN AP74502Q -> LM74801QDRRRQ1; Manufacturer Power_Path_Custom -> Texas Instruments; Package TSOT-23-8 -> WSON-12 (DRR) 3x3; SelectionNote Özdisan (21.09.2026): Stokta yok. İdeal diyot kategorisi in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 -> Özdisan 1044371; stok 912 (22.09.2026); Uygun. AP74502Q sto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
Connections:
- net +3.3V: now also C35.1, U13.5 (VCC)
- net GATE_DRV: now also U12.8 (HGATE); no longer Q5.4 (G), U12.6 (GATE)
- net GND: now also U12.7 (GND), C35.2, R61.2, U13.3 (GND); no longer U12.2 (GND)
- net INA_ALERT: now also U13.2; no longer R58.1, U12.1 (EN/UVLO)
- net OUT_EN: now also R61.1, U13.1
- net OV_SENSE: now also U12.5 (OV); no longer U12.7 (OV)
- net SRC_COMMON: now also U12.2 (A), U12.9 (OUT); no longer U12.8 (SRC)
- net SW_OUT: now also U12.12 (C)
- net V_PRE: now also U12.10 (VS), U12.3 (VSNS), U12.4 (SW); no longer U12.5 (VS)
- net at C31.2: now also U12.11 (CAP); no longer U12.4 (VCAP)
- new net DGATE: Q5.4 (G), U12.1 (DGATE)
- new net SW_EN: R58.1, U12.6 (EN/UVLO), U13.4
Other:
- note added: "LM74801 CIKIS ANAHTARI + IDEAL DIYOT"
- note added: "U13: SW_EN = OUT_EN AND ~{ALERT} ALERT low -> U12 kapanir; R61 reset boyunca OUT_EN low."
- note removed: "AP74502Q CIKIS ANAHTARI"
- moved on the sheet: C32

Commit message: hardware: L1'i FPI0705-220K'ya geçir, U1/U2 tedarikini karara bağla (TASK-002)
L1 (AOZ1284 buck bobini): SRI0704-220M Özdisan'da stokta yok.
"Sabit İndüktörler" kategorisinde 22 µH taraması datasheet'lerle
karşılaştırıldı; FPI0705-220K seçildi (Özdisan 507505, stok 3467, 8,28 TL):
- 22 µH ±10%, RDC 0,11 Ω max (tasarımdakiyle aynı), IDC 1,95 -> 2,3 A.
- Gövde 7,3x7,3x4,5 -> 7,8x7,0x5,0 mm; yeni footprint
  Inductor_Custom:L_CoreMaster_FPI0705_7.8x7.0mm_H5.0 (land 7,5x3,25 mm
  iki ped, 2,0 mm boşluk; spec DWG MY0212071), fp-lib-table'a eklendi.
- Reddedilenler: TPY0705-220M (mevcut footprint'e uyuyor ama 0,35 Ω),
  SRI0704-330M (aynı ayak, 0,25 Ω / 1,2 A), FPI1005-220M (0,07 Ω / 3,4 A,
  10x9 mm), IHLP2525CZER220M11 (62 TL).

U1 AP33772S ve U2 ESP32-C6-WROOM-1: Özdisan'da yok, karşılayan muadil de
yok (ESP32-C3-MINI-1-N4 GPIO sayısı yetmiyor; ESP32-WROOM-32E-N4 native
USB yok). Mouser/DigiKey katalogundan alınacak.

Kararlar SelectionNote alanlarına işlendi. Doğrulama: ERC 0 hata / 0 uyarı,
netlist farkı YOK, field_geometry farkı boş.

Ayrıntı: design_decisions/output/PARCA_TEDARIK_KARARLARI_20260922.md
Kayıt: CHANGES.TXT REV_C. TASK-002 Done.

Ayrıca kicad-schematic SKILL.md: alan görünürlüğü assert örneğindeki
O(n^2) tuzağı düzeltildi (field_visibility döngü içinde çağrılıyordu;
gerçek betikte 3+ dakika sürüyordu).

Co-Authored-By: Claude Opus 5 <noreply@anthropic.com>
Parts:
- L1: footprint Inductor_SMD:L_7.3x7.3_H4.5 -> Inductor_Custom:L_CoreMaster_FPI0705_7.8x7.0mm_H5.0; DesignNote 22uH, 1.95A, 0.11ohm max; 1.95A'de 18.2uH (L -17%). -> 22uH +-10%, RDC 0.11 ohm max, IDC 2.3 A max (spec DWG MY021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; MPN SRI0704-220M -> FPI0705-220K; Manufacturer CORE MASTER -> Core Master; Package 7.3x7.3x4.5mm -> 7.8x7.0x5.0mm; SelectionNote Özdisan (21.09.2026): Stokta yok. 11.09 raporunda Özdisan s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 -> Özdisan 507505; stok 3467 (22.09.2026); Uygun. SRI0704-220M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
- U1: SelectionNote Özdisan (21.09.2026): Stokta yok. Özdisan indeksinde (stoks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 -> Özdisan (21.09.2026): stokta yok; 22.09.2026 indeksinde (st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
Changed lines of the file:
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@@
 			)
 		)
-		(property "SelectionNote" "Özdisan (21.09.2026): Stokta yok. Özdisan indeksinde (stoksuz dahil) bulunamadı. Başka tedarikçiden alınmalı."
+		(property "SelectionNote" "Özdisan (21.09.2026): stokta yok; 22.09.2026 indeksinde (stoksuz dahil) AP33772 hic gecmiyor. Karar: Mouser/DigiKey katalogundan alinacak (stok/fiyat satin alma oncesi dogrulanacak)."
 			(at 81.28 95.25 0)
 			(hide yes)
@@
 			)
 		)
-		(property "Footprint" "Inductor_SMD:L_7.3x7.3_H4.5"
+		(property "Footprint" "Inductor_Custom:L_CoreMaster_FPI0705_7.8x7.0mm_H5.0"
 			(at 281.94 191.77 0)
 			(hide yes)
@@
 			)
 		)
-		(property "Manufacturer" "CORE MASTER"
+		(property "Manufacturer" "Core Master"
 			(at 281.94 191.77 90)
 			(hide yes)
@@
 			)
 		)
-		(property "MPN" "SRI0704-220M"
+		(property "MPN" "FPI0705-220K"
 			(at 281.94 191.77 90)
 			(hide yes)
@@
 			)
 		)
-		(property "Package" "7.3x7.3x4.5mm"
+		(property "Package" "7.8x7.0x5.0mm"
 			(at 281.94 191.77 0)
 			(hide yes)
@@
 			)
 		)
-		(property "DesignNote" "22uH, 1.95A, 0.11ohm max; 1.95A'de 18.2uH (L -17%)."
+		(property "DesignNote" "22uH +-10%, RDC 0.11 ohm max, IDC 2.3 A max (spec DWG MY0212071). Tepe akim ~0.83 A (0.7 A yuk + dalga/2) -> 2.8x marj."
 			(at 281.94 191.77 0)
 			(hide yes)
@@
 			)
 		)
-		(property "SelectionNote" "Özdisan (21.09.2026): Stokta yok. 11.09 raporunda Özdisan stoklu seçilmişti; bugün indekste yok (aynı serinin başka değerleri stokta). Aynı ayağa uyan 22µH stokta yok. En yakını ETQP5M220YFM (22µH 3.7A, 7.5x7 mm, 434 stok); farklı footprint."
+		(property "SelectionNote" "Özdisan 507505; stok 3467 (22.09.2026); Uygun. SRI0704-220M stokta yok. Ayni ayaktaki SRI0704-330M (33uH) 0.25 ohm / 1.2 A ile DCR ve marji kotulestiriyordu; TPY0705-220M mevcut footprinte uyuyor ama 0.35 ohm. FPI0705-220K DCR-yi (0.11 ohm) korur, akimi 1.95 -> 2.3 A yukseltir, en ucuz (8.28 TL). Alternatif: FPI1005-220M (0.07 ohm / 3.4 A, 10x9 mm)."
 			(at 281.94 191.77 0)
 			(hide yes)

Commit message: hardware: L3 boost bobinini SRI0704-6R8M'e geçir (TASK-001)
Eski parça B82422H1682K000 (1210 çip) 6,8 µH ama yalnız 0,35 A / 570 mΩ
veriyordu; TPS55340 pre-boost'un tepe bobin akımı 1,24 A. Özdisan stoğu da
10 adete inmişti.

Gereksinim TPS55340 datasheet'iyle (SLVSBD4E, denk. 11-16) hesaplandı:
Vin(min) 3,3 V PPS, Vout 5,02 V, VD 0,45 V, fsw 600 kHz, V_PRE yükü 0,6 A
-> D 0,397, IL(ort) 1,07 A, dalgalanma 0,32 A, tepe 1,24 A. KIND 0,3 için
L(min) 6,78 µH; şemadaki 6,8 µH doğru değer, değiştirilmedi (kompanzasyon
aynen geçerli).

Seçilen: SRI0704-6R8M (Özdisan 587796, 15,05 TL, stok 657): 6,8 µH ±20%,
RDC 0,04 Ω max, IDC 3,5 A (tepe akımın 2,8 katı). Footprint 1210 ->
Inductor_SMD:L_7.3x7.3_H4.5 (KiCad'de hazır, yeni çizim gerekmedi).

Elenenler: FPI0705-100M (10 µH, 0,058 Ω / 3,4 A, 8,28 TL, L1 ile ortak
footprint) L değişimi RHP sıfırını %32 aşağı taşırdı; FPI0504-6R8M (2,7 A,
stok 108); SRI0605B-6R8M (0,08 Ω); 74437356068 (5,1 A ama stok 34).

Doğrulama: ERC 0 hata / 0 uyarı, netlist farkı YOK, field_geometry farkı boş.

Ayrıntı: design_decisions/output/PARCA_TEDARIK_KARARLARI_20260922.md
Kayıt: CHANGES.TXT REV_C. TASK-001 Done.

Co-Authored-By: Claude Opus 5 <noreply@anthropic.com>
Parts:
- L3: footprint Inductor_SMD:L_1210_3225Metric -> Inductor_SMD:L_7.3x7.3_H4.5; DCR TBD -> 40mOhm; DesignNote TBD -> TPS55340 pre-boost, 600 kHz, Vin(min) 3.3 V PPS -> V_PRE 5.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; MPN B82422H1682K000 -> SRI0704-6R8M; Manufacturer TDK (EPCOS) -> Core Master; Package 1210 (3225 Metric) -> 7.3x7.3x4.5mm; SelectionNote Özdisan 489001; stok 10 (21.09.2026); Uyarı. Footprint'e uy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 -> Özdisan 587796; stok 657 (23.09.2026); Uygun. B82422H1682K0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
Changed lines of the file:
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@@
 			)
 		)
-		(property "Footprint" "Inductor_SMD:L_1210_3225Metric"
+		(property "Footprint" "Inductor_SMD:L_7.3x7.3_H4.5"
 			(at 92.71 154.94 0)
 			(hide yes)
@@
 			)
 		)
-		(property "Manufacturer" "TDK (EPCOS)"
-			(at 92.71 154.94 0)
-			(hide yes)
-			(show_name no)
-			(do_not_autoplace no)
-			(effects
-				(font
-					(size 1.27 1.27)
-				)
-			)
-		)
-		(property "MPN" "B82422H1682K000"
-			(at 92.71 154.94 0)
-			(hide yes)
-			(show_name no)
-			(do_not_autoplace no)
-			(effects
-				(font
-					(size 1.27 1.27)
-				)
-			)
-		)
-		(property "Package" "1210 (3225 Metric)"
+		(property "Manufacturer" "Core Master"
+			(at 92.71 154.94 0)
+			(hide yes)
+			(show_name no)
+			(do_not_autoplace no)
+			(effects
+				(font
+					(size 1.27 1.27)
+				)
+			)
+		)
+		(property "MPN" "SRI0704-6R8M"
+			(at 92.71 154.94 0)
+			(hide yes)
+			(show_name no)
+			(do_not_autoplace no)
+			(effects
+				(font
+					(size 1.27 1.27)
+				)
+			)
+		)
+		(property "Package" "7.3x7.3x4.5mm"
 			(at 92.71 154.94 0)
 			(hide yes)
@@
 			)
 		)
-		(property "DesignNote" "TBD"
-			(at 92.71 154.94 0)
-			(hide yes)
-			(show_name no)
-			(do_not_autoplace no)
-			(effects
-				(font
-					(size 1.27 1.27)
-				)
-			)
-		)
-		(property "SelectionNote" "Özdisan 489001; stok 10 (21.09.2026); Uyarı. Footprint'e uyan tek parça. TPS55340 boost bobini için 1210 çip bobinin akımı (yüzlerce mA) yetersiz; tasarımda bobin/footprint kontrolü gerekli. Stok 10."
+		(property "DesignNote" "TPS55340 pre-boost, 600 kHz, Vin(min) 3.3 V PPS -> V_PRE 5.02 V, Iout 0.6 A. Datasheet denk. 11-16: D 0.397, IL(avg) 1.07 A, dalga 0.32 A, tepe 1.24 A; KIND 0.3 icin Lmin 6.78 uH -> 6.8 uH. IDC 3.5 A = 2.8x tepe. TPS55340 akim limiti 5.25-7.75 A; tam muhafazakar yaklasim (Isat > limit) bu kartta 12x12 mm bobin isterdi."
+			(at 92.71 154.94 0)
+			(hide yes)
+			(show_name no)
+			(do_not_autoplace no)
+			(effects
+				(font
+					(size 1.27 1.27)
+				)
+			)
+		)
+		(property "SelectionNote" "Özdisan 587796; stok 657 (23.09.2026); Uygun. B82422H1682K000 (1210) yalniz 0.35 A / 570 mOhm - tepe akimin (1.24 A) altinda, ayrica stok 10. Adaylar: FPI0705-100M (10 uH, 0.058 ohm / 3.4 A, 8.28 TL, L1 ile ortak footprint) L degisimi RHP sifirini %32 asagi tasiyacagi icin elendi; FPI0504-6R8M (0.065 ohm / 2.7 A, 5.64 TL, stok 108); SRI0605B-6R8M (0.08 ohm / 2.8 A); 74437356068 (5.1 A ama stok 34, 56 TL)."
 			(at 92.71 154.94 0)
 			(hide yes)
@@
 			)
 		)
-		(property "DCR" "TBD"
-			(at 92.71 154.94 0)
-			(hide yes)
+		(property "DCR" "40mOhm"
+			(at 92.71 154.94 0)
+			(hide yes)
