File: hardware/userinterface.kicad_sch (KiCad schematic)
At the start: 16 parts, among them J3 NHD-2.4-240320AF-CSXP, SW3 L-KLS4-EC1121S-E5A-F12.5, U7 TPS61023DRLR, U8 CAT4104V-GT3

Commit message: hardware: komponent alanlarını standarda oturt, yalnız Value+Reference göster
134 komponentin alan seti design_decisions/standards/komponent-field-standardi.csv
uyarınca yeniden kuruldu (3.144 alan). Her komponent grup koduna atandı ve ALL +
gruba özel alanlar standarttaki sırayla yazıldı; CSV'de koşullu işaretli alanlar
(Sadece Zener / Sadece ADC / Sadece RTC) yalnız ilgili parçaya kondu.

Eski alan adları standarda birleşti: Manufacturer Part Number ve DisplayMPN ->
MPN, Voltage -> VoltageRating, Field5 -> DesignNote / TerminationStyle,
Supplier + Battery -> SelectionNote / DesignNote. Sim.* alanları korundu.

Value IEC 60062 koduna çevrildi (10 kΩ/4,7k/100K/10kR karışıktı -> 10k/4k7/100k).
Value'dan çıkan gerilim, güç, tolerans ve dielektrik kendi alanlarına taşındı.
L1 ve D2'de Value MPN'di; parametrik değere çevrilip sipariş kodu MPN'e alındı.

Görünürlük tek kurala indi: yalnız Reference + Value. Description 119 sembolde
açıktı, kapandı. Güç sembolleri depo kuralına oturdu (Reference gizli, GND ve
PWR_FLAG değeri gizli, +3.3V görünür).

Parça verisi gerektiren 1.755 alan TBD bırakıldı; yalnız depodan (footprint,
lib_id, BOM_PRELIMINARY, tasarım notları) doğrulanabilen değerler yazıldı,
MPN veya datasheet parametresi uydurulmadı.

Okunabilirlik: C3 değeri PD_VBUS_SENSED telinin üstündeydi, TP5 referansı
PD_GATE etiketiyle çakışıyordu; ikisinin de yalnız metin konumu kaydırıldı.

gopo.kicad_pro'ya 10 çekirdek alanın Field Name Templates kaydı eklendi.

Bu commit ayrıca KiCad 10'un kendi kaydını taşır: güç sembollerinden
(fields_autoplaced no) düştü ve C4/TP4 elle boş alana taşındı.

Doğrulama: netlist farkı YOK, ERC 2 uyarı (değişmedi), lint 6/1/0/0 (değişmedi),
field_geometry farkı yalnız C3 ve TP5.

Co-Authored-By: Claude Opus 5 <noreply@anthropic.com>
Parts:
- C20, C21: value 22uF -> 22u; AssemblyNote (none) -> TBD; Category (none) -> Capacitors; DesignNote X7R; C12+C13 effective capacitance >=10uF at 28V; verify ac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 -> X7R.; Height (none) -> TBD; Lifecycle (none) -> TBD; MPN (none) -> TBD; Manufacturer (none) -> TBD; MountingType (none) -> Surface Mount; OperatingTemp (none) -> TBD; Package (none) -> 0402 (1005 Metric); RoHS (none) -> TBD; Subcategory (none) -> Ceramic Capacitors; Tolerance (none) -> TBD; Voltage 50V -> (none); VoltageRating 16V -> 50V
- C22: value 100nF / 16V -> 100n; AssemblyNote (none) -> TBD; Category (none) -> Capacitors; DesignNote X7R; C12+C13 effective capacitance >=10uF at 28V; verify ac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 -> X7R.; Dielectric (none) -> X7R; EffectiveCapacitance (none) -> TBD; Height (none) -> TBD; Lifecycle (none) -> TBD; MPN (none) -> TBD; Manufacturer (none) -> TBD; MountingType (none) -> Surface Mount; OperatingTemp (none) -> TBD; Package (none) -> 0402 (1005 Metric); RoHS (none) -> TBD; SelectionNote (none) -> TBD; Subcategory (none) -> Ceramic Capacitors; Tolerance (none) -> TBD; Voltage 50V -> (none); VoltageRating (none) -> 16V
- J3: AssemblyNote (none) -> TBD; Category (none) -> Connectors, Interconnects; ConnectorType (none) -> Receptacle; ContactPlating (none) -> TBD; CurrentRating (none) -> TBD; DesignNote (none) -> TFT modulu (NHD-2.4-240320AF-CSXP) bu konnektore takilir; m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; DisplayMPN NHD-2.4-240320AF-CSXP -> (none); Height (none) -> TBD; Lifecycle (none) -> TBD; MatingCycles (none) -> TBD; MountingType (none) -> Surface Mount; OperatingTemp (none) -> TBD; Orientation (none) -> TBD; Package (none) -> FPC 0.5mm 40-pos SMD; Pitch (none) -> 0.5mm; PositionCount (none) -> 40; RoHS (none) -> TBD; RowCount (none) -> 1; SelectionNote (none) -> TBD; Series (none) -> TBD; Shielding (none) -> TBD; Subcategory (none) -> -; VoltageRating (none) -> TBD
- L2: value 2.2uH -> 2u2; AssemblyNote (none) -> TBD; Category (none) -> Inductors, Coils, Chokes; CurrentRMS (none) -> TBD; CurrentSaturation (none) -> TBD; DCR (none) -> TBD; DesignNote Isat >=2A and Irms >=1.5A at max temperature; fault current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 -> Isat >=2A ve Irms >=1.5A (max sicaklikta) gerekir; ariza ak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; Height (none) -> TBD; Lifecycle (none) -> TBD; MountingType (none) -> Surface Mount; OperatingTemp (none) -> TBD; Package (none) -> MAPI-4030 (4.0x3.0mm); RoHS (none) -> TBD; SRF (none) -> TBD; SelectionNote (none) -> TBD; Shielding (none) -> TBD; Subcategory (none) -> Fixed Inductors; Tolerance (none) -> TBD
- R28, R34, R35, R36: AssemblyNote (none) -> TBD; Category (none) -> Resistors; Composition (none) -> TBD; DesignNote (none) -> TBD; Height (none) -> TBD; Lifecycle (none) -> TBD; MPN (none) -> TBD; Manufacturer (none) -> TBD; MountingType (none) -> Surface Mount; OperatingTemp (none) -> TBD; Package (none) -> 0402 (1005 Metric); PowerRating (none) -> TBD; RoHS (none) -> TBD; SelectionNote (none) -> TBD; Subcategory (none) -> Chip Resistor - Surface Mount; TempCoefficient (none) -> TBD; Tolerance (none) -> TBD; VoltageRating (none) -> TBD
- R29: value 100kR -> 100k; AssemblyNote (none) -> TBD; Category (none) -> Resistors; Composition (none) -> TBD; DesignNote (none) -> TBD; Height (none) -> TBD; Lifecycle (none) -> TBD; MPN (none) -> TBD; Manufacturer (none) -> TBD; MountingType (none) -> Surface Mount; OperatingTemp (none) -> TBD; Package (none) -> 0402 (1005 Metric); PowerRating (none) -> TBD; RoHS (none) -> TBD; SelectionNote (none) -> TBD; Subcategory (none) -> Chip Resistor - Surface Mount; TempCoefficient (none) -> TBD; Tolerance (none) -> TBD; VoltageRating (none) -> TBD
- R44: value 604kR 0.1% -> 604k; AssemblyNote (none) -> TBD; Category (none) -> Resistors; Composition (none) -> TBD; DesignNote (none) -> TBD; Height (none) -> TBD; Lifecycle (none) -> TBD; MPN (none) -> TBD; Manufacturer (none) -> TBD; MountingType (none) -> Surface Mount; OperatingTemp (none) -> TBD; Package (none) -> 0402 (1005 Metric); PowerRating (none) -> TBD; RoHS (none) -> TBD; SelectionNote (none) -> TBD; Subcategory (none) -> Chip Resistor - Surface Mount; TempCoefficient (none) -> TBD; Tolerance (none) -> +/-0.1%; VoltageRating (none) -> TBD
- R45: value 100kR 0.1% -> 100k; AssemblyNote (none) -> TBD; Category (none) -> Resistors; Composition (none) -> TBD; DesignNote (none) -> TBD; Height (none) -> TBD; Lifecycle (none) -> TBD; MPN (none) -> TBD; Manufacturer (none) -> TBD; MountingType (none) -> Surface Mount; OperatingTemp (none) -> TBD; Package (none) -> 0402 (1005 Metric); PowerRating (none) -> TBD; RoHS (none) -> TBD; SelectionNote (none) -> TBD; Subcategory (none) -> Chip Resistor - Surface Mount; TempCoefficient (none) -> TBD; Tolerance (none) -> +/-0.1%; VoltageRating (none) -> TBD
- R46: value 3.24kR 0.1% -> 3k24; AssemblyNote (none) -> TBD; Category (none) -> Resistors; Composition (none) -> TBD; DesignNote (none) -> TBD; Height (none) -> TBD; Lifecycle (none) -> TBD; MPN (none) -> TBD; Manufacturer (none) -> TBD; MountingType (none) -> Surface Mount; OperatingTemp (none) -> TBD; Package (none) -> 0402 (1005 Metric); PowerRating (none) -> TBD; RoHS (none) -> TBD; SelectionNote (none) -> TBD; Subcategory (none) -> Chip Resistor - Surface Mount; TempCoefficient (none) -> TBD; Tolerance (none) -> +/-0.1%; VoltageRating (none) -> TBD
- SW3: ActuationForce (none) -> TBD; AssemblyNote (none) -> TBD; Category (none) -> Switches; DesignNote (none) -> TBD; Detents (none) -> TBD; Function (none) -> Rotary Encoder with Switch; Height (none) -> TBD; Lifecycle (none) -> TBD; MPN (none) -> L-KLS4-EC1121S-E5A-F12.5; Manufacturer (none) -> KLS Electronic; MountingType (none) -> Through Hole; OperatingTemp (none) -> TBD; Package (none) -> EC1121S Vertical THT; PulsesPerRevolution (none) -> TBD; RoHS (none) -> TBD; RotationalLife (none) -> TBD; SelectionNote (none) -> BOM_PRELIMINARY_20260911 bu referans icin L-KLS4-EC12-01242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; ShaftLength (none) -> 12.5mm; ShaftType (none) -> TBD; Subcategory (none) -> Rotary Encoders / Tactile Switches; SwitchContactRating (none) -> TBD
- U7: AssemblyNote (none) -> TBD; Category (none) -> Integrated Circuits; ControlMode (none) -> TBD; DesignNote (none) -> TBD; Height (none) -> TBD; InputVoltage (none) -> TBD; IntegratedSwitch (none) -> TBD; InterfaceType (none) -> None; Lifecycle (none) -> TBD; MountingType (none) -> Surface Mount; OperatingTemp (none) -> TBD; OutputCurrent (none) -> TBD; OutputVoltage (none) -> TBD; Package (none) -> TBD; PinCount (none) -> TBD; RoHS (none) -> TBD; SelectionNote (none) -> TBD; Subcategory (none) -> PMIC - Voltage Regulators - DC DC Switching; SupplyVoltage (none) -> TBD; SwitchingFrequency (none) -> TBD; Synchronous (none) -> TBD; ThermalPad (none) -> TBD; Topology (none) -> Boost
- U8: AssemblyNote (none) -> TBD; Category (none) -> Integrated Circuits; ChannelCount (none) -> 4; ControlLogic (none) -> TBD; DesignNote (none) -> TBD; Height (none) -> TBD; InterfaceType (none) -> None; Lifecycle (none) -> TBD; MountingType (none) -> Surface Mount; OperatingTemp (none) -> TBD; OutputCurrent (none) -> TBD; Package (none) -> SOIC-8; PinCount (none) -> TBD; RoHS (none) -> TBD; SelectionNote (none) -> TBD; Subcategory (none) -> PMIC - LED Drivers; SupplyVoltage (none) -> TBD; ThermalPad (none) -> TBD

Commit message: hardware: RTC'yi BQ32000 + süper kapasitöre geçir, Özdisan BOM'unu şemaya aktar
RTC (mcu):
- U4 RV-3028-C7 -> BQ32000DR (SOIC-8, I2C 0x68, open-drain IRQ, dahili
  trickle charger). Y1 ABS25-32.768KHZ-T (CL 12,5 pF, harici yük C yok),
  C33 Korchip DCL5R5155HF 1,5 F/5,5 V (H-tipi yatay coin, ~22 gün yedek).
- BT1 (CR2032), R22, R23, C10 kaldırıldı; C9 100n -> 1u0 (datasheet >= 1 uF).
- Yeni footprint: Power_Output_Custom:Korchip_DCL_H-Type_D19.0mm_P20.00mm_Horizontal
  (Korchip DCL datasheet çiziminden; numune ile doğrulanmalı).
- Beklenen netlist farkı yalnız RTC netleri: RTC_SCL/SDA/INT U4 pin
  numaraları, Net-(U4-OSCI/OSCO/VBACK) yeni; Net-(BT1-+), Net-(U4-EVI),
  Net-(U4-VBACKUP), U4 CLKOUT kalktı. ERC değişmedi (0 hata, 2 eski uyarı).

Özdisan BOM aktarımı (tüm sayfalar):
- MPN, Manufacturer, parametrik alanlar ve SelectionNote (Özdisan kodu,
  stok 21.09.2026, durum) BOM_OZDISAN_REV_C_20260921.xlsx'ten yazıldı.
- Onaylı değişiklikler: C5/C20/C21 0805; C8/C12/C13/C25/C27/C28 4u7 50V
  X7R 1210; C15/C29 47u 35V hibrit (Device:C_Polarized, CP_Elec_6.3x5.8);
  C31 0603 25V; R59 0805 1/3W; R40 3k24 + R39 10k2 (VOUT 3,3185 V);
  U6 TL431AIDBZR; D4 SX36.
- Stokta olmayan parçalarda (U1, U2, U7, U8, U10, U12, L1, L2, C19) MPN
  korundu, öneri SelectionNote ve todo.txt'de. Alan geometrisi ve
  görünürlük değişmedi. PCB şemadan henüz güncellenmedi.

Aynı commit'te önceden commit edilmemiş çalışma: Q3/Q5 SQJB60EP ve U3
INA226 entegrasyonu, raporları ve datasheet'leri.

Co-Authored-By: Claude Opus 5 <noreply@anthropic.com>
Parts:
- C20, C21: footprint Capacitor_SMD:C_0402_1005Metric -> Capacitor_SMD:C_0805_2012Metric; Dielectric X7R -> X6S; MPN TBD -> GRT21BC81A226ME13K; Manufacturer TBD -> Murata; Package 0402 (1005 Metric) -> 0805 (2012 Metric); SelectionNote Verify DC-bias curve for final capacitor MPN -> Özdisan 810882; stok 709 (21.09.2026); Uygun. 21.09 üçüncü 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; Tolerance TBD -> +/-20%; VoltageRating 50V -> 10V
- C22: MPN TBD -> CC0402KRX7R9BB104; Manufacturer TBD -> Yageo; SelectionNote TBD -> Özdisan 609906; stok 117450 (21.09.2026); Uygun. Tek MPN: C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; Tolerance TBD -> +/-10%; VoltageRating 16V -> 50V
- J3: SelectionNote TBD -> Özdisan 1325143; stok 13297 (21.09.2026); Uygun. 21.09 ikin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
- L2: SelectionNote TBD -> Özdisan (21.09.2026): Stokta yok. Özdisan'da bulunamadı. MA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
- R28: Composition TBD -> Thin Film; MPN TBD -> TC0250B1000TCC; Manufacturer TBD -> Royalohm; PowerRating TBD -> 0.0625W; SelectionNote TBD -> Özdisan 569711; stok 7445 (21.09.2026); Uygun.; TempCoefficient TBD -> +/-50ppm/C; Tolerance TBD -> +/-0.1%; VoltageRating TBD -> 25V
- R29: Composition TBD -> Thick Film; MPN TBD -> CQ02WGF1003TCE; Manufacturer TBD -> Royalohm; PowerRating TBD -> 0.0625W; SelectionNote TBD -> Özdisan 587906; stok 99900 (21.09.2026); Uygun.; TempCoefficient TBD -> +/-100ppm/C; Tolerance TBD -> +/-1%; VoltageRating TBD -> 50V
- R34, R35, R36: Composition TBD -> Thin Film; MPN TBD -> TC0250B1002TCC; Manufacturer TBD -> Royalohm; PowerRating TBD -> 0.0625W; SelectionNote TBD -> Özdisan 569744; stok 4220 (21.09.2026); Uygun. Özdisan'da 0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; TempCoefficient TBD -> +/-50ppm/C; Tolerance TBD -> +/-0.1%; VoltageRating TBD -> 25V
- R44: Composition TBD -> Thick Film; MPN TBD -> 0402WGF6043TCE; Manufacturer TBD -> Royalohm; PowerRating TBD -> 0.0625W; SelectionNote TBD -> Özdisan 506466; stok 42500 (21.09.2026); Uygun. 21.09 üçünc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; TempCoefficient TBD -> +/-100ppm/C; Tolerance +/-0.1% -> +/-1%; VoltageRating TBD -> 50V
- R45: Composition TBD -> Thin Film; MPN TBD -> TC0250B1003TCC; Manufacturer TBD -> Royalohm; PowerRating TBD -> 0.0625W; SelectionNote TBD -> Özdisan 569693; stok 368 (21.09.2026); Uygun. %0,1 şartı (B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; TempCoefficient TBD -> +/-50ppm/C; VoltageRating TBD -> 25V
- R46: Composition TBD -> Precision Thick Film; MPN TBD -> ERJ2RKF3241X; Manufacturer TBD -> Panasonic; PowerRating TBD -> 0.1W; SelectionNote TBD -> Özdisan 494659; stok 76745 (21.09.2026); Uygun. 21.09 üçünc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; TempCoefficient TBD -> +/-100ppm/C; Tolerance +/-0.1% -> +/-1%; VoltageRating TBD -> 50V
- SW3: SelectionNote BOM_PRELIMINARY_20260911 bu referans icin L-KLS4-EC12-01242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 -> Özdisan 533942; stok 1013 (21.09.2026); Uygun. Şema sembolü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
- U7: MPN TPS61023DRLR -> RT4812GJ8F; Manufacturer Texas Instruments -> RICHTEK; SelectionNote TBD -> Özdisan 614996; stok 308 (21.09.2026); Muadil. 21.09 üçüncü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
- U8: SelectionNote TBD -> Özdisan (21.09.2026): Stokta yok. Özdisan indeksinde buluna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
