File: hardware/userinterface.kicad_sch (KiCad schematic)
At the start: 10 parts, among them J3 TFT032B018, Q7 IRLML6344, SW3 L-KLS4-EC1121S-E5A-F12.5

Commit message: PCB tasarimi guncellendi
Parts:
- added J9: ENCODER CABLE, Connector_Wire:SolderWire-0.25sqmm_1x05_P4.2mm_D0.65mm_OD1.7mm, symbol Connector_Generic:Conn_01x05
- SW3: footprint L-KLS4-EC1121S-E5A-F12.5:L-KLS4-EC1121S-E5A-F12.5 -> (none); DesignNote TBD -> TASK-066: panel-mounted encoder, five wires to J9; pin 1=A,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; Mounting (none) -> Panel; housing retained by enclosure bracket; not soldered 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
Connections:
- net ENCODER_A: now also J9.1 (Pin_1)
- net ENCODER_B: now also J9.3 (Pin_3)
- net ENCODER_SW: now also J9.4 (Pin_4)
- net GND: now also J9.2 (Pin_2), J9.5 (Pin_5)
Other:
- note added: "1=A 2=C/GND 3=B 4=S1 5=S2/GND 5 x 0.14mm2 stranded wire, length <=150mm. Solder pads only; enclosure provides strain relief. Insulated knob; keep cable away from switching nodes. Firmware: quadrature state validation + switch debounce."
- note added: "A=GPIO22, B=GPIO23, SW=GPIO21. R34-R36: 10k pull-ups on PCB; no RC fitted. SW3: panel mounted, five wires to J9 below."
- note added: "ENCODER: SW3 PANEL / PULL-UPS PCB"
- note added: "PCB WIRE PADS - J9"
- note removed: "ENCODER: A=GPIO22, B=GPIO23, SW=GPIO21 3.3V pull-ups; contacts close to GND. Firmware: quadrature state decoding and switch debounce required."
- note removed: "ROTARY ENCODER"
