File: hardware/mcu.kicad_sch (KiCad schematic)
At the start: 30 parts, among them SW1 BOOT / PTS810, SW2 RESET / PTS810, U2 ESP32-C6-WROOM-1, U4 RV-3028-C7

Commit message: usb_pd_controller: tüm güç zincirini tek A3 sayfasında topla
powergeneration (TPS55340 ön-boost + AOZ1284 buck) ve poweroutput (panel
konnektörleri) blokları bu sayfaya taşındı. Sayfa A2'den A3'e indirildi;
bloklar altı slota yeniden çizildi:
  satır 1: PD kontrolcü + VBUS şönt/anahtar | AP74502Q çıkış anahtarı |
           INA228 ölçüm + panel çıkışı (TVS ve boşaltma direnci dahil)
  satır 2: TPS55340 ön-boost | AOZ1284 buck | I2C seviye dönüştürücü

Okunurluk için: buck bloğu iki satıra bölünüp sütun aralıkları 12.7 mm'ye
çıkarıldı, PD kontrolcüde V5V rayı kapı hattının üstüne alındı, INA228 ile
panel konnektörleri tek blokta birleşti, V_PRE artık ön-boost çıkışından
buck girişine gerçek telle gidiyor.

Boş kalan sayfalar silindi: powergeneration, poweroutput, powersensing,
calc_usb_pd_controller, CALC_MCU, CALC_USB_C_INPUT (sayfa sembolleri ve
gopo.kicad_pro kayıtları dahil). Şematik 12 sayfadan 6 sayfaya indi.

Bağlantılar isimden bağımsız karşılaştırmayla doğrulandı: kayıp/yeni net
yok; yalnızca sayfa kapsamı değişen 9 net yeniden adlandı
(/POWER GENERATION/* -> /USB_PD_CONTROLLER/*). ERC değişmedi
(0 hata, 2 eski uyarı), lint temiz.

Co-Authored-By: Claude Opus 5 <noreply@anthropic.com>
Other:
- removed sheet CALC_MCU
Changed lines of the file:
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@@
-		)
-	)
-	(sheet
-		(at 15.24 183.515)
-		(size 12.7 10.16)
-		(exclude_from_sim no)
-		(in_bom yes)
-		(on_board yes)
-		(dnp no)
-		(fields_autoplaced yes)
-		(stroke
-			(width 0.1524)
-			(type solid)
-		)
-		(fill
-			(color 255 95 239 1)
-		)
-		(property "Sheetname" "CALC_MCU"
-			(at 15.24 182.8034 0)
-			(show_name no)
-			(do_not_autoplace no)
-			(effects
-				(font
-					(size 1.27 1.27)
-				)
-				(justify left bottom)
-			)
-		)
-		(property "Sheetfile" "CALC_MCU.kicad_sch"
-			(at 15.24 194.2596 0)
-			(show_name no)
-			(do_not_autoplace no)
-			(effects
-				(font
-					(size 1.27 1.27)
-				)
-				(justify left top)
-			)
-		)
-		(property "Field2" ""
-			(at 15.24 183.515 0)
-			(hide yes)
-			(show_name no)
-			(do_not_autoplace no)
-			(effects
-				(font
-					(size 1.27 1.27)
-				)
-			)
-		)
-		(instances
-			(project "gopo"
-				(path "/a43081a6-9aa2-4898-9347-bbcb5849dafd/d73c21d5-7478-4a02-ac94-6607c580f283"
-					(page "11")
-				)
-			)
 		)
 	)

Commit message: hardware: komponent alanlarını standarda oturt, yalnız Value+Reference göster
134 komponentin alan seti design_decisions/standards/komponent-field-standardi.csv
uyarınca yeniden kuruldu (3.144 alan). Her komponent grup koduna atandı ve ALL +
gruba özel alanlar standarttaki sırayla yazıldı; CSV'de koşullu işaretli alanlar
(Sadece Zener / Sadece ADC / Sadece RTC) yalnız ilgili parçaya kondu.

Eski alan adları standarda birleşti: Manufacturer Part Number ve DisplayMPN ->
MPN, Voltage -> VoltageRating, Field5 -> DesignNote / TerminationStyle,
Supplier + Battery -> SelectionNote / DesignNote. Sim.* alanları korundu.

Value IEC 60062 koduna çevrildi (10 kΩ/4,7k/100K/10kR karışıktı -> 10k/4k7/100k).
Value'dan çıkan gerilim, güç, tolerans ve dielektrik kendi alanlarına taşındı.
L1 ve D2'de Value MPN'di; parametrik değere çevrilip sipariş kodu MPN'e alındı.

Görünürlük tek kurala indi: yalnız Reference + Value. Description 119 sembolde
açıktı, kapandı. Güç sembolleri depo kuralına oturdu (Reference gizli, GND ve
PWR_FLAG değeri gizli, +3.3V görünür).

Parça verisi gerektiren 1.755 alan TBD bırakıldı; yalnız depodan (footprint,
lib_id, BOM_PRELIMINARY, tasarım notları) doğrulanabilen değerler yazıldı,
MPN veya datasheet parametresi uydurulmadı.

Okunabilirlik: C3 değeri PD_VBUS_SENSED telinin üstündeydi, TP5 referansı
PD_GATE etiketiyle çakışıyordu; ikisinin de yalnız metin konumu kaydırıldı.

gopo.kicad_pro'ya 10 çekirdek alanın Field Name Templates kaydı eklendi.

Bu commit ayrıca KiCad 10'un kendi kaydını taşır: güç sembollerinden
(fields_autoplaced no) düştü ve C4/TP4 elle boş alana taşındı.

Doğrulama: netlist farkı YOK, ERC 2 uyarı (değişmedi), lint 6/1/0/0 (değişmedi),
field_geometry farkı yalnız C3 ve TP5.

Co-Authored-By: Claude Opus 5 <noreply@anthropic.com>
Parts:
- BT1: AssemblyNote (none) -> TBD; Battery CR2032 3V PRIMARY; cell purchased separately; RTC trickle c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 -> (none); BatteryType (none) -> CR2032; Capacity (none) -> TBD; Category (none) -> Battery Products; CellSize (none) -> CR2032; Chemistry (none) -> Lithium Manganese Dioxide; DesignNote (none) -> CR2032 3V primary; hucre ayri satin alinir. RTC trickle cha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; Height (none) -> TBD; HolderMounting (none) -> Surface Mount; Lifecycle (none) -> TBD; MountingType (none) -> Surface Mount; NominalVoltage (none) -> 3V; OperatingTemp (none) -> TBD; Package (none) -> CR2032 Holder SMD; RoHS (none) -> TBD; SelectionNote (none) -> Tedarik: Ozdisan 497433; Subcategory (none) -> Batteries / Battery Holders; Supplier Ozdisan 497433 -> (none)
- C10, C6, C9: value 100nF -> 100n; AssemblyNote (none) -> TBD; Category (none) -> Capacitors; DesignNote (none) -> TBD; Dielectric (none) -> TBD; EffectiveCapacitance (none) -> TBD; Height (none) -> TBD; Lifecycle (none) -> TBD; MPN (none) -> TBD; Manufacturer (none) -> TBD; MountingType (none) -> Surface Mount; OperatingTemp (none) -> TBD; Package (none) -> 0402 (1005 Metric); RoHS (none) -> TBD; SelectionNote (none) -> TBD; Subcategory (none) -> Ceramic Capacitors; Tolerance (none) -> TBD; VoltageRating (none) -> TBD
- C5: value 22uF -> 22u; AssemblyNote (none) -> TBD; Category (none) -> Capacitors; DesignNote (none) -> TBD; Dielectric (none) -> TBD; EffectiveCapacitance (none) -> TBD; Height (none) -> TBD; Lifecycle (none) -> TBD; MPN (none) -> TBD; Manufacturer (none) -> TBD; MountingType (none) -> Surface Mount; OperatingTemp (none) -> TBD; Package (none) -> 0402 (1005 Metric); RoHS (none) -> TBD; SelectionNote (none) -> TBD; Subcategory (none) -> Ceramic Capacitors; Tolerance (none) -> TBD; VoltageRating (none) -> TBD
- C7: value 1uF -> 1u0; AssemblyNote (none) -> TBD; Category (none) -> Capacitors; DesignNote (none) -> TBD; Dielectric (none) -> TBD; EffectiveCapacitance (none) -> TBD; Height (none) -> TBD; Lifecycle (none) -> TBD; MPN (none) -> TBD; Manufacturer (none) -> TBD; MountingType (none) -> Surface Mount; OperatingTemp (none) -> TBD; Package (none) -> 0402 (1005 Metric); RoHS (none) -> TBD; SelectionNote (none) -> TBD; Subcategory (none) -> Ceramic Capacitors; Tolerance (none) -> TBD; VoltageRating (none) -> TBD
- R1: value 10 kΩ -> 10k; AssemblyNote (none) -> TBD; Category (none) -> Resistors; Composition (none) -> TBD; DesignNote (none) -> TBD; Height (none) -> TBD; Lifecycle (none) -> TBD; MPN (none) -> TBD; Manufacturer (none) -> TBD; MountingType (none) -> Surface Mount; OperatingTemp (none) -> TBD; Package (none) -> 0402 (1005 Metric); PowerRating (none) -> TBD; RoHS (none) -> TBD; SelectionNote (none) -> TBD; Subcategory (none) -> Chip Resistor - Surface Mount; TempCoefficient (none) -> TBD; Tolerance (none) -> TBD; VoltageRating (none) -> TBD
- R10, R16, R23: AssemblyNote (none) -> TBD; Category (none) -> Resistors; Composition (none) -> TBD; DesignNote (none) -> TBD; Height (none) -> TBD; Lifecycle (none) -> TBD; MPN (none) -> TBD; Manufacturer (none) -> TBD; MountingType (none) -> Surface Mount; OperatingTemp (none) -> TBD; Package (none) -> 0402 (1005 Metric); PowerRating (none) -> TBD; RoHS (none) -> TBD; SelectionNote (none) -> TBD; Subcategory (none) -> Chip Resistor - Surface Mount; TempCoefficient (none) -> TBD; Tolerance (none) -> TBD; VoltageRating (none) -> TBD
- R15: value 22 R -> 22R; AssemblyNote (none) -> TBD; Category (none) -> Resistors; Composition (none) -> TBD; DesignNote (none) -> TBD; Height (none) -> TBD; Lifecycle (none) -> TBD; MPN (none) -> TBD; Manufacturer (none) -> TBD; MountingType (none) -> Surface Mount; OperatingTemp (none) -> TBD; Package (none) -> 0402 (1005 Metric); PowerRating (none) -> TBD; RoHS (none) -> TBD; SelectionNote (none) -> TBD; Subcategory (none) -> Chip Resistor - Surface Mount; TempCoefficient (none) -> TBD; Tolerance (none) -> TBD; VoltageRating (none) -> TBD
- R2, R3: value 22Ω -> 22R; AssemblyNote (none) -> TBD; Category (none) -> Resistors; Composition (none) -> TBD; DesignNote (none) -> TBD; Height (none) -> TBD; Lifecycle (none) -> TBD; MPN (none) -> TBD; Manufacturer (none) -> TBD; MountingType (none) -> Surface Mount; OperatingTemp (none) -> TBD; Package (none) -> 0402 (1005 Metric); PowerRating (none) -> TBD; RoHS (none) -> TBD; SelectionNote (none) -> TBD; Subcategory (none) -> Chip Resistor - Surface Mount; TempCoefficient (none) -> TBD; Tolerance (none) -> TBD; VoltageRating (none) -> TBD
- R22: value 1K -> 1k0; AssemblyNote (none) -> TBD; Category (none) -> Resistors; Composition (none) -> TBD; DesignNote (none) -> TBD; Height (none) -> TBD; Lifecycle (none) -> TBD; MPN (none) -> TBD; Manufacturer (none) -> TBD; MountingType (none) -> Surface Mount; OperatingTemp (none) -> TBD; Package (none) -> 0402 (1005 Metric); PowerRating (none) -> TBD; RoHS (none) -> TBD; SelectionNote (none) -> TBD; Subcategory (none) -> Chip Resistor - Surface Mount; TempCoefficient (none) -> TBD; Tolerance (none) -> TBD; VoltageRating (none) -> TBD
- R24: value 4,7k -> 4k7; AssemblyNote (none) -> TBD; Category (none) -> Resistors; Composition (none) -> TBD; DesignNote (none) -> TBD; Height (none) -> TBD; Lifecycle (none) -> TBD; MPN (none) -> TBD; Manufacturer (none) -> TBD; MountingType (none) -> Surface Mount; OperatingTemp (none) -> TBD; Package (none) -> 0402 (1005 Metric); PowerRating (none) -> TBD; RoHS (none) -> TBD; SelectionNote (none) -> TBD; Subcategory (none) -> Chip Resistor - Surface Mount; TempCoefficient (none) -> TBD; Tolerance (none) -> TBD; VoltageRating (none) -> TBD
- R25: value 4.7k -> 4k7; AssemblyNote (none) -> TBD; Category (none) -> Resistors; Composition (none) -> TBD; DesignNote (none) -> TBD; Height (none) -> TBD; Lifecycle (none) -> TBD; MPN (none) -> TBD; Manufacturer (none) -> TBD; MountingType (none) -> Surface Mount; OperatingTemp (none) -> TBD; Package (none) -> 0402 (1005 Metric); PowerRating (none) -> TBD; RoHS (none) -> TBD; SelectionNote (none) -> TBD; Subcategory (none) -> Chip Resistor - Surface Mount; TempCoefficient (none) -> TBD; Tolerance (none) -> TBD; VoltageRating (none) -> TBD
- R26: value 4.7K -> 4k7; AssemblyNote (none) -> TBD; Category (none) -> Resistors; Composition (none) -> TBD; DesignNote (none) -> TBD; Height (none) -> TBD; Lifecycle (none) -> TBD; MPN (none) -> TBD; Manufacturer (none) -> TBD; MountingType (none) -> Surface Mount; OperatingTemp (none) -> TBD; Package (none) -> 0402 (1005 Metric); PowerRating (none) -> TBD; RoHS (none) -> TBD; SelectionNote (none) -> TBD; Subcategory (none) -> Chip Resistor - Surface Mount; TempCoefficient (none) -> TBD; Tolerance (none) -> TBD; VoltageRating (none) -> TBD
- R37: value 10kR -> 10k; AssemblyNote (none) -> TBD; Category (none) -> Resistors; Composition (none) -> TBD; DesignNote (none) -> TBD; Height (none) -> TBD; Lifecycle (none) -> TBD; MPN (none) -> TBD; Manufacturer (none) -> TBD; MountingType (none) -> Surface Mount; OperatingTemp (none) -> TBD; Package (none) -> 0402 (1005 Metric); PowerRating (none) -> TBD; RoHS (none) -> TBD; SelectionNote (none) -> TBD; Subcategory (none) -> Chip Resistor - Surface Mount; TempCoefficient (none) -> TBD; Tolerance (none) -> TBD; VoltageRating (none) -> TBD
- SW1: ActuationForce (none) -> TBD; AssemblyNote (none) -> TBD; Category (none) -> Switches; DesignNote (none) -> BOOT butonu; 4.2x3.2 mm SMD. Tedarik: Ozdisan.; Detents (none) -> TBD; Function (none) -> Tactile Switch, SPST-NO; Height (none) -> TBD; Lifecycle (none) -> TBD; MPN (none) -> PTS810 SJS 250 SMTR LFS; Manufacturer (none) -> C&K; MountingType (none) -> Surface Mount; OperatingTemp (none) -> TBD; Package (none) -> PTS810 SMD (4.2x3.2mm); PulsesPerRevolution (none) -> TBD; RoHS (none) -> TBD; RotationalLife (none) -> TBD; SelectionNote (none) -> TBD; ShaftLength (none) -> TBD; ShaftType (none) -> TBD; Subcategory (none) -> Rotary Encoders / Tactile Switches; SwitchContactRating (none) -> TBD
- SW2: ActuationForce (none) -> TBD; AssemblyNote (none) -> TBD; Category (none) -> Switches; DesignNote (none) -> RESET butonu; 4.2x3.2 mm SMD. Tedarik: Ozdisan.; Detents (none) -> TBD; Function (none) -> Tactile Switch, SPST-NO; Height (none) -> TBD; Lifecycle (none) -> TBD; MPN (none) -> PTS810 SJS 250 SMTR LFS; Manufacturer (none) -> C&K; MountingType (none) -> Surface Mount; OperatingTemp (none) -> TBD; Package (none) -> PTS810 SMD (4.2x3.2mm); PulsesPerRevolution (none) -> TBD; RoHS (none) -> TBD; RotationalLife (none) -> TBD; SelectionNote (none) -> TBD; ShaftLength (none) -> TBD; ShaftType (none) -> TBD; Subcategory (none) -> Rotary Encoders / Tactile Switches; SwitchContactRating (none) -> TBD
- TP10, TP11, TP12, TP13, TP6, TP7, TP8, TP9: AssemblyNote (none) -> TBD; Category (none) -> Test and Measurement; DesignNote (none) -> 1.0 mm SMD test pedi; satin alinan parca degildir.; HardwareType (none) -> Test Point; Height (none) -> TBD; Lifecycle (none) -> N/A; MPN (none) -> N/A; Manufacturer (none) -> N/A; MountingType (none) -> Surface Mount; OperatingTemp (none) -> TBD; Package (none) -> SMD Pad D1.0mm; PadDiameter (none) -> 1.0mm; RoHS (none) -> N/A; SelectionNote (none) -> TBD; Subcategory (none) -> Test Points
- U2: AntennaType (none) -> PCB Trace; AssemblyNote (none) -> TBD; Category (none) -> Integrated Circuits; Certification (none) -> TBD; ClockFrequency (none) -> TBD; CoreArchitecture (none) -> RISC-V 32-bit; DesignNote (none) -> Modul varyanti / flash kapasitesi satin alma oncesi sabitle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; FlashSize (none) -> TBD; Height (none) -> TBD; IOCount (none) -> TBD; InterfaceType (none) -> TBD; Lifecycle (none) -> TBD; ModuleDimensions (none) -> 18x25.5x3.1mm; MountingType (none) -> Surface Mount; OperatingTemp (none) -> TBD; Package (none) -> WROOM-1 Module (18x25.5mm); PeripheralInterfaces (none) -> TBD; PinCount (none) -> TBD; RAMSize (none) -> TBD; RoHS (none) -> TBD; SelectionNote (none) -> TBD; Subcategory (none) -> Embedded - Microcontrollers / RF Modules; SupplyVoltage (none) -> TBD; ThermalPad (none) -> TBD; WirelessProtocol (none) -> TBD
- U4: AssemblyNote (none) -> TBD; Category (none) -> Integrated Circuits; ChannelCount (none) -> TBD; DesignNote (none) -> Trickle charge kapali kullanilacak.; Function (none) -> RTC, I2C; Height (none) -> TBD; InterfaceType (none) -> I2C; Lifecycle (none) -> TBD; LogicFamily (none) -> TBD; MountingType (none) -> Surface Mount; OperatingTemp (none) -> TBD; OutputType (none) -> TBD; Package (none) -> C7 SON-8 (1.5x3.2mm); PinCount (none) -> TBD; RoHS (none) -> TBD; SelectionNote (none) -> TBD; Subcategory (none) -> Logic / Memory / Clock-Timing; SupplyVoltage (none) -> TBD; ThermalPad (none) -> TBD; TimekeepingAccuracy (none) -> TBD

Commit message: hardware: RTC'yi BQ32000 + süper kapasitöre geçir, Özdisan BOM'unu şemaya aktar
RTC (mcu):
- U4 RV-3028-C7 -> BQ32000DR (SOIC-8, I2C 0x68, open-drain IRQ, dahili
  trickle charger). Y1 ABS25-32.768KHZ-T (CL 12,5 pF, harici yük C yok),
  C33 Korchip DCL5R5155HF 1,5 F/5,5 V (H-tipi yatay coin, ~22 gün yedek).
- BT1 (CR2032), R22, R23, C10 kaldırıldı; C9 100n -> 1u0 (datasheet >= 1 uF).
- Yeni footprint: Power_Output_Custom:Korchip_DCL_H-Type_D19.0mm_P20.00mm_Horizontal
  (Korchip DCL datasheet çiziminden; numune ile doğrulanmalı).
- Beklenen netlist farkı yalnız RTC netleri: RTC_SCL/SDA/INT U4 pin
  numaraları, Net-(U4-OSCI/OSCO/VBACK) yeni; Net-(BT1-+), Net-(U4-EVI),
  Net-(U4-VBACKUP), U4 CLKOUT kalktı. ERC değişmedi (0 hata, 2 eski uyarı).

Özdisan BOM aktarımı (tüm sayfalar):
- MPN, Manufacturer, parametrik alanlar ve SelectionNote (Özdisan kodu,
  stok 21.09.2026, durum) BOM_OZDISAN_REV_C_20260921.xlsx'ten yazıldı.
- Onaylı değişiklikler: C5/C20/C21 0805; C8/C12/C13/C25/C27/C28 4u7 50V
  X7R 1210; C15/C29 47u 35V hibrit (Device:C_Polarized, CP_Elec_6.3x5.8);
  C31 0603 25V; R59 0805 1/3W; R40 3k24 + R39 10k2 (VOUT 3,3185 V);
  U6 TL431AIDBZR; D4 SX36.
- Stokta olmayan parçalarda (U1, U2, U7, U8, U10, U12, L1, L2, C19) MPN
  korundu, öneri SelectionNote ve todo.txt'de. Alan geometrisi ve
  görünürlük değişmedi. PCB şemadan henüz güncellenmedi.

Aynı commit'te önceden commit edilmemiş çalışma: Q3/Q5 SQJB60EP ve U3
INA226 entegrasyonu, raporları ve datasheet'leri.

Co-Authored-By: Claude Opus 5 <noreply@anthropic.com>
Parts:
- removed BT1: CR2032 holder, Power_Output_Custom:KLS_CR2032_05, symbol Device:Battery_Cell
- removed C10: 100n, Capacitor_SMD:C_0402_1005Metric, symbol Device:C
- removed R22: 1k0, Resistor_SMD:R_0402_1005Metric, symbol Device:R
- removed R23: 10k, Resistor_SMD:R_0402_1005Metric, symbol Device:R
- added C33: 1F5, Power_Output_Custom:Korchip_DCL_H-Type_D19.0mm_P20.00mm_Horizontal, symbol Device:C_Polarized
- added Y1: 32.768kHz, Crystal:Crystal_SMD_Abracon_ABS25-4Pin_8.0x3.8mm, symbol Device:Crystal_GND23
- C5: footprint Capacitor_SMD:C_0402_1005Metric -> Capacitor_SMD:C_0805_2012Metric; Dielectric TBD -> X6S; MPN TBD -> GRT21BC81A226ME13K; Manufacturer TBD -> Murata; Package 0402 (1005 Metric) -> 0805 (2012 Metric); SelectionNote TBD -> Özdisan 810882; stok 709 (21.09.2026); Uygun. 21.09 üçüncü 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; Tolerance TBD -> +/-20%; VoltageRating TBD -> 10V
- C6: Dielectric TBD -> X7R; MPN TBD -> CC0402KRX7R9BB104; Manufacturer TBD -> Yageo; SelectionNote TBD -> Özdisan 609906; stok 117450 (21.09.2026); Uygun. Tek MPN: C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; Tolerance TBD -> +/-10%; VoltageRating TBD -> 50V
- C7: Dielectric TBD -> X5R; MPN TBD -> EMK105BJ105KVHF; Manufacturer TBD -> Taiyo Yuden; SelectionNote TBD -> Özdisan 623573; stok 5005 (21.09.2026); Uygun. C4 (PD_5V) i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; Tolerance TBD -> +/-10%; VoltageRating TBD -> 16V
- C9: value 100n -> 1u0; DesignNote TBD -> BQ32000 VCC dekuplaji; datasheet >=1uF seramik, VCC/GND pin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; Dielectric TBD -> X5R; MPN TBD -> EMK105BJ105KVHF; Manufacturer TBD -> Taiyo Yuden; SelectionNote TBD -> Özdisan 623573; stok 5005 (21.09.2026); Uygun. C4 (PD_5V) i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; Tolerance TBD -> +/-10%; VoltageRating TBD -> 16V
- R1, R10, R37: Composition TBD -> Thin Film; MPN TBD -> TC0250B1002TCC; Manufacturer TBD -> Royalohm; PowerRating TBD -> 0.0625W; SelectionNote TBD -> Özdisan 569744; stok 4220 (21.09.2026); Uygun. Özdisan'da 0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; TempCoefficient TBD -> +/-50ppm/C; Tolerance TBD -> +/-0.1%; VoltageRating TBD -> 25V
- R15, R16, R2, R3: Composition TBD -> Thick Film; MPN TBD -> RC0402FR-0722RP; Manufacturer TBD -> Yageo; PowerRating TBD -> 0.0625W; SelectionNote TBD -> Özdisan 839397; stok 4562 (21.09.2026); Uygun.; TempCoefficient TBD -> +/-100ppm/C; Tolerance TBD -> +/-1%; VoltageRating TBD -> 50V
- R24, R25, R26: Composition TBD -> High Power Thick Film; MPN TBD -> HP02WAF4701TCE; Manufacturer TBD -> Royalohm; PowerRating TBD -> 0.1W; SelectionNote TBD -> Özdisan 603918; stok 9400 (21.09.2026); Uygun.; TempCoefficient TBD -> +/-100ppm/C; Tolerance TBD -> +/-1%; VoltageRating TBD -> 50V
- SW1, SW2: Manufacturer C&K -> C&K (Littelfuse); SelectionNote TBD -> Özdisan 994927; stok 315791 (21.09.2026); Uygun.
- TP10, TP11, TP12, TP13, TP6, TP7, TP8, TP9: SelectionNote TBD -> Özdisan (21.09.2026): Satın alınmaz. Kart üzerindeki pad; s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
- U2: SelectionNote TBD -> Özdisan (21.09.2026): Stokta yok. 21.09 üçüncü tur: ESP32-C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
- U4: value RV-3028-C7 -> BQ32000; footprint Package_SON:MicroCrystal_C7_SON-8_1.5x3.2mm_P0.9mm -> Package_SO:SOIC-8_3.9x4.9mm_P1.27mm; symbol Timer_RTC:RV-3028-C7 -> Timer_RTC:BQ32000; ChannelCount TBD -> 1; DesignNote Trickle charge kapali kullanilacak. -> BQ32000: VCC 3.0-3.6V, I2C 0x68, IRQ open-drain (R24 pull-u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; Function RTC, I2C -> RTC, backup switchover, trickle charger; InterfaceType I2C -> I2C (0x68); LogicFamily TBD -> N/A; MPN RV-3028-C7 -> BQ32000DR; Manufacturer Micro Crystal -> Texas Instruments; OperatingTemp TBD -> -40C to 85C; OutputType TBD -> Open-drain IRQ; Package C7 SON-8 (1.5x3.2mm) -> SOIC-8; PinCount TBD -> 8; RoHS TBD -> Yes; SelectionNote TBD -> Özdisan 467622; stok 8985 (21.09.2026); Uygun. 21.09 RTC re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; SupplyVoltage TBD -> 3V to 3.6V; ThermalPad TBD -> No; TimekeepingAccuracy TBD -> +/-35ppm pre-calibration @25C
Connections:
- net +3.3V: now also R26.1, U4.8 (VCC); no longer R26.2, U4.7 (VDD)
- net GND: now also U4.4 (GND), C33.2, Y1.2 (G), Y1.3 (G); no longer U4.5 (VSS)
- net RTC_INT: now also U4.7 (~{IRQ}); no longer U4.2 (~{INT})
- net RTC_SCL: now also U4.6 (SCL); no longer U4.3 (SCL)
- net RTC_SDA: now also R26.2, U4.5 (SDA); no longer R26.1, U4.4 (SDA)
- net at U4.1 (OSCI): now also Y1.1
- new net: C33.1, U4.3 (VBACK)
- new net: U4.2 (OSCO), Y1.4
- no-connect marks 1 -> 0
Other:
- note added: "C33 Korchip DCL5R5155HF 1.5F/5.5V: BQ32000 trickle charge ile şarj. FW: TCHE=0x5, TCH2=1, TCFE=1 -> VBACK ~3.3V, ~3 hafta yedek. Y1 ABS25 CL=12.5pF: dahili yük kapasitesi, harici C YOK."
- note added: "RTC BQ32000 + 1F5 süper kapasitör"
- note removed: "BT1: L-KLS5-CR2032-05-R1 holder. CR2032 primary cell: disable RTC trickle charge. Pad 1 positive, pad 2 GND."
- note removed: "RTC RV-3028-C7 + CR2032"
- note removed: "RTC pil konusu netleştirilecek."
- moved on the sheet: C9, R24, R25, R26, U4

Commit message: hardware: ekranı TFT032B018'e geçir, todo'yu güncelle, Imax 3 A kararını kaydet
TFT032B018 (userinterface):
- J3 Conn_01x40 (Molex 54132-4062) -> Conn_01x30, KLS L-KLS1-242I-2.0-30-R;
  yeni footprint Connector_FPC_Custom:KLS_L-KLS1-242I-2.0-30_1x30-2MP_P0.50mm_Horizontal
  (fp-lib-table'a eklendi). SPI: 16=DC, 17=SCLK, 18=CS, 19=MOSI, 20=RST;
  21 IM=3.3V; DB0..7, RDX GND; TE ve dokunmatik pinleri boş. C34 1u0 dekuplaj.
- Backlight: TPS61023 boost (U7, L2, C20, C21, R44, R45) ve CAT4104 (U8,
  C22, R46) kalktı; +3.3V -> R60 5R6 -> BL_A, BL_K -> Q7 IRLML6344
  (R28/R29 ile TFT_BL_PWM).
- Beklenen netlist farkı: BACKLIGHT_4V2, BL_BOOST_*, BL_K1..4, Net-(U8-*)
  kalktı; BL_A, BL_K, Net-(Q7-G) eklendi; TFT_* netleri J3'ün yeni pin
  numaralarına geçti. ERC değişmedi (0 hata, 2 eski uyarı).
- Özdisan alanları (J3, Q7, R60, C34) ve BOM tablosu güncellendi; ekran modülü
  şema dışı satır olarak BOM'da (stok 5).
- mcu/userinterface: kullanılmayan lib_symbols tanımları silindi
  (Device:Battery_Cell, AO3400A); netlist farkı YOK.

Kayıtlar:
- todo.txt: tamamlanan şema maddeleri
  design_decisions/output/SEMA_TAMAMLANAN_TODO_REV_C_20260922.md'ye taşındı;
  AP74502Q sembolü Diodes datasheet'iyle doğrulandı (datasheet eklendi),
  U12 paket (SOT28) kontrolü ve SMBJ30A PCB maddesi güncellendi.
- Maksimum çıkış akımı 3 A: design_decisions/output/CIKIS_AKIMI_3A_KARARI_20260922.md.
  "Imax kesinleştir" ve "3.3 V adaptör başlığı" maddeleri kapandı; prototip ve
  INA226 firmware değerleri 3 A'e göre güncellendi, RShunt1 5 mOhm'da kaldı.

Co-Authored-By: Claude Opus 5 <noreply@anthropic.com>
Parts:
- C5: SelectionNote Özdisan 810882; stok 709 (21.09.2026); Uygun. 21.09 üçüncü tur: Footprint 0402 → 0805. 10V X6S (+105°C), 3.3V/4.2V raylarında 6.3V parçalardan daha az DC-bias kaybı; TPS61023/RT4812 çıkış efektif ≥4 µF şartını rahat karşılar. Ucuz alternatif: CL21A226MQQNNNE 6,3V X5R (47890 stok, 2,18 TL). -> Özdisan 810882; stok 709 (21.09.2026); Uygun. 21.09 üçüncü tur: Footprint 0402 → 0805. 10V X6S (+105°C); ESP32 +3.3V bulk. (22.09: C20/C21 TFT032B018 revizyonunda kalktı.)
- C7, C9: SelectionNote Özdisan 623573; stok 5005 (21.09.2026); Uygun. C4 (PD_5V) için ≥10V şartını karşılar. C9: BQ32000 VCC dekuplajı, datasheet ≥1 µF istiyor (100n → 1u0). -> Özdisan 623573; stok 5005 (21.09.2026); Uygun. C4 (PD_5V) için ≥10V şartını karşılar. C9: BQ32000 VCC dekuplajı, datasheet ≥1 µF istiyor (100n → 1u0). C34: TFT032B018 VCI/IOVCC dekuplajı (J3 yanında).
Changed lines of the file:
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@@
 			)
 		)
-		(property "SelectionNote" "Özdisan 623573; stok 5005 (21.09.2026); Uygun. C4 (PD_5V) için ≥10V şartını karşılar. C9: BQ32000 VCC dekuplajı, datasheet ≥1 µF istiyor (100n → 1u0)."
+		(property "SelectionNote" "Özdisan 623573; stok 5005 (21.09.2026); Uygun. C4 (PD_5V) için ≥10V şartını karşılar. C9: BQ32000 VCC dekuplajı, datasheet ≥1 µF istiyor (100n → 1u0). C34: TFT032B018 VCI/IOVCC dekuplajı (J3 yanında)."
 			(at 55.88 82.55 0)
 			(hide yes)
@@
 			)
 		)
-		(property "SelectionNote" "Özdisan 623573; stok 5005 (21.09.2026); Uygun. C4 (PD_5V) için ≥10V şartını karşılar. C9: BQ32000 VCC dekuplajı, datasheet ≥1 µF istiyor (100n → 1u0)."
+		(property "SelectionNote" "Özdisan 623573; stok 5005 (21.09.2026); Uygun. C4 (PD_5V) için ≥10V şartını karşılar. C9: BQ32000 VCC dekuplajı, datasheet ≥1 µF istiyor (100n → 1u0). C34: TFT032B018 VCI/IOVCC dekuplajı (J3 yanında)."
 			(at 234.95 57.15 0)
 			(hide yes)
@@
 			)
 		)
-		(property "SelectionNote" "Özdisan 810882; stok 709 (21.09.2026); Uygun. 21.09 üçüncü tur: Footprint 0402 → 0805. 10V X6S (+105°C), 3.3V/4.2V raylarında 6.3V parçalardan daha az DC-bias kaybı; TPS61023/RT4812 çıkış efektif ≥4 µF şartını rahat karşılar. Ucuz alternatif: CL21A226MQQNNNE 6,3V X5R (47890 stok, 2,18 TL)."
+		(property "SelectionNote" "Özdisan 810882; stok 709 (21.09.2026); Uygun. 21.09 üçüncü tur: Footprint 0402 → 0805. 10V X6S (+105°C); ESP32 +3.3V bulk. (22.09: C20/C21 TFT032B018 revizyonunda kalktı.)"
 			(at 124.46 69.85 0)
 			(hide yes)
